Commit message: Adjusted joints to revolute and added pretty realistic <limit> tags

File: orion_ws/src/orion_description/xacro/arm.xacro (robot description, xacro)
@@ -17,7 +17,7 @@
   <xacro:property name="base_z"        value="0.105"/>
   <xacro:property name="arm_mount_h"   value="0.024"/>
-  <xacro:property name="shoulder_h"    value="0.055"/>
-  <xacro:property name="upper_arm_l"   value="0.150"/>
-  <xacro:property name="forearm_l"     value="0.120"/>
+  <xacro:property name="shoulder_h"    value="0.12"/>
+  <xacro:property name="upper_arm_l"   value="0.15"/>
+  <xacro:property name="forearm_l"     value="0.06"/>
   <xacro:property name="hand_l"        value="0.055"/>
   <xacro:property name="r0"  value="0.020"/>
@@ -84,9 +84,10 @@
     <!-- base_link → shoulder  ── PITCH (Y)  ─────────────────────── -->
     <!-- No yaw: the mecanum base handles in-place rotation entirely.  -->
-    <joint name="shoulder_joint" type="continuous">
+    <joint name="shoulder_joint" type="revolute">
       <parent link="base_link"/>
       <child  link="shoulder_link"/>
       <origin xyz="0 0 ${base_z/2.0 + arm_mount_h}" rpy="0 0 0"/>
       <axis xyz="0 1 0"/>
+      <limit lower="-0.5" upper="1.5" effort="25.0" velocity="1.5"/>
       <dynamics damping="0.08" friction="0.10"/>
     </joint>
@@ -110,9 +111,10 @@
     </link>
     <!-- shoulder → upper_arm  ── PITCH (Y) ──────────────────────── -->
-    <joint name="elbow_joint" type="continuous">
+    <joint name="elbow_joint" type="revolute">
       <parent link="shoulder_link"/>
       <child  link="upper_arm_link"/>
       <origin xyz="0 0 ${shoulder_h}" rpy="0 0 0"/>
       <axis xyz="0 1 0"/>
+      <limit lower="-1" upper="1" effort="20.0" velocity="1.5"/>
       <dynamics damping="0.06" friction="0.08"/>
     </joint>
@@ -136,9 +138,10 @@
     </link>
     <!-- upper_arm → forearm  ── PITCH (Y) ───────────────────────── -->
-    <joint name="wrist_joint" type="continuous">
+    <joint name="wrist_joint" type="revolute">
       <parent link="upper_arm_link"/>
       <child  link="forearm_link"/>
       <origin xyz="${upper_arm_l} 0 0" rpy="0 0 0"/>
       <axis xyz="0 1 0"/>
+      <limit lower="0" upper="2.79" effort="15.0" velocity="2.0"/>
       <dynamics damping="0.04" friction="0.06"/>
     </joint>

File: orion_ws/src/orion_description/xacro/sensors.xacro (robot description, xacro)
@@ -1,20 +1,4 @@
 <?xml version="1.0"?>
 <robot xmlns:xacro="http://www.ros.org/wiki/xacro">
-  <!-- ================================================================
-       ORION SENSORS  —  LiDAR on rear mast
-         Max arm height above base_link (worst case — arm straight up):
-           shoulder mount  :  base_z/2 + arm_mount_h  = 0.0525 + 0.024  = 0.0765 m
-           shoulder riser  :  + 0.055                                    = 0.1315 m
-           upper_arm       :  + 0.150  (pointing straight up)            = 0.2815 m
-           forearm         :  + 0.120                                    = 0.4015 m
-         LiDAR scan plane must be above 0.40 m above base_link.
-         Mast height chosen so scan plane clears arm with 50 mm margin:
-           mast_h = 0.25 m  →  scan plane at base_z/2 + mast_h + lidar_h
-                             = 0.0525 + 0.25 + 0.041  ≈  0.344 m  ... insufficient
-         Use mast_h = 0.36 m:
-           scan plane  ≈  0.0525 + 0.36 + 0.041  =  0.454 m  ✓ (50 mm clear)
-         Mast is mounted at the rear of the base (x = −0.10 m) so it is
-         well behind the arm mount (x = 0) and does not obstruct the scan.
-       ================================================================ -->
   <xacro:property name="base_z"    value="0.105"/>
   <!-- Mast -->

Commit message: Resetting gazebo related files due to failed debugging

File: orion_ws/src/orion_description/xacro/arm.xacro (robot description, xacro)
@@ -222,87 +222,4 @@
       <origin xyz="0.050 0 0" rpy="0 0 0"/>
     </joint>
-    <!--Gazebo link colours-->
-    <gazebo reference="shoulder_link">   <material>Gazebo/Grey</material></gazebo>
-    <gazebo reference="upper_arm_link">  <material>Gazebo/Grey</material></gazebo>
-    <gazebo reference="forearm_link">    <material>Gazebo/Grey</material></gazebo>
-    <gazebo reference="hand_link">       <material>Gazebo/Grey</material></gazebo>
-    <gazebo reference="gripper_base_link"><material>Gazebo/DarkGrey</material></gazebo>
-    <gazebo reference="gripper_left_link"><material>Gazebo/Grey</material></gazebo>
-    <gazebo reference="gripper_right_link"><material>Gazebo/Grey</material></gazebo>
-    <!--Gazebo joint friction-->
-    <gazebo reference="shoulder_joint">
-      <implicitSpringDamper>true</implicitSpringDamper>
-      <provideFeedback>true</provideFeedback>
-    </gazebo>
-    <gazebo reference="elbow_joint">
-      <implicitSpringDamper>true</implicitSpringDamper>
-      <provideFeedback>true</provideFeedback>
-    </gazebo>
-    <gazebo reference="wrist_joint">
-      <implicitSpringDamper>true</implicitSpringDamper>
-      <provideFeedback>true</provideFeedback>
-    </gazebo>
-    <gazebo reference="wrist_roll_joint">
-      <implicitSpringDamper>true</implicitSpringDamper>
-      <provideFeedback>true</provideFeedback>
-    </gazebo>
-    <!--ROS2 Control plugin-->
-    <ros2_control name="orion_arm" type="system">
-      <hardware>
-        <plugin>gz_ros2_control/GazeboSimSystem</plugin>
-      </hardware>
-      <joint name="shoulder_joint">
-        <command_interface name="position"/>
-        <state_interface   name="position">
-          <param name="initial_value">0.0</param>
-        </state_interface>
-        <state_interface name="velocity"/>
-        <state_interface name="effort"/>
-      </joint>
-      <joint name="elbow_joint">
-        <command_interface name="position"/>
-        <state_interface   name="position">
-          <param name="initial_value">0.0</param>
-        </state_interface>
-        <state_interface name="velocity"/>
-        <state_interface name="effort"/>
-      </joint>
-      <joint name="wrist_joint">
-        <command_interface name="position"/>
-        <state_interface   name="position">
-          <param name="initial_value">0.0</param>
-        </state_interface>
-        <state_interface name="velocity"/>
-        <state_interface name="effort"/>
-      </joint>
-      <joint name="wrist_roll_joint">
-        <command_interface name="position"/>
-        <state_interface   name="position">
-          <param name="initial_value">0.0</param>
-        </state_interface>
-        <state_interface name="velocity"/>
-        <state_interface name="effort"/>
-      </joint>
-      <joint name="gripper_left_joint">
-        <command_interface name="position">
-          <param name="min">0.0</param>
-          <param name="max">0.025</param>
-        </command_interface>
-        <state_interface name="position">
-          <param name="initial_value">0.0</param>
-        </state_interface>
-        <state_interface name="velocity"/>
-      </joint>
-      <joint name="gripper_right_joint">
-        <command_interface name="position">
-          <param name="min">0.0</param>
-          <param name="max">0.025</param>
-        </command_interface>
-        <state_interface name="position">
-          <param name="initial_value">0.0</param>
-        </state_interface>
-        <state_interface name="velocity"/>
-      </joint>
-    </ros2_control>
   </xacro:macro>
 </robot>

File: orion_ws/src/orion_description/xacro/base.xacro (robot description, xacro)
@@ -64,30 +64,4 @@
       </inertial>
     </link>
-    <gazebo reference="base_link">
-      <material>Gazebo/DarkGrey</material>
-      <surface>
-        <friction>
-          <ode>
-            <mu>0.3</mu>
-            <mu2>0.3</mu2>
-          </ode>
-        </friction>
-        <contact>
-          <ode>
-            <kp>1e6</kp>
-            <kd>100.0</kd>
-          </ode>
-        </contact>
-      </surface>
-    </gazebo>
-    <gazebo>
-      <plugin filename="gz_ros2_control-system"
-              name="gz_ros2_control::GazeboSimROS2ControlPlugin">
-        <parameters>$(find orion_description)/config/ros2_controllers.yaml</parameters>
-        <ros>
-          <remapping>~/robot_description:=/robot_description</remapping>
-        </ros>
-      </plugin>
-    </gazebo>
   </xacro:macro>
 </robot>

File: orion_ws/src/orion_description/xacro/orion.xacro (robot description, xacro)
@@ -12,14 +12,3 @@
   <xacro:sensors/>
   <xacro:arm/>
-  <!--GZ Sensor activation system-->
-  <gazebo>
-    <plugin filename="gz-sim-sensors-system"
-            name="gz::sim::systems::Sensors">
-      <render_engine>ogre2</render_engine>
-    </plugin>
-  </gazebo>
-  <gazebo>
-    <plugin filename="gz-sim-imu-system"
-            name="gz::sim::systems::Imu"/>
-  </gazebo>
 </robot>

File: orion_ws/src/orion_description/xacro/sensors.xacro (robot description, xacro)
@@ -75,46 +75,4 @@
       <origin xyz="0 0 ${mast_h}" rpy="0 0 0"/>
     </joint>
-    <!--LiDAR GZ Plugin-->
-    <gazebo reference="lidar_link">
-      <material>Gazebo/Black</material>
-      <sensor name="lidar_sensor" type="gpu_lidar">
-        <pose>0 0 ${lidar_h/2.0} 0 0 0</pose>
-        <topic>/scan</topic>
-        <gz_frame_id>lidar_link</gz_frame_id>
-        <update_rate>10</update_rate>
-        <visualize>false</visualize>
-        <always_on>true</always_on>
-        <lidar>
-          <scan>
-            <horizontal>
-              <samples>360</samples>
-              <resolution>1</resolution>
-              <min_angle>-3.14159265</min_angle>
-              <max_angle> 3.14159265</max_angle>
-            </horizontal>
-            <vertical>
-              <samples>1</samples>
-              <resolution>1</resolution>
-              <min_angle>0</min_angle>
-              <max_angle>0</max_angle>
-            </vertical>
-          </scan>
-          <range>
-            <min>0.15</min>
-            <max>12.0</max>
-            <resolution>0.01</resolution>
-          </range>
-          <noise>
-            <type>gaussian</type>
-            <mean>0.0</mean>
-            <stddev>0.005</stddev>
-          </noise>
-        </lidar>
-      </sensor>
-    </gazebo>
-    <!-- Mast colour -->
-    <gazebo reference="lidar_mast_link">
-      <material>Gazebo/DarkGrey</material>
-    </gazebo>
     <!--IMU Link-->
     <link name="imu_link">
@@ -138,25 +96,4 @@
       <origin xyz="0 0 ${base_z}" rpy="0 0 0"/>
     </joint>
-    <!--IMU Gz plugin-->
-    <gazebo reference="imu_link">
-      <sensor name="imu_sensor" type="imu">
-        <always_on>true</always_on>
-        <update_rate>100</update_rate>
-        <topic>/imu/data</topic>
-        <gz_frame_id>imu_link</gz_frame_id>
-        <imu>
-          <angular_velocity>
-            <x><noise type="gaussian" mean="0" stddev="0.001"/></x>
-            <y><noise type="gaussian" mean="0" stddev="0.001"/></y>
-            <z><noise type="gaussian" mean="0" stddev="0.001"/></z>
-          </angular_velocity>
-          <linear_acceleration>
-            <x><noise type="gaussian" mean="0" stddev="0.01"/></x>
-            <y><noise type="gaussian" mean="0" stddev="0.01"/></y>
-            <z><noise type="gaussian" mean="0" stddev="0.01"/></z>
-          </linear_acceleration>
-        </imu>
-      </sensor>
-    </gazebo>
   </xacro:macro>
 </robot>

File: orion_ws/src/orion_description/xacro/wheels.xacro (robot description, xacro)
@@ -41,60 +41,10 @@
       <dynamics damping="0.01" friction="0.01"/>
     </joint>
-    <gazebo reference="${name}_wheel_link">
-      <material>Gazebo/Black</material>
-      <collision>
-        <surface>
-          <friction>
-            <ode>
-              <mu>1.0</mu>
-              <mu2>0.1</mu2>
-              <fdir1>0.7071 ${fdir1_y} 0</fdir1>
-            </ode>
-          </friction>
-          <contact>
-            <ode>
-              <kp>1e6</kp>
-              <kd>1.0</kd>
-              <min_depth>0.001</min_depth>
-              <max_vel>0.1</max_vel>
-            </ode>
-          </contact>
-        </surface>
-      </collision>
-    </gazebo>
   </xacro:macro>
   <xacro:macro name="wheels">
-    <!-- Signs have NO leading spaces: "1" not " 1", "-1" not "-1" -->
     <xacro:mecanum_wheel name="front_left"  x_sign="1"  y_sign="1"  fdir1_y="-0.7071"/>
     <xacro:mecanum_wheel name="front_right" x_sign="1"  y_sign="-1" fdir1_y="0.7071"/>
     <xacro:mecanum_wheel name="rear_left"   x_sign="-1" y_sign="1"  fdir1_y="0.7071"/>
     <xacro:mecanum_wheel name="rear_right"  x_sign="-1" y_sign="-1" fdir1_y="-0.7071"/>
-    <!-- ros2_control block — all 4 wheels velocity-controlled via
-         forward_command_controller + mecanum_ik_node. -->
-    <ros2_control name="orion_base" type="system">
-      <hardware>
-        <plugin>gz_ros2_control/GazeboSimSystem</plugin>
-      </hardware>
-      <joint name="front_left_wheel_joint">
-        <command_interface name="velocity"/>
-        <state_interface name="position"/>
-        <state_interface name="velocity"/>
-      </joint>
-      <joint name="front_right_wheel_joint">
-        <command_interface name="velocity"/>
-        <state_interface name="position"/>
-        <state_interface name="velocity"/>
-      </joint>
-      <joint name="rear_left_wheel_joint">
-        <command_interface name="velocity"/>
-        <state_interface name="position"/>
-        <state_interface name="velocity"/>
-      </joint>
-      <joint name="rear_right_wheel_joint">
-        <command_interface name="velocity"/>
-        <state_interface name="position"/>
-        <state_interface name="velocity"/>
-      </joint>
-    </ros2_control>
   </xacro:macro>
 </robot>
