Commit message: Added <ros2_control> blocks to wheels.xacro and base.xacro. Updated ros2_controllers.yaml to use mecanum_drive_controller/MecanumDriveController instead of wheel_velocity_controller/WheelVelocityController

File: orion_ws/src/orion_description/xacro/base.xacro (robot description, xacro)
@@ -64,4 +64,9 @@
       </inertial>
     </link>
+    <gazebo>
+      <plugin filename="gz_ros2_control-system" name="gz_ros2_control::GazeboSimROS2ControlPlugin">
+        <parameters>$(find orion_description)/config/ros2_controllers.yaml</parameters>
+      </plugin>
+    <gazebo>
   </xacro:macro>
 </robot>

File: orion_ws/src/orion_description/xacro/wheels.xacro (robot description, xacro)
@@ -41,4 +41,17 @@
       <dynamics damping="0.01" friction="0.01"/>
     </joint>
+    <gazebo reference="${name}_wheel_link">
+      <collision>
+        <surface>
+          <friction>
+            <ode>
+              <mu>1.0</mu>
+              <mu2>0.1</mu2>
+              <fdir1>1 $(fdir1_y) 0 </fdir1>
+            </ode>
+          </friction>
+        </surface>
+      </collision>
+    </gazebo>
   </xacro:macro>
   <xacro:macro name="wheels">
