Commit message: Initial attempt at modelling base_link and shoulder_link

File: orion_ws/src/orion_description/xacro/orion.xacro (robot description, xacro)
@@ -20,7 +20,7 @@
       <!-- Inertia tensor must be relative to COM, not world -->
       <inertia
-        ixx="0.05067488516"
-        iyy="0.05067488516"
-        izz="0.05968310366"
+        ixx="0.05"
+        iyy="0.05"
+        izz="0.06"
         ixy="0.0"
         ixz="0.0"
@@ -28,8 +28,7 @@
     </inertial>
     <visual>
-      <!-- Position relative to the link -->
       <origin xyz="0 0 0.25" rpy="0 0 0"/>
       <geometry>
-        <cylinder radius="0.3454941495" length="0.5"/>
+        <cylinder radius="0.2" length="0.5"/>
       </geometry>
       <material name="cyan">
@@ -43,5 +42,5 @@
     <child link="shoulder_link"/>
     <!-- Joint is at top of base -->
-    <origin xyz="0 0 0.1" rpy="0 0 0"/>
+    <origin xyz="0 0 0.2" rpy="0 0 0"/>
     <axis xyz="0 0 1"/>
   </joint>

Commit message: Update orion.xacro with improved properties and collision models, fix launch file duplicate nodes

File: orion_ws/src/orion_description/xacro/orion.xacro (robot description, xacro)
@@ -1,47 +1,72 @@
 <?xml version="1.0"?>
 <robot name="orion" xmlns:xacro="http://www.ros.org/wiki/xacro">
-  <!-- ================= BASE LINK ================= -->
+  <xacro:property name="base_size" value="0.5 0.5 0.2"/>
+  <xacro:property name="shoulder_radius" value="0.2"/>
+  <xacro:property name="shoulder_length" value="0.5"/>
+  <xacro:property name="link1_radius" value="0.15"/>
+  <xacro:property name="link1_length" value="1.0"/>
+  <xacro:property name="base_mass" value="2.0"/>
+  <xacro:property name="shoulder_mass" value="1.0"/>
+  <xacro:property name="link1_mass" value="1.0"/>
   <link name="base_link">
+    <inertial>
+      <origin xyz="0 0 0" rpy="0 0 0"/>
+      <mass value="${base_mass}"/>
+      <inertia ixx="0.08" iyy="0.08" izz="0.08" ixy="0.0" ixz="0.0" iyz="0.0"/>
+    </inertial>
     <visual>
-      <geometry>
-        <box size="0.5 0.5 0.2"/>
-      </geometry>
-      <material name="blue">
-        <color rgba="0 0 1 1"/>
-      </material>
+      <origin xyz="0 0 0" rpy="0 0 0"/>
+      <geometry><box size="${base_size}"/></geometry>
+      <material name="blue"><color rgba="0 0 1 1"/></material>
     </visual>
+    <collision>
+      <origin xyz="0 0 0" rpy="0 0 0"/>
+      <geometry><box size="${base_size}"/></geometry>
+    </collision>
   </link>
-  <!-- ================= SHOULDER LINK ================= -->
   <link name="shoulder_link">
     <inertial>
-      <!-- Keep inertial at the link origin (IMPORTANT) -->
-      <origin xyz="0 0 0" rpy="0 0 0"/>
-      <mass value="1"/>
-      <!-- Inertia tensor must be relative to COM, not world -->
-      <inertia
-        ixx="0.05"
-        iyy="0.05"
-        izz="0.06"
-        ixy="0.0"
-        ixz="0.0"
-        iyz="0.0"/>
+      <origin xyz="0 0 ${shoulder_length/2}" rpy="0 0 0"/>
+      <mass value="${shoulder_mass}"/>
+      <inertia ixx="0.02" iyy="0.02" izz="0.02" ixy="0.0" ixz="0.0" iyz="0.0"/>
     </inertial>
     <visual>
-      <origin xyz="0 0 0.25" rpy="0 0 0"/>
-      <geometry>
-        <cylinder radius="0.2" length="0.5"/>
-      </geometry>
-      <material name="cyan">
-        <color rgba="0 1.0 1.0 1.0"/>
-      </material>
+      <origin xyz="0 0 ${shoulder_length/2}" rpy="0 0 0"/>
+      <geometry><cylinder radius="${shoulder_radius}" length="${shoulder_length}"/></geometry>
+      <material name="cyan"><color rgba="0 1 1 1"/></material>
     </visual>
+    <collision>
+      <origin xyz="0 0 ${shoulder_length/2}" rpy="0 0 0"/>
+      <geometry><cylinder radius="${shoulder_radius}" length="${shoulder_length}"/></geometry>
+    </collision>
   </link>
-  <!-- ================= JOINT ================= -->
   <joint name="shoulder_joint" type="continuous">
     <parent link="base_link"/>
     <child link="shoulder_link"/>
-    <!-- Joint is at top of base -->
-    <origin xyz="0 0 0.2" rpy="0 0 0"/>
+    <origin xyz="0 0 0.1" rpy="0 0 0"/>
     <axis xyz="0 0 1"/>
   </joint>
+  <link name="link1">
+    <inertial>
+      <origin xyz="0 0 ${link1_length/2}" rpy="0 0 0"/>
+      <mass value="${link1_mass}"/>
+      <inertia ixx="0.02" iyy="0.02" izz="0.02" ixy="0.0" ixz="0.0" iyz="0.0"/>
+    </inertial>
+    <visual>
+      <origin xyz="0 0 ${link1_length/2}" rpy="0 0 0"/>
+      <geometry><cylinder radius="${link1_radius}" length="${link1_length}"/></geometry>
+      <material name="cyan"><color rgba="0 1 1 1"/></material>
+    </visual>
+    <collision>
+      <origin xyz="0 0 ${link1_length/2}" rpy="0 0 0"/>
+      <geometry><cylinder radius="${link1_radius}" length="${link1_length}"/></geometry>
+    </collision>
+  </link>
+  <joint name="shoulder_to_link1_joint" type="revolute">
+    <parent link="shoulder_link"/>
+    <child link="link1"/>
+    <origin xyz="0 0 ${shoulder_length}" rpy="0 0 0"/>
+    <axis xyz="0 1 0"/>
+    <limit lower="-1.57" upper="1.57" effort="10" velocity="1.0"/>
+  </joint>
 </robot>

Commit message: Add parameters and update robot structure in xacro

File: orion_ws/src/orion_description/xacro/orion.xacro (robot description, xacro)
@@ -1,72 +1,190 @@
 <?xml version="1.0"?>
 <robot name="orion" xmlns:xacro="http://www.ros.org/wiki/xacro">
-  <xacro:property name="base_size" value="0.5 0.5 0.2"/>
-  <xacro:property name="shoulder_radius" value="0.2"/>
-  <xacro:property name="shoulder_length" value="0.5"/>
-  <xacro:property name="link1_radius" value="0.15"/>
-  <xacro:property name="link1_length" value="1.0"/>
-  <xacro:property name="base_mass" value="2.0"/>
-  <xacro:property name="shoulder_mass" value="1.0"/>
-  <xacro:property name="link1_mass" value="1.0"/>
+  <!-- ================= PARAMETERS ================= -->
+  <xacro:property name="wheel_radius" value="0.05"/>
+  <xacro:property name="wheel_width" value="0.02"/>
+  <xacro:property name="wheel_sep" value="0.20"/>
+  <xacro:property name="arm_length" value="0.2"/>
+  <xacro:property name="arm_radius" value="0.02"/>
+  <!-- ================= BASE ================= -->
   <link name="base_link">
-    <inertial>
-      <origin xyz="0 0 0" rpy="0 0 0"/>
-      <mass value="${base_mass}"/>
-      <inertia ixx="0.08" iyy="0.08" izz="0.08" ixy="0.0" ixz="0.0" iyz="0.0"/>
-    </inertial>
     <visual>
-      <origin xyz="0 0 0" rpy="0 0 0"/>
-      <geometry><box size="${base_size}"/></geometry>
-      <material name="blue"><color rgba="0 0 1 1"/></material>
+      <geometry>
+        <box size="0.3 0.2 0.1"/>
+      </geometry>
     </visual>
     <collision>
-      <origin xyz="0 0 0" rpy="0 0 0"/>
-      <geometry><box size="${base_size}"/></geometry>
+      <geometry>
+        <box size="0.3 0.2 0.1"/>
+      </geometry>
     </collision>
+    <inertial>
+      <mass value="2.0"/>
+      <origin xyz="0 0 0"/>
+      <inertia ixx="0.02" iyy="0.02" izz="0.02"
+               ixy="0.0" ixz="0.0" iyz="0.0"/>
+    </inertial>
   </link>
+  <!-- ================= WHEELS ================= -->
+  <xacro:macro name="wheel" params="name y_pos">
+    <link name="${name}">
+      <visual>
+        <geometry>
+          <cylinder radius="${wheel_radius}" length="${wheel_width}"/>
+        </geometry>
+        <origin rpy="1.57 0 0"/>
+      </visual>
+      <inertial>
+        <mass value="0.5"/>
+        <origin xyz="0 0 0"/>
+        <inertia ixx="0.001" iyy="0.001" izz="0.0005"
+                 ixy="0.0" ixz="0.0" iyz="0.0"/>
+      </inertial>
+    </link>
+    <joint name="${name}_joint" type="continuous">
+      <parent link="base_link"/>
+      <child link="${name}"/>
+      <origin xyz="0 ${y_pos} -0.05"/>
+      <axis xyz="0 1 0"/>
+    </joint>
+  </xacro:macro>
+  <xacro:wheel name="left_wheel"  y_pos="${wheel_sep/2}"/>
+  <xacro:wheel name="right_wheel" y_pos="-${wheel_sep/2}"/>
+  <!-- ================= CASTER ================= -->
+  <link name="caster">
+    <visual>
+      <geometry>
+        <sphere radius="0.03"/>
+      </geometry>
+    </visual>
+  </link>
+  <joint name="caster_joint" type="fixed">
+    <parent link="base_link"/>
+    <child link="caster"/>
+    <origin xyz="-0.1 0 -0.05"/>
+  </joint>
+  <!-- ================= SHOULDER ================= -->
   <link name="shoulder_link">
+    <visual>
+      <geometry>
+        <box size="0.05 0.05 0.05"/>
+      </geometry>
+    </visual>
     <inertial>
-      <origin xyz="0 0 ${shoulder_length/2}" rpy="0 0 0"/>
-      <mass value="${shoulder_mass}"/>
-      <inertia ixx="0.02" iyy="0.02" izz="0.02" ixy="0.0" ixz="0.0" iyz="0.0"/>
+      <mass value="0.3"/>
+      <origin xyz="0 0 0"/>
+      <inertia ixx="0.000125" iyy="0.000125" izz="0.000125"
+               ixy="0.0" ixz="0.0" iyz="0.0"/>
     </inertial>
-    <visual>
-      <origin xyz="0 0 ${shoulder_length/2}" rpy="0 0 0"/>
-      <geometry><cylinder radius="${shoulder_radius}" length="${shoulder_length}"/></geometry>
-      <material name="cyan"><color rgba="0 1 1 1"/></material>
-    </visual>
-    <collision>
-      <origin xyz="0 0 ${shoulder_length/2}" rpy="0 0 0"/>
-      <geometry><cylinder radius="${shoulder_radius}" length="${shoulder_length}"/></geometry>
-    </collision>
   </link>
-  <joint name="shoulder_joint" type="continuous">
+  <joint name="shoulder_joint" type="revolute">
     <parent link="base_link"/>
     <child link="shoulder_link"/>
-    <origin xyz="0 0 0.1" rpy="0 0 0"/>
+    <origin xyz="0 0 0.1"/>
     <axis xyz="0 0 1"/>
   </joint>
+  <!-- ================= ARM LINK 1 ================= -->
   <link name="link1">
+    <visual>
+      <geometry>
+        <cylinder radius="${arm_radius}" length="${arm_length}"/>
+      </geometry>
+      <origin rpy="0 1.57 0"/>
+    </visual>
     <inertial>
-      <origin xyz="0 0 ${link1_length/2}" rpy="0 0 0"/>
-      <mass value="${link1_mass}"/>
-      <inertia ixx="0.02" iyy="0.02" izz="0.02" ixy="0.0" ixz="0.0" iyz="0.0"/>
+      <mass value="1.0"/>
+      <origin xyz="0 0 0"/>
+      <inertia ixx="0.0034" iyy="0.0034" izz="0.0002"
+               ixy="0.0" ixz="0.0" iyz="0.0"/>
     </inertial>
-    <visual>
-      <origin xyz="0 0 ${link1_length/2}" rpy="0 0 0"/>
-      <geometry><cylinder radius="${link1_radius}" length="${link1_length}"/></geometry>
-      <material name="cyan"><color rgba="0 1 1 1"/></material>
-    </visual>
-    <collision>
-      <origin xyz="0 0 ${link1_length/2}" rpy="0 0 0"/>
-      <geometry><cylinder radius="${link1_radius}" length="${link1_length}"/></geometry>
-    </collision>
   </link>
-  <joint name="shoulder_to_link1_joint" type="revolute">
+  <joint name="joint1" type="revolute">
     <parent link="shoulder_link"/>
     <child link="link1"/>
-    <origin xyz="0 0 ${shoulder_length}" rpy="0 0 0"/>
+    <origin xyz="0 0 0.05"/>
     <axis xyz="0 1 0"/>
-    <limit lower="-1.57" upper="1.57" effort="10" velocity="1.0"/>
   </joint>
+  <!-- ================= ARM LINK 2 ================= -->
+  <link name="link2">
+    <visual>
+      <geometry>
+        <cylinder radius="${arm_radius}" length="${arm_length}"/>
+      </geometry>
+      <origin rpy="0 1.57 0"/>
+    </visual>
+    <inertial>
+      <mass value="0.8"/>
+      <origin xyz="0 0 0"/>
+      <inertia ixx="0.0027" iyy="0.0027" izz="0.00016"
+               ixy="0.0" ixz="0.0" iyz="0.0"/>
+    </inertial>
+  </link>
+  <joint name="joint2" type="revolute">
+    <parent link="link1"/>
+    <child link="link2"/>
+    <origin xyz="0 0 ${arm_length}"/>
+    <axis xyz="0 1 0"/>
+  </joint>
+  <!-- ================= SENSORS ================= -->
+  <!-- LiDAR -->
+  <link name="lidar_link">
+    <visual>
+      <geometry>
+        <cylinder radius="0.03" length="0.05"/>
+      </geometry>
+    </visual>
+  </link>
+  <joint name="lidar_joint" type="fixed">
+    <parent link="base_link"/>
+    <child link="lidar_link"/>
+    <origin xyz="0.1 0 0.15"/>
+  </joint>
+  <!-- IMU -->
+  <link name="imu_link"/>
+  <joint name="imu_joint" type="fixed">
+    <parent link="base_link"/>
+    <child link="imu_link"/>
+    <origin xyz="0 0 0.1"/>
+  </joint>
+  <!-- Camera -->
+  <link name="camera_link">
+    <visual>
+      <geometry>
+        <box size="0.03 0.03 0.03"/>
+      </geometry>
+    </visual>
+  </link>
+  <joint name="camera_joint" type="fixed">
+    <parent link="base_link"/>
+    <child link="camera_link"/>
+    <origin xyz="0.15 0 0.2"/>
+  </joint>
+  <!-- ================= ROS2 CONTROL ================= -->
+  <ros2_control name="orion_system" type="system">
+    <hardware>
+      <plugin>gazebo_ros2_control/GazeboSystem</plugin>
+    </hardware>
+    <joint name="left_wheel_joint">
+      <command_interface name="velocity"/>
+      <state_interface name="velocity"/>
+      <state_interface name="position"/>
+    </joint>
+    <joint name="right_wheel_joint">
+      <command_interface name="velocity"/>
+      <state_interface name="velocity"/>
+      <state_interface name="position"/>
+    </joint>
+    <joint name="shoulder_joint">
+      <command_interface name="position"/>
+      <state_interface name="position"/>
+    </joint>
+    <joint name="joint1">
+      <command_interface name="position"/>
+      <state_interface name="position"/>
+    </joint>
+    <joint name="joint2">
+      <command_interface name="position"/>
+      <state_interface name="position"/>
+    </joint>
+  </ros2_control>
 </robot>

Commit message: Made a couple refinements to Model 1

File: orion_ws/src/orion_description/xacro/orion.xacro (robot description, xacro)
@@ -2,9 +2,9 @@
 <robot name="orion" xmlns:xacro="http://www.ros.org/wiki/xacro">
   <!-- ================= PARAMETERS ================= -->
-  <xacro:property name="wheel_radius" value="0.08"/>
-  <xacro:property name="wheel_width" value="0.04"/>
-  <xacro:property name="wheel_sep" value="0.30"/>
-  <xacro:property name="arm_length" value="0.30"/>
-  <xacro:property name="arm_radius" value="0.03"/>
+<xacro:property name="wheel_radius" value="0.08"/>
+<xacro:property name="wheel_width" value="0.04"/>
+<xacro:property name="wheel_sep" value="0.30"/>
+<xacro:property name="arm_length" value="0.30"/>
+<xacro:property name="arm_radius" value="0.03"/>
   <!-- ================= BASE ================= -->
   <link name="base_link">
@@ -14,44 +14,41 @@
       </geometry>
       <material name="Blue">
-      <color rgba="0 0 1 1"/>
+        <color rgba="0 0 1 1"/>
       </material>
     </visual>
-    <collision>
-      <geometry>
-        <box size="0.5 0.4 0.15"/>
-      </geometry>
-    </collision>
-    <inertial>
-      <mass value="5.0"/>
-      <origin xyz="0 0 0"/>
-      <inertia ixx="0.1" iyy="0.1" izz="0.1"
-               ixy="0.0" ixz="0.0" iyz="0.0"/>
-    </inertial>
+```
+<collision>
+  <geometry>
+    <box size="0.3 0.2 0.15"/>
+  </geometry>
+</collision>
+<inertial>
+  <mass value="5.0"/>
+  <origin xyz="0 0 0"/>
+  <inertia ixx="0.1" iyy="0.1" izz="0.1"
+           ixy="0.0" ixz="0.0" iyz="0.0"/>
+</inertial>
+```
   </link>
   <!-- ================= WHEELS ================= -->
-  <xacro:macro name="wheel" params="name y_pos">
-    <link name="${name}">
-      <visual>
-        <geometry>
-          <cylinder radius="${wheel_radius}" length="${wheel_width}"/>
-        </geometry>
-        <origin rpy="1.57 0 0"/>
-      </visual>
-      <inertial>
-        <mass value="1.0"/>
-        <origin xyz="0 0 0"/>
-        <inertia ixx="0.005" iyy="0.005" izz="0.01"
-                 ixy="0.0" ixz="0.0" iyz="0.0"/>
-      </inertial>
-    </link>
-    <joint name="${name}_joint" type="continuous">
-      <parent link="base_link"/>
-      <child link="${name}"/>
-      <origin xyz="0 ${y_pos} -0.05"/>
-      <axis xyz="0 1 0"/>
-    </joint>
-  </xacro:macro>
-  <xacro:wheel name="left_wheel"  y_pos="${wheel_sep/2}"/>
-  <xacro:wheel name="right_wheel" y_pos="-${wheel_sep/2}"/>
+<xacro:macro name="wheel" params="name y_pos"> <link name="${name}"> <visual> <geometry> <cylinder radius="${wheel_radius}" length="${wheel_width}"/> </geometry> <origin rpy="1.57 0 0"/> </visual>
+```
+  <inertial>
+    <mass value="1.0"/>
+    <origin xyz="0 0 0"/>
+    <inertia ixx="0.005" iyy="0.005" izz="0.01"
+             ixy="0.0" ixz="0.0" iyz="0.0"/>
+  </inertial>
+</link>
+<joint name="${name}_joint" type="continuous">
+  <parent link="base_link"/>
+  <child link="${name}"/>
+  <origin xyz="0 ${y_pos} -${wheel_radius}"/>
+  <axis xyz="0 1 0"/>
+</joint>
+```
+</xacro:macro>
+<xacro:wheel name="left_wheel"  y_pos="${wheel_sep/2}"/>
+<xacro:wheel name="right_wheel" y_pos="-${wheel_sep/2}"/>
   <!-- ================= CASTER ================= -->
   <link name="caster">
@@ -74,10 +71,12 @@
       </geometry>
     </visual>
-    <inertial>
-      <mass value="0.5"/>
-      <origin xyz="0 0 0"/>
-      <inertia ixx="0.0005" iyy="0.0005" izz="0.0005"
-               ixy="0.0" ixz="0.0" iyz="0.0"/>
-    </inertial>
+```
+<inertial>
+  <mass value="0.5"/>
+  <origin xyz="0 0 0"/>
+  <inertia ixx="0.0005" iyy="0.0005" izz="0.0005"
+           ixy="0.0" ixz="0.0" iyz="0.0"/>
+</inertial>
+```
   </link>
   <joint name="shoulder_joint" type="continuous">
@@ -93,15 +92,17 @@
         <cylinder radius="${arm_radius}" length="${arm_length}"/>
       </geometry>
-      <origin xyz= "0.15 0 0" rpy="0 1.57 0"/>
+      <origin xyz="${arm_length/2} 0 0" rpy="0 1.57 0"/>
       <material name="Blue">
-      <color rgba="0 0 1 1"/>
+        <color rgba="0 0 1 1"/>
       </material>
     </visual>
-    <inertial>
-      <mass value="2.0"/>
-      <origin xyz="0 0 0"/>
-      <inertia ixx="0.01" iyy="0.01" izz="0.005"
-               ixy="0.0" ixz="0.0" iyz="0.0"/>
-    </inertial>
+```
+<inertial>
+  <mass value="2.0"/>
+  <origin xyz="${arm_length/2} 0 0"/>
+  <inertia ixx="0.01" iyy="0.01" izz="0.005"
+           ixy="0.0" ixz="0.0" iyz="0.0"/>
+</inertial>
+```
   </link>
   <joint name="joint1" type="revolute">
@@ -118,17 +119,19 @@
         <cylinder radius="${arm_radius}" length="${arm_length}"/>
       </geometry>
-      <origin xyz="0.15 0 0" rpy="0 1.57 0"/>
+      <origin xyz="${arm_length/2} 0 0" rpy="0 1.57 0"/>
     </visual>
-    <inertial>
-      <mass value="1.5"/>
-      <origin xyz="0 0 0"/>
-      <inertia ixx="0.0075" iyy="0.0075" izz="0.00375"
-               ixy="0.0" ixz="0.0" iyz="0.0"/>
-    </inertial>
+```
+<inertial>
+  <mass value="1.5"/>
+  <origin xyz="${arm_length/2} 0 0"/>
+  <inertia ixx="0.0075" iyy="0.0075" izz="0.00375"
+           ixy="0.0" ixz="0.0" iyz="0.0"/>
+</inertial>
+```
   </link>
   <joint name="joint2" type="revolute">
     <parent link="link1"/>
     <child link="link2"/>
-    <origin xyz="0.3 0 0"/>
+    <origin xyz="${arm_length} 0 0"/>
     <axis xyz="0 1 0"/>
     <limit lower="-1.57" upper="1.57" effort="10" velocity="1.0"/>
@@ -138,7 +141,11 @@
   <link name="lidar_link">
     <visual>
-      <geometry>
-        <cylinder radius="0.03" length="0.05"/>
-      </geometry>
+    <geometry>
+        <cylinder radius="0.05" length="0.01"/>
+    </geometry>
+    <origin xyz="0 0 0" rpy="0 0 0"/>
+    <material name="Green">
+        <color rgba="0 1 0 1"/>
+    </material>
     </visual>
   </link>
@@ -146,40 +153,39 @@
     <parent link="base_link"/>
     <child link="lidar_link"/>
-    <origin xyz="0.1 0 0.07"/>
+    <origin xyz="0.1 0 0.075"/>
   </joint>
   <!-- IMU -->
   <link name="imu_link"/>
   <joint name="imu_joint" type="fixed">
-    <parent link="shoulder_link"/>
+    <parent link="base_link"/>
     <child link="imu_link"/>
     <origin xyz="0 0 0.1"/>
   </joint>
   <!-- ================= ROS2 CONTROL ================= -->
-  <ros2_control name="orion_system" type="system">
-    <hardware>
-      <plugin>gazebo_ros2_control/GazeboSystem</plugin>
-    </hardware>
-    <joint name="left_wheel_joint">
-      <command_interface name="velocity"/>
-      <state_interface name="velocity"/>
-      <state_interface name="position"/>
-    </joint>
-    <joint name="right_wheel_joint">
-      <command_interface name="velocity"/>
-      <state_interface name="velocity"/>
-      <state_interface name="position"/>
-    </joint>
-    <joint name="shoulder_joint">
-      <command_interface name="position"/>
-      <state_interface name="position"/>
-    </joint>
-    <joint name="joint1">
-      <command_interface name="position"/>
-      <state_interface name="position"/>
-    </joint>
-    <joint name="joint2">
-      <command_interface name="position"/>
-      <state_interface name="position"/>
-    </joint>
-  </ros2_control>
+<ros2_control name="orion_system" type="system"> <hardware> <plugin>gazebo_ros2_control/GazeboSystem</plugin> </hardware>
+```
+<joint name="left_wheel_joint">
+  <command_interface name="velocity"/>
+  <state_interface name="velocity"/>
+  <state_interface name="position"/>
+</joint>
+<joint name="right_wheel_joint">
+  <command_interface name="velocity"/>
+  <state_interface name="velocity"/>
+  <state_interface name="position"/>
+</joint>
+<joint name="shoulder_joint">
+  <command_interface name="position"/>
+  <state_interface name="position"/>
+</joint>
+<joint name="joint1">
+  <command_interface name="position"/>
+  <state_interface name="position"/>
+</joint>
+<joint name="joint2">
+  <command_interface name="position"/>
+  <state_interface name="position"/>
+</joint>
+```
+</ros2_control>
 </robot>
