Commit message: Redesigned ORION to Model 2

File: orion_ws/src/orion_description/xacro/orion.xacro (robot description, xacro)
@@ -1,191 +1,13 @@
 <?xml version="1.0"?>
 <robot name="orion" xmlns:xacro="http://www.ros.org/wiki/xacro">
-  <!-- ================= PARAMETERS ================= -->
-<xacro:property name="wheel_radius" value="0.08"/>
-<xacro:property name="wheel_width" value="0.04"/>
-<xacro:property name="wheel_sep" value="0.30"/>
-<xacro:property name="arm_length" value="0.30"/>
-<xacro:property name="arm_radius" value="0.03"/>
-  <!-- ================= BASE ================= -->
-  <link name="base_link">
-    <visual>
-      <geometry>
-        <box size="0.3 0.2 0.15"/>
-      </geometry>
-      <material name="Blue">
-        <color rgba="0 0 1 1"/>
-      </material>
-    </visual>
-```
-<collision>
-  <geometry>
-    <box size="0.3 0.2 0.15"/>
-  </geometry>
-</collision>
-<inertial>
-  <mass value="5.0"/>
-  <origin xyz="0 0 0"/>
-  <inertia ixx="0.1" iyy="0.1" izz="0.1"
-           ixy="0.0" ixz="0.0" iyz="0.0"/>
-</inertial>
-```
-  </link>
-  <!-- ================= WHEELS ================= -->
-<xacro:macro name="wheel" params="name y_pos"> <link name="${name}"> <visual> <geometry> <cylinder radius="${wheel_radius}" length="${wheel_width}"/> </geometry> <origin rpy="1.57 0 0"/> </visual>
-```
-  <inertial>
-    <mass value="1.0"/>
-    <origin xyz="0 0 0"/>
-    <inertia ixx="0.005" iyy="0.005" izz="0.01"
-             ixy="0.0" ixz="0.0" iyz="0.0"/>
-  </inertial>
-</link>
-<joint name="${name}_joint" type="continuous">
-  <parent link="base_link"/>
-  <child link="${name}"/>
-  <origin xyz="0 ${y_pos} -${wheel_radius}"/>
-  <axis xyz="0 1 0"/>
-</joint>
-```
-</xacro:macro>
-<xacro:wheel name="left_wheel"  y_pos="${wheel_sep/2}"/>
-<xacro:wheel name="right_wheel" y_pos="-${wheel_sep/2}"/>
-  <!-- ================= CASTER ================= -->
-  <link name="caster">
-    <visual>
-      <geometry>
-        <sphere radius="0.05"/>
-      </geometry>
-    </visual>
-  </link>
-  <joint name="caster_joint" type="fixed">
-    <parent link="base_link"/>
-    <child link="caster"/>
-    <origin xyz="-0.1 0 -0.05"/>
-  </joint>
-  <!-- ================= SHOULDER ================= -->
-  <link name="shoulder_link">
-    <visual>
-      <geometry>
-        <cylinder radius="0.05" length="0.2"/>
-      </geometry>
-    </visual>
-```
-<inertial>
-  <mass value="0.5"/>
-  <origin xyz="0 0 0"/>
-  <inertia ixx="0.0005" iyy="0.0005" izz="0.0005"
-           ixy="0.0" ixz="0.0" iyz="0.0"/>
-</inertial>
-```
-  </link>
-  <joint name="shoulder_joint" type="continuous">
-    <parent link="base_link"/>
-    <child link="shoulder_link"/>
-    <origin xyz="0 0 0.075"/>
-    <axis xyz="0 0 1"/>
-  </joint>
-  <!-- ================= ARM LINK 1 ================= -->
-  <link name="link1">
-    <visual>
-      <geometry>
-        <cylinder radius="${arm_radius}" length="${arm_length}"/>
-      </geometry>
-      <origin xyz="${arm_length/2} 0 0" rpy="0 1.57 0"/>
-      <material name="Blue">
-        <color rgba="0 0 1 1"/>
-      </material>
-    </visual>
-```
-<inertial>
-  <mass value="2.0"/>
-  <origin xyz="${arm_length/2} 0 0"/>
-  <inertia ixx="0.01" iyy="0.01" izz="0.005"
-           ixy="0.0" ixz="0.0" iyz="0.0"/>
-</inertial>
-```
-  </link>
-  <joint name="joint1" type="revolute">
-    <parent link="shoulder_link"/>
-    <child link="link1"/>
-    <origin xyz="0 0 0.1"/>
-    <axis xyz="0 1 0"/>
-    <limit lower="-3.71" upper="0.5" effort="10" velocity="1.0"/>
-  </joint>
-  <!-- ================= ARM LINK 2 ================= -->
-  <link name="link2">
-    <visual>
-      <geometry>
-        <cylinder radius="${arm_radius}" length="${arm_length}"/>
-      </geometry>
-      <origin xyz="${arm_length/2} 0 0" rpy="0 1.57 0"/>
-    </visual>
-```
-<inertial>
-  <mass value="1.5"/>
-  <origin xyz="${arm_length/2} 0 0"/>
-  <inertia ixx="0.0075" iyy="0.0075" izz="0.00375"
-           ixy="0.0" ixz="0.0" iyz="0.0"/>
-</inertial>
-```
-  </link>
-  <joint name="joint2" type="revolute">
-    <parent link="link1"/>
-    <child link="link2"/>
-    <origin xyz="${arm_length} 0 0"/>
-    <axis xyz="0 1 0"/>
-    <limit lower="-1.57" upper="1.57" effort="10" velocity="1.0"/>
-  </joint>
-  <!-- ================= SENSORS ================= -->
-  <!-- LiDAR -->
-  <link name="lidar_link">
-    <visual>
-    <geometry>
-        <cylinder radius="0.05" length="0.01"/>
-    </geometry>
-    <origin xyz="0 0 0" rpy="0 0 0"/>
-    <material name="Green">
-        <color rgba="0 1 0 1"/>
-    </material>
-    </visual>
-  </link>
-  <joint name="lidar_joint" type="fixed">
-    <parent link="base_link"/>
-    <child link="lidar_link"/>
-    <origin xyz="0.1 0 0.075"/>
-  </joint>
-  <!-- IMU -->
-  <link name="imu_link"/>
-  <joint name="imu_joint" type="fixed">
-    <parent link="base_link"/>
-    <child link="imu_link"/>
-    <origin xyz="0 0 0.1"/>
-  </joint>
-  <!-- ================= ROS2 CONTROL ================= -->
-<ros2_control name="orion_system" type="system"> <hardware> <plugin>gazebo_ros2_control/GazeboSystem</plugin> </hardware>
-```
-<joint name="left_wheel_joint">
-  <command_interface name="velocity"/>
-  <state_interface name="velocity"/>
-  <state_interface name="position"/>
-</joint>
-<joint name="right_wheel_joint">
-  <command_interface name="velocity"/>
-  <state_interface name="velocity"/>
-  <state_interface name="position"/>
-</joint>
-<joint name="shoulder_joint">
-  <command_interface name="position"/>
-  <state_interface name="position"/>
-</joint>
-<joint name="joint1">
-  <command_interface name="position"/>
-  <state_interface name="position"/>
-</joint>
-<joint name="joint2">
-  <command_interface name="position"/>
-  <state_interface name="position"/>
-</joint>
-```
-</ros2_control>
+  <!-- Materials defined ONCE here — do NOT include in sub-files -->
+  <xacro:include filename="$(find orion_description)/xacro/materials.xacro"/>
+  <xacro:include filename="$(find orion_description)/xacro/base.xacro"/>
+  <xacro:include filename="$(find orion_description)/xacro/wheels.xacro"/>
+  <xacro:include filename="$(find orion_description)/xacro/sensors.xacro"/>
+  <xacro:include filename="$(find orion_description)/xacro/arm.xacro"/>
+  <xacro:base/>
+  <xacro:wheels/>
+  <xacro:sensors/>
+  <xacro:arm/>
 </robot>
