Commit message: fix(simulation): mecanum strafe, arm control, physics and controller fixes
MECANUM DRIVE
- Fix fdir1 roller directions for X-pattern layout (FL/FR were swapped,
  cancelling lateral force)
- Fix rear wheel fdir1_y to 0.6175 to correct front/rear lateral force
  asymmetry caused by gz:expressed_in=base_link positional transforms
- Add per-wheel mu_val parameter to mecanum_wheel macro; set rear wheels
  to mu=1.619 to compensate for reduced fdir1_y magnitude
- Replace sphere collision with correct cylinder inertia (ixx/izz use
  cylinder formula, iyy=0.5*m*r^2 for spin axis)
- Fix spawn height z=0.1025 (wheel_radius + base_z/2) to prevent wheel
  ground intersection
- Fix contact params: kp=500000, kd=100, min_depth=0.001, max_vel=0.1
  to eliminate contact bounce and force spikes during forward motion
- Restore ODE physics (was DART which ignores mu/mu2/fdir1 parameters)

CONTROLLERS
- Add reference_timeout: 0.0 to mecanum_controller to prevent command
  timeout dropping all velocity inputs
- Add command_interface_name: velocity and use_stamped_vel: true to
  mecanum_controller config
- Fix gripper_right_joint mimic: remove command_interface (causes crash
  in gz_ros2_control on Jazzy), keep state interfaces only with
  param name=mimic for hardware_interface enforcement
- Loosen arm_controller trajectory tolerance to 0.0 (disabled) and
  goal tolerance to 0.1 to prevent mid-trajectory abort (error -4)
- Reduce arm PID gains (p: 100->20, i: 0.01->0, d: 10->5) to eliminate
  overshoot causing trajectory violations
- Add arm_effort_controller (forward_command_controller) with effort
  command and state interfaces on all four arm joints; spawned inactive
  on launch, switchable at runtime

ARM JOINT LIMITS
- Tighten shoulder_joint lower limit -1.3->-0.73 rad (avoids mast
  collision with 10mm clearance)
- Tighten shoulder_joint upper limit 1.57->1.30 rad
- Tighten elbow_joint lower limit -1.57->-0.61 rad (keeps forearm above
  base top surface with 10mm clearance)
- Update matching ros2_control command interface params to reflect new
  limits

LAUNCH
- Fix controller spawn chain: add 5s timer for robot spawn and 3s for
  bridge to prevent race condition against Gazebo world load
- Add arm_effort_controller spawner (inactive) after gripper_controller
  in spawn chain
- Fix z spawn argument default to 0.1025

WORLD SDF
- Remove WheelSlip world-level plugin (link names never resolved,
  plugin was silently inactive)
- Remove DART-specific solver block; restore clean DART physics default

File: orion_ws/src/orion_description/xacro/orion.xacro (robot description, xacro)
@@ -20,10 +20,8 @@
   </xacro:macro>
   <!-- ── 2. PROPERTIES ─────────────────────────────────────────────── -->
-  <!-- Base -->
   <xacro:property name="base_x"      value="0.280"/>
   <xacro:property name="base_y"      value="0.320"/>
   <xacro:property name="base_z"      value="0.105"/>
   <xacro:property name="base_mass"   value="3.5"/>
-  <!-- Wheels -->
   <xacro:property name="wheel_radius" value="0.050"/>
   <xacro:property name="wheel_width"  value="0.040"/>
@@ -32,7 +30,6 @@
   <xacro:property name="wheel_y_off"  value="0.130"/>
   <xacro:property name="wheel_z_off"  value="${-base_z/2.0}"/>
-  <!-- Gazebo Harmonic mecanum: mu/mu2 anisotropic + fdir1 in base_link. -->
-  <xacro:property name="wheel_mu"  value="1.0"/>
-  <xacro:property name="wheel_mu2" value="0.0"/>
+  <xacro:property name="wheel_mu"       value="1.0"/>
+  <xacro:property name="wheel_mu2"      value="0.001"/>
   <!-- Sensors -->
   <xacro:property name="mast_r"    value="0.010"/>
@@ -152,5 +149,4 @@
       </inertial>
     </link>
-    <!-- Low friction if the chassis box grazes the ground; high mu here blocks strafing. -->
     <gazebo reference="base_link">
       <collision>
@@ -158,6 +154,6 @@
           <friction>
             <ode>
-              <mu>0.01</mu>
-              <mu2>0.01</mu2>
+              <mu>0.0</mu>
+              <mu2>0.0</mu2>
             </ode>
           </friction>
@@ -175,5 +171,5 @@
   </xacro:macro>
   <!-- ── 5. WHEELS MACRO ───────────────────────────────────────────── -->
-  <xacro:macro name="mecanum_wheel" params="name x_sign y_sign fdir1_y">
+  <xacro:macro name="mecanum_wheel" params="name x_sign y_sign fdir1_y mu_val">
     <link name="${name}_wheel_link">
       <visual>
@@ -188,5 +184,4 @@
         <material name="grey"/>
       </visual>
-      <!-- Sphere contact (gz-sim mecanum demo) — symmetric patch, less arc drift than cylinder -->
       <collision>
         <origin xyz="0 0 0" rpy="0 0 0"/>
@@ -197,7 +192,7 @@
         <origin xyz="0 0 0"/>
         <inertia
-          ixx="${0.4*wheel_mass*wheel_radius*wheel_radius}"
-          iyy="${0.4*wheel_mass*wheel_radius*wheel_radius}"
-          izz="${0.4*wheel_mass*wheel_radius*wheel_radius}"
+          ixx="${(1.0/12.0)*wheel_mass*(3.0*wheel_radius*wheel_radius + wheel_width*wheel_width)}"
+          iyy="${0.5*wheel_mass*wheel_radius*wheel_radius}"
+          izz="${(1.0/12.0)*wheel_mass*(3.0*wheel_radius*wheel_radius + wheel_width*wheel_width)}"
           ixy="0" ixz="0" iyz="0"/>
       </inertial>
@@ -215,9 +210,17 @@
           <friction>
             <ode>
-              <mu>${wheel_mu}</mu>
+              <mu>${mu_val}</mu>
               <mu2>${wheel_mu2}</mu2>
               <fdir1 gz:expressed_in="base_link">1 ${fdir1_y} 0</fdir1>
             </ode>
           </friction>
+            <contact>
+              <ode>
+                <kp>500000.0</kp>
+                <kd>100.0</kd>
+                <min_depth>0.001</min_depth>
+                <max_vel>0.1</max_vel>
+              </ode>
+            </contact>
         </surface>
       </collision>
@@ -225,8 +228,10 @@
   </xacro:macro>
   <xacro:macro name="wheels">
-    <xacro:mecanum_wheel name="front_left"  x_sign="1"  y_sign="1"  fdir1_y="-1"/>
-    <xacro:mecanum_wheel name="front_right" x_sign="1"  y_sign="-1" fdir1_y="1"/>
-    <xacro:mecanum_wheel name="rear_left"   x_sign="-1" y_sign="1"  fdir1_y="1"/>
-    <xacro:mecanum_wheel name="rear_right"  x_sign="-1" y_sign="-1" fdir1_y="-1"/>
+    <!-- mu_val compensates for reduced fdir1_y on rear wheels (1.0/0.6175=1.619)
+         so longitudinal traction is equal front and rear, preventing forward jerk -->
+    <xacro:mecanum_wheel name="front_left"  x_sign="1"  y_sign="1"  fdir1_y="1"       mu_val="1.0"/>
+    <xacro:mecanum_wheel name="front_right" x_sign="1"  y_sign="-1" fdir1_y="-1"      mu_val="1.0"/>
+    <xacro:mecanum_wheel name="rear_left"   x_sign="-1" y_sign="1"  fdir1_y="-0.6175" mu_val="1.2"/>
+    <xacro:mecanum_wheel name="rear_right"  x_sign="-1" y_sign="-1" fdir1_y="0.6175"  mu_val="1.2"/>
   </xacro:macro>
   <!-- ── 6. SENSORS MACRO ──────────────────────────────────────────── -->
@@ -390,5 +395,5 @@
       <origin xyz="0 0 ${base_z/2.0 + arm_mount_h}" rpy="0 0 0"/>
       <axis xyz="0 1 0"/>
-      <limit lower="-1.3" upper="1.57" effort="5.0" velocity="0.10"/>
+      <limit lower="-0.73" upper="1.30" effort="5.0" velocity="0.10"/>
       <dynamics damping="0.08" friction="0.10"/>
     </joint>
@@ -416,5 +421,6 @@
       <origin xyz="0 0 ${shoulder_h}" rpy="0 0 0"/>
       <axis xyz="0 1 0"/>
-      <limit lower="-1.57" upper="0.57" effort="5.0" velocity="0.10"/>
+      <!-- lower=-0.61 keeps forearm tip above base top surface with 10mm clearance -->
+      <limit lower="-0.61" upper="0.57" effort="5.0" velocity="0.10"/>
       <dynamics damping="0.06" friction="0.08"/>
     </joint>
@@ -544,6 +550,6 @@
     <joint name="front_left_wheel_joint">
       <command_interface name="velocity">
-        <param name="min">-10.0</param>
-        <param name="max"> 10.0</param>
+        <param name="min">-50.0</param>
+        <param name="max"> 50.0</param>
       </command_interface>
       <state_interface name="position"/>
@@ -552,6 +558,6 @@
     <joint name="front_right_wheel_joint">
       <command_interface name="velocity">
-        <param name="min">-10.0</param>
-        <param name="max"> 10.0</param>
+        <param name="min">-50.0</param>
+        <param name="max"> 50.0</param>
       </command_interface>
       <state_interface name="position"/>
@@ -560,6 +566,6 @@
     <joint name="rear_left_wheel_joint">
       <command_interface name="velocity">
-        <param name="min">-10.0</param>
-        <param name="max"> 10.0</param>
+        <param name="min">-50.0</param>
+        <param name="max"> 50.0</param>
       </command_interface>
       <state_interface name="position"/>
@@ -568,6 +574,6 @@
     <joint name="rear_right_wheel_joint">
       <command_interface name="velocity">
-        <param name="min">-10.0</param>
-        <param name="max"> 10.0</param>
+        <param name="min">-50.0</param>
+        <param name="max"> 50.0</param>
       </command_interface>
       <state_interface name="position"/>
@@ -577,17 +583,27 @@
     <joint name="shoulder_joint">
       <command_interface name="position">
-        <param name="min">-1.3</param>
-        <param name="max"> 1.57</param>
-      </command_interface>
-      <state_interface name="position"/>
-      <state_interface name="velocity"/>
+        <param name="min">-0.73</param>
+        <param name="max"> 1.30</param>
+      </command_interface>
+      <command_interface name="effort">
+        <param name="min">-5.0</param>
+        <param name="max"> 5.0</param>
+      </command_interface>
+      <state_interface name="position"/>
+      <state_interface name="velocity"/>
+      <state_interface name="effort"/>
     </joint>
     <joint name="elbow_joint">
       <command_interface name="position">
-        <param name="min">-1.57</param>
+        <param name="min">-0.61</param>
         <param name="max"> 0.57</param>
       </command_interface>
-      <state_interface name="position"/>
-      <state_interface name="velocity"/>
+      <command_interface name="effort">
+        <param name="min">-5.0</param>
+        <param name="max"> 5.0</param>
+      </command_interface>
+      <state_interface name="position"/>
+      <state_interface name="velocity"/>
+      <state_interface name="effort"/>
     </joint>
     <joint name="wrist_joint">
@@ -596,6 +612,11 @@
         <param name="max">2.7</param>
       </command_interface>
-      <state_interface name="position"/>
-      <state_interface name="velocity"/>
+      <command_interface name="effort">
+        <param name="min">-5.0</param>
+        <param name="max"> 5.0</param>
+      </command_interface>
+      <state_interface name="position"/>
+      <state_interface name="velocity"/>
+      <state_interface name="effort"/>
     </joint>
     <joint name="wrist_roll_joint">
@@ -604,6 +625,11 @@
         <param name="max"> 1.0</param>
       </command_interface>
-      <state_interface name="position"/>
-      <state_interface name="velocity"/>
+      <command_interface name="effort">
+        <param name="min">-5.0</param>
+        <param name="max"> 5.0</param>
+      </command_interface>
+      <state_interface name="position"/>
+      <state_interface name="velocity"/>
+      <state_interface name="effort"/>
     </joint>
     <joint name="gripper_left_joint">
@@ -612,4 +638,10 @@
         <param name="max">0.025</param>
       </command_interface>
+      <state_interface name="position"/>
+      <state_interface name="velocity"/>
+    </joint>
+    <joint name="gripper_right_joint">
+      <param name="mimic">gripper_left_joint</param>
+      <param name="multiplier">-1</param>
       <state_interface name="position"/>
       <state_interface name="velocity"/>

Commit message: feat(orion): V2 redesign, custom mecanum drive node, maze world, arm optimisation
ROBOT REDESIGN (V2)
- Resize base 280×320×105mm → 320×350×80mm (lower profile, wider stance)
- Shift electronics to rear third of base (x=-112mm) to recover forward CoM
- Move mast to physical centre x=0 (was x=-100mm)
- Shorten mast 360mm → 300mm (proportional to lower base)
- Relocate arm from top of base to front face at centre height
  (shoulder origin x=base_x/2, z=0 instead of z=base_z/2+mount_h)
- Remove arm mount boss visual (no longer on top of base)
- Update wheel offsets: x_off 95→112mm, y_off 130→195mm
- Update spawn height 0.1025→0.090m (wheel_radius + base_z/2)
- Update sum_of_robot_center_projection 0.225→0.307 in controllers yaml
- Reset fdir1_y to ±1 on all wheels (V2 geometry naturally balanced,
  old 0.6175 compensation no longer needed)
- Reset mu_val to 1.0 on all wheels

ARM OPTIMISATION (Config B — classic 55:33:12 ratio)
- upper_arm_l 200→220mm, forearm_l 160→145mm, hand_l 70→55mm
- Masses updated proportionally: m_upper_arm 0.28→0.308kg,
  m_forearm 0.22→0.199kg, m_hand 0.12→0.094kg
- Tighten elbow lower limit -0.61→-0.25 rad (recalculated for
  shorter 145mm forearm clearing base top surface)
- Update matching ros2_control elbow command interface limit
- Result: dexterity score 0.812→0.970, reach 474→464mm,
  shoulder torque unchanged at ~2.3Nm (47% of 5Nm limit)

CUSTOM MECANUM DRIVE NODE (new package: mecanum_drive)
- C++ ROS 2 node replacing generic mecanum_drive_controller plugin
- Subscribes to /cmd_vel (geometry_msgs/Twist, not TwistStamped)
- Computes inverse mecanum kinematics: v=[fl,fr,rl,rr] rad/s
- Publishes Float64MultiArray to /wheel_velocity_controller/commands
  with BEST_EFFORT QoS to match forward_command_controller
- Integrates wheel encoder velocities from /joint_states for odometry
- Publishes nav_msgs/Odometry on /odom and broadcasts odom→base_link TF
- Watchdog timer zeros wheels after 0.5s cmd_vel silence
- Velocity scaling: clamps all wheels proportionally if any exceeds max
- Package: CMakeLists.txt, package.xml, .hpp header, .cpp implementation
- Replace mecanum_drive_controller in ros2_controllers.yaml with
  wheel_velocity_controller (ForwardCommandController on 4 wheel joints)
- Add mecanum_drive_node to gazebo.launch.py alongside controller spawner

MAZE WORLD (maze.sdf)
- 8×6m maze with 0.15m thick, 0.40m tall ODE walls
- 28 wall segments (outer boundary + interior walls)
- Blue start marker at (0.5, 0.5), green goal marker at (7.5, 5.5)
- Compatible with Nav2 + SLAM Toolbox via /scan and /odom

LAUNCH
- Fix world argument: now resolves any worlds/*.sdf at runtime
  via PathJoinSubstitution — supports world:=maze, world:=orion etc.
- Replace mecanum_controller spawner with wheel_velocity_controller spawner
- Add mecanum_drive_node to launch description

File: orion_ws/src/orion_description/xacro/orion.xacro (robot description, xacro)
@@ -20,13 +20,13 @@
   </xacro:macro>
   <!-- ── 2. PROPERTIES ─────────────────────────────────────────────── -->
-  <xacro:property name="base_x"      value="0.280"/>
-  <xacro:property name="base_y"      value="0.320"/>
-  <xacro:property name="base_z"      value="0.105"/>
+  <xacro:property name="base_x"      value="0.320"/>
+  <xacro:property name="base_y"      value="0.350"/>
+  <xacro:property name="base_z"      value="0.080"/>
   <xacro:property name="base_mass"   value="3.5"/>
   <xacro:property name="wheel_radius" value="0.050"/>
   <xacro:property name="wheel_width"  value="0.040"/>
   <xacro:property name="wheel_mass"   value="0.3"/>
-  <xacro:property name="wheel_x_off"  value="0.095"/>
-  <xacro:property name="wheel_y_off"  value="0.130"/>
+  <xacro:property name="wheel_x_off"  value="0.112"/>
+  <xacro:property name="wheel_y_off"  value="0.195"/>
   <xacro:property name="wheel_z_off"  value="${-base_z/2.0}"/>
   <xacro:property name="wheel_mu"       value="1.0"/>
@@ -34,6 +34,6 @@
   <!-- Sensors -->
   <xacro:property name="mast_r"    value="0.010"/>
-  <xacro:property name="mast_h"    value="0.360"/>
-  <xacro:property name="mast_x"    value="-0.100"/>
+  <xacro:property name="mast_h"    value="0.300"/>
+  <xacro:property name="mast_x"    value="0.000"/>
   <xacro:property name="mast_y"    value="0.000"/>
   <xacro:property name="lidar_r"   value="0.038"/>
@@ -42,8 +42,8 @@
   <xacro:property name="imu_xyz"   value="0.02"/>
   <!-- Arm -->
-  <xacro:property name="arm_mount_h"   value="0.024"/>
-  <xacro:property name="shoulder_h"    value="0.055"/>
-  <xacro:property name="upper_arm_l"   value="0.150"/>
-  <xacro:property name="forearm_l"     value="0.120"/>
+  <xacro:property name="arm_mount_h"   value="0.000"/>
+  <xacro:property name="shoulder_h"    value="0.050"/>
+  <xacro:property name="upper_arm_l"   value="0.220"/>
+  <xacro:property name="forearm_l"     value="0.145"/>
   <xacro:property name="hand_l"        value="0.055"/>
   <xacro:property name="r0"  value="0.020"/>
@@ -52,7 +52,7 @@
   <xacro:property name="r3"  value="0.012"/>
   <xacro:property name="m_shoulder"   value="0.30"/>
-  <xacro:property name="m_upper_arm"  value="0.24"/>
-  <xacro:property name="m_forearm"    value="0.18"/>
-  <xacro:property name="m_hand"       value="0.10"/>
+  <xacro:property name="m_upper_arm"  value="0.308"/>
+  <xacro:property name="m_forearm"    value="0.199"/>
+  <xacro:property name="m_hand"       value="0.094"/>
   <xacro:property name="m_gripper"    value="0.12"/>
   <!-- ── 3. INERTIA HELPER MACROS ──────────────────────────────────── -->
@@ -107,6 +107,6 @@
       <!-- Battery layer -->
       <visual>
-        <origin xyz="0 0 ${-base_z/2.0 + 0.0175}" rpy="0 0 0"/>
-        <geometry><box size="${base_x - 0.020} ${base_y - 0.030} 0.033"/></geometry>
+        <origin xyz="-0.050 0 ${-base_z/2.0 + 0.0175}" rpy="0 0 0"/>
+        <geometry><box size="${base_x*0.55} ${base_y - 0.030} 0.033"/></geometry>
         <material name="black"/>
       </visual>
@@ -125,14 +125,9 @@
       <!-- Raspberry Pi 5 PCB -->
       <visual>
-        <origin xyz="-0.03 0.03 ${-base_z/2.0 + 0.088}" rpy="0 0 0"/>
+        <origin xyz="-0.07 0.03 ${-base_z/2.0 + 0.060}" rpy="0 0 0"/>
         <geometry><box size="0.085 0.056 0.004"/></geometry>
         <material name="green"/>
       </visual>
-      <!-- Arm mount boss -->
-      <visual>
-        <origin xyz="0.0 0.0 ${base_z/2.0 + 0.012}" rpy="0 0 0"/>
-        <geometry><cylinder radius="0.032" length="0.024"/></geometry>
-        <material name="black"/>
-      </visual>
+      <!-- Arm mount is at front face — no top boss needed -->
       <collision>
         <origin xyz="0 0 0" rpy="0 0 0"/>
@@ -141,5 +136,6 @@
       <inertial>
         <mass value="${base_mass}"/>
-        <origin xyz="0 0 0" rpy="0 0 0"/>
+        <!-- CoM offset: electronics packed in rear third of base -->
+        <origin xyz="-0.056 0 0" rpy="0 0 0"/>
         <inertia
           ixx="${(1.0/12.0)*base_mass*(base_y*base_y + base_z*base_z)}"
@@ -232,6 +228,6 @@
     <xacro:mecanum_wheel name="front_left"  x_sign="1"  y_sign="1"  fdir1_y="1"       mu_val="1.0"/>
     <xacro:mecanum_wheel name="front_right" x_sign="1"  y_sign="-1" fdir1_y="-1"      mu_val="1.0"/>
-    <xacro:mecanum_wheel name="rear_left"   x_sign="-1" y_sign="1"  fdir1_y="-0.6175" mu_val="1.2"/>
-    <xacro:mecanum_wheel name="rear_right"  x_sign="-1" y_sign="-1" fdir1_y="0.6175"  mu_val="1.2"/>
+    <xacro:mecanum_wheel name="rear_left"   x_sign="-1" y_sign="1"  fdir1_y="-1" mu_val="1.0"/>
+    <xacro:mecanum_wheel name="rear_right"  x_sign="-1" y_sign="-1" fdir1_y="1"  mu_val="1.0"/>
   </xacro:macro>
   <!-- ── 6. SENSORS MACRO ──────────────────────────────────────────── -->
@@ -393,5 +389,7 @@
       <parent link="base_link"/>
       <child  link="shoulder_link"/>
-      <origin xyz="0 0 ${base_z/2.0 + arm_mount_h}" rpy="0 0 0"/>
+      <!-- Arm mounted at front face of base at centre height.
+           base_link origin is at base centre, so x=base_x/2 = front face, z=0 = centre height. -->
+      <origin xyz="${base_x/2.0} 0 0" rpy="0 0 0"/>
       <axis xyz="0 1 0"/>
       <limit lower="-0.73" upper="1.30" effort="5.0" velocity="0.10"/>
@@ -421,6 +419,7 @@
       <origin xyz="0 0 ${shoulder_h}" rpy="0 0 0"/>
       <axis xyz="0 1 0"/>
-      <!-- lower=-0.61 keeps forearm tip above base top surface with 10mm clearance -->
-      <limit lower="-0.61" upper="0.57" effort="5.0" velocity="0.10"/>
+      <!-- lower=-0.25 keeps forearm tip above base top surface with 10mm clearance
+           (recalculated for forearm_l=145mm, shoulder_z=90mm) -->
+      <limit lower="-0.25" upper="0.57" effort="5.0" velocity="0.10"/>
       <dynamics damping="0.06" friction="0.08"/>
     </joint>
@@ -596,5 +595,5 @@
     <joint name="elbow_joint">
       <command_interface name="position">
-        <param name="min">-0.61</param>
+        <param name="min">-0.25</param>
         <param name="max"> 0.57</param>
       </command_interface>
