Commit message: Updated gripper design + added mass and length values to robot model in arm kinematics logic package

File: orion_ws/src/orion_description/xacro/orion.xacro (robot description, xacro)
@@ -4,5 +4,106 @@
        xmlns:gz="http://gazebosim.org/schema">
   <xacro:arg name="controllers_file" default="config/ros2_controllers.yaml"/>
-  <!-- ── 1. MATERIALS ─────────────────────────────────────────────── -->
+  <!-- ════════════════════════════════════════════════════════════════════
+       1.  ALL CONSTANTS
+       ════════════════════════════════════════════════════════════════════ -->
+  <!-- ── Base ─────────────────────────────────────────────────────────── -->
+  <xacro:property name="base_x"    value="0.320"/>  <!-- length  [m] -->
+  <xacro:property name="base_y"    value="0.350"/>  <!-- width   [m] -->
+  <xacro:property name="base_z"    value="0.080"/>  <!-- height  [m] -->
+  <xacro:property name="base_mass" value="3.5"/>    <!-- kg -->
+  <!-- ── Wheels ───────────────────────────────────────────────────────── -->
+  <xacro:property name="wheel_radius" value="0.050"/>              <!-- m -->
+  <xacro:property name="wheel_width"  value="0.040"/>              <!-- m -->
+  <xacro:property name="wheel_mass"   value="0.3"/>                <!-- kg -->
+  <xacro:property name="wheel_x_off"  value="0.112"/>              <!-- m from base centre -->
+  <xacro:property name="wheel_y_off"  value="0.195"/>              <!-- m from base centre -->
+  <xacro:property name="wheel_z_off"  value="${-base_z/2.0}"/>     <!-- m (wheel axle at base bottom) -->
+  <xacro:property name="wheel_mu"     value="1.0"/>                <!-- longitudinal friction -->
+  <xacro:property name="wheel_mu2"    value="0.001"/>              <!-- lateral friction -->
+  <!-- ── Sensors ──────────────────────────────────────────────────────── -->
+  <xacro:property name="mast_r"  value="0.010"/>   <!-- LiDAR mast radius  [m] -->
+  <xacro:property name="mast_h"  value="0.300"/>   <!-- LiDAR mast height  [m] -->
+  <xacro:property name="mast_x"  value="0.000"/>   <!-- mast X offset from base centre [m] -->
+  <xacro:property name="mast_y"  value="0.000"/>   <!-- mast Y offset from base centre [m] -->
+  <xacro:property name="lidar_r" value="0.038"/>   <!-- LiDAR body radius  [m] -->
+  <xacro:property name="lidar_h" value="0.041"/>   <!-- LiDAR body height  [m] -->
+  <xacro:property name="lidar_m" value="0.185"/>   <!-- LiDAR mass         [kg] -->
+  <xacro:property name="imu_xyz" value="0.02"/>    <!-- IMU cube side      [m] -->
+  <!-- ── Arm geometry ─────────────────────────────────────────────────── -->
+  <!--
+    Chain: base_link
+             └─ shoulder_joint (revolute, Y-axis)
+                  └─ shoulder_link  (vertical stub)
+                       └─ elbow_joint (revolute, Y-axis)
+                            └─ upper_arm_link  (extends along +X)
+                                 └─ wrist_joint (revolute, Y-axis)
+                                      └─ forearm_link  (extends along +X)
+                                           └─ gripper_pitch_joint  ─┐
+                                                └─ gripper_pitch_link │ ball-and-socket
+                                                     └─ gripper_yaw_joint │ (3 × revolute,
+                                                          └─ gripper_yaw_link │  zero-length
+                                                               └─ gripper_roll_joint ┘  links)
+                                                                    └─ gripper_base_link
+                                                                         ├─ gripper_left_joint
+                                                                         └─ gripper_right_joint
+    All arm revolute axes are +Y (rotation in the sagittal / x-z plane).
+    Ball-and-socket is decomposed into pitch (+Y), yaw (+Z), roll (+X) at the
+    same physical point — this is the standard URDF approximation of a spherical
+    joint, which has no native URDF type.
+  -->
+  <!-- Arm mount: shoulder joint sits at base front face, vertically centred -->
+  <xacro:property name="shoulder_mount_x" value="${base_x/2.0}"/>  <!-- = 0.160 m -->
+  <xacro:property name="shoulder_mount_z" value="0.0"/>            <!-- base_link origin is mid-height -->
+  <!-- Link lengths [m] -->
+  <xacro:property name="shoulder_h"   value="0.050"/>  <!-- shoulder stub (vertical, +Z) -->
+  <xacro:property name="upper_arm_l"  value="0.220"/>  <!-- upper arm (along +X after elbow) -->
+  <xacro:property name="forearm_l"    value="0.145"/>  <!-- forearm (along +X after wrist) -->
+  <xacro:property name="gripper_l"    value="0.055"/>  <!-- gripper body depth along +X -->
+  <xacro:property name="gripper_tcp"  value="0.050"/>  <!-- gripper base → TCP tip along +X -->
+  <!-- Link cross-section radii [m] (cylinder approximations) -->
+  <xacro:property name="r_shoulder"  value="0.020"/>
+  <xacro:property name="r_upper_arm" value="0.018"/>
+  <xacro:property name="r_forearm"   value="0.015"/>
+  <xacro:property name="r_gripper"   value="0.012"/>
+  <!-- Link masses [kg] -->
+  <xacro:property name="m_shoulder"  value="0.300"/>
+  <xacro:property name="m_upper_arm" value="0.308"/>
+  <xacro:property name="m_forearm"   value="0.199"/>
+  <xacro:property name="m_gripper"   value="0.120"/>  <!-- gripper body (fingers split below) -->
+  <!-- Joint limits [rad] — arm revolutes -->
+  <xacro:property name="shoulder_lo"  value="-0.73"/>  <!-- −41.8 ° -->
+  <xacro:property name="shoulder_hi"  value=" 1.30"/>  <!--  74.5 ° -->
+  <xacro:property name="elbow_lo"     value="-0.25"/>  <!-- −14.3 ° -->
+  <xacro:property name="elbow_hi"     value=" 0.57"/>  <!--  32.7 ° -->
+  <xacro:property name="wrist_lo"     value=" 0.00"/>  <!--   0.0 ° -->
+  <xacro:property name="wrist_hi"     value=" 2.70"/>  <!-- 154.7 ° -->
+  <!-- Joint limits [rad] — ball-and-socket (gripper) -->
+  <xacro:property name="gp_lo"  value="-1.57"/>  <!-- pitch ±90 ° -->
+  <xacro:property name="gp_hi"  value=" 1.57"/>
+  <xacro:property name="gy_lo"  value="-1.57"/>  <!-- yaw   ±90 ° -->
+  <xacro:property name="gy_hi"  value=" 1.57"/>
+  <xacro:property name="gr_lo"  value="-1.57"/>  <!-- roll  ±90 ° -->
+  <xacro:property name="gr_hi"  value=" 1.57"/>
+  <!-- Joint dynamics -->
+  <xacro:property name="shoulder_damp"  value="0.08"/>  <xacro:property name="shoulder_fric" value="0.10"/>
+  <xacro:property name="elbow_damp"     value="0.06"/>  <xacro:property name="elbow_fric"    value="0.08"/>
+  <xacro:property name="wrist_damp"     value="0.04"/>  <xacro:property name="wrist_fric"    value="0.06"/>
+  <xacro:property name="gripper_damp"   value="0.02"/>  <xacro:property name="gripper_fric"  value="0.03"/>
+  <!-- Actuator limits -->
+  <xacro:property name="arm_effort"    value="5.0"/>   <!-- Nm, all arm joints -->
+  <xacro:property name="arm_vel"       value="1.0"/>   <!-- rad/s (raised from 0.10 for sim) -->
+  <xacro:property name="gripper_effort" value="5.0"/>  <!-- N -->
+  <xacro:property name="gripper_vel"    value="0.10"/> <!-- m/s -->
+  <xacro:property name="gripper_stroke" value="0.025"/><!-- m, each finger from centre -->
+  <!-- Gripper finger geometry (L-shaped: rail + jaw) -->
+  <xacro:property name="finger_w"         value="0.012"/>  <!-- rail width (thin slab along base side) [m] -->
+  <xacro:property name="finger_h"         value="0.018"/>  <!-- finger height — matches gripper_base [m] -->
+  <xacro:property name="finger_jaw_l"     value="0.055"/>  <!-- jaw forward protrusion past base [m] -->
+  <xacro:property name="finger_jaw_w"     value="0.020"/>  <!-- jaw width (inward-facing pad) [m] -->
+  <xacro:property name="finger_bracket_l" value="0.018"/>  <!-- rear bracket depth behind base [m] -->
+  <xacro:property name="finger_bracket_w" value="0.028"/>  <!-- rear bracket inward span [m] -->
+  <!-- ════════════════════════════════════════════════════════════════════
+       2.  MATERIALS
+       ════════════════════════════════════════════════════════════════════ -->
   <material name="grey">      <color rgba="0.60 0.60 0.60 1.0"/></material>
   <material name="dark_grey"> <color rgba="0.25 0.25 0.25 1.0"/></material>
@@ -19,42 +120,8 @@
     </gazebo>
   </xacro:macro>
-  <!-- ── 2. PROPERTIES ─────────────────────────────────────────────── -->
-  <xacro:property name="base_x"      value="0.320"/>
-  <xacro:property name="base_y"      value="0.350"/>
-  <xacro:property name="base_z"      value="0.080"/>
-  <xacro:property name="base_mass"   value="3.5"/>
-  <xacro:property name="wheel_radius" value="0.050"/>
-  <xacro:property name="wheel_width"  value="0.040"/>
-  <xacro:property name="wheel_mass"   value="0.3"/>
-  <xacro:property name="wheel_x_off"  value="0.112"/>
-  <xacro:property name="wheel_y_off"  value="0.195"/>
-  <xacro:property name="wheel_z_off"  value="${-base_z/2.0}"/>
-  <xacro:property name="wheel_mu"       value="1.0"/>
-  <xacro:property name="wheel_mu2"      value="0.001"/>
-  <!-- Sensors -->
-  <xacro:property name="mast_r"    value="0.010"/>
-  <xacro:property name="mast_h"    value="0.300"/>
-  <xacro:property name="mast_x"    value="0.000"/>
-  <xacro:property name="mast_y"    value="0.000"/>
-  <xacro:property name="lidar_r"   value="0.038"/>
-  <xacro:property name="lidar_h"   value="0.041"/>
-  <xacro:property name="lidar_m"   value="0.185"/>
-  <xacro:property name="imu_xyz"   value="0.02"/>
-  <!-- Arm -->
-  <xacro:property name="arm_mount_h"   value="0.000"/>
-  <xacro:property name="shoulder_h"    value="0.050"/>
-  <xacro:property name="upper_arm_l"   value="0.220"/>
-  <xacro:property name="forearm_l"     value="0.145"/>
-  <xacro:property name="hand_l"        value="0.055"/>
-  <xacro:property name="r0"  value="0.020"/>
-  <xacro:property name="r1"  value="0.018"/>
-  <xacro:property name="r2"  value="0.015"/>
-  <xacro:property name="r3"  value="0.012"/>
-  <xacro:property name="m_shoulder"   value="0.30"/>
-  <xacro:property name="m_upper_arm"  value="0.308"/>
-  <xacro:property name="m_forearm"    value="0.199"/>
-  <xacro:property name="m_hand"       value="0.094"/>
-  <xacro:property name="m_gripper"    value="0.12"/>
-  <!-- ── 3. INERTIA HELPER MACROS ──────────────────────────────────── -->
+  <!-- ════════════════════════════════════════════════════════════════════
+       3.  INERTIA HELPER MACROS
+       ════════════════════════════════════════════════════════════════════ -->
+  <!-- Cylinder with long axis along +Z, CoM at geometric centre -->
   <xacro:macro name="inertia_cyl_z" params="m r l">
     <inertial>
@@ -68,4 +135,5 @@
     </inertial>
   </xacro:macro>
+  <!-- Cylinder with long axis along +X, CoM at geometric centre -->
   <xacro:macro name="inertia_cyl_x" params="m r l">
     <inertial>
@@ -79,4 +147,5 @@
     </inertial>
   </xacro:macro>
+  <!-- Box with CoM at (ox, oy, oz) from the link origin -->
   <xacro:macro name="inertia_box" params="m x y z ox oy oz">
     <inertial>
@@ -90,5 +159,15 @@
     </inertial>
   </xacro:macro>
-  <!-- ── 4. BASE MACRO ─────────────────────────────────────────────── -->
+  <!-- Point mass (for zero-length ball-socket intermediate links) -->
+  <xacro:macro name="inertia_point" params="m">
+    <inertial>
+      <mass value="${m}"/>
+      <origin xyz="0 0 0" rpy="0 0 0"/>
+      <inertia ixx="1e-6" iyy="1e-6" izz="1e-6" ixy="0" ixz="0" iyz="0"/>
+    </inertial>
+  </xacro:macro>
+  <!-- ════════════════════════════════════════════════════════════════════
+       4.  BASE
+       ════════════════════════════════════════════════════════════════════ -->
   <xacro:macro name="base">
     <link name="base_link">
@@ -129,5 +208,4 @@
         <material name="green"/>
       </visual>
-      <!-- Arm mount is at front face — no top boss needed -->
       <collision>
         <origin xyz="0 0 0" rpy="0 0 0"/>
@@ -136,6 +214,5 @@
       <inertial>
         <mass value="${base_mass}"/>
-        <!-- CoM offset: electronics packed in rear third of base -->
-        <origin xyz="-0.056 0 0" rpy="0 0 0"/>
+        <origin xyz="-0.056 0 0" rpy="0 0 0"/>  <!-- CoM: electronics in rear third -->
         <inertia
           ixx="${(1.0/12.0)*base_mass*(base_y*base_y + base_z*base_z)}"
@@ -148,10 +225,5 @@
       <collision>
         <surface>
-          <friction>
-            <ode>
-              <mu>0.0</mu>
-              <mu2>0.0</mu2>
-            </ode>
-          </friction>
+          <friction><ode><mu>0.0</mu><mu2>0.0</mu2></ode></friction>
         </surface>
       </collision>
@@ -166,5 +238,7 @@
     </gazebo>
   </xacro:macro>
-  <!-- ── 5. WHEELS MACRO ───────────────────────────────────────────── -->
+  <!-- ════════════════════════════════════════════════════════════════════
+       5.  WHEELS (mecanum)
+       ════════════════════════════════════════════════════════════════════ -->
   <xacro:macro name="mecanum_wheel" params="name x_sign y_sign fdir1_y mu_val">
     <link name="${name}_wheel_link">
@@ -174,5 +248,4 @@
         <material name="black"/>
       </visual>
-      <!-- Hub detail -->
       <visual>
         <origin xyz="0 0 0" rpy="${pi/2} 0 0"/>
@@ -211,12 +284,12 @@
             </ode>
           </friction>
-            <contact>
-              <ode>
-                <kp>500000.0</kp>
-                <kd>100.0</kd>
-                <min_depth>0.001</min_depth>
-                <max_vel>0.1</max_vel>
-              </ode>
-            </contact>
+          <contact>
+            <ode>
+              <kp>500000.0</kp>
+              <kd>100.0</kd>
+              <min_depth>0.001</min_depth>
+              <max_vel>0.1</max_vel>
+            </ode>
+          </contact>
         </surface>
       </collision>
@@ -224,12 +297,12 @@
   </xacro:macro>
   <xacro:macro name="wheels">
-    <!-- mu_val compensates for reduced fdir1_y on rear wheels (1.0/0.6175=1.619)
-         so longitudinal traction is equal front and rear, preventing forward jerk -->
-    <xacro:mecanum_wheel name="front_left"  x_sign="1"  y_sign="1"  fdir1_y="1"       mu_val="1.0"/>
-    <xacro:mecanum_wheel name="front_right" x_sign="1"  y_sign="-1" fdir1_y="-1"      mu_val="1.0"/>
-    <xacro:mecanum_wheel name="rear_left"   x_sign="-1" y_sign="1"  fdir1_y="-1" mu_val="1.0"/>
-    <xacro:mecanum_wheel name="rear_right"  x_sign="-1" y_sign="-1" fdir1_y="1"  mu_val="1.0"/>
-  </xacro:macro>
-  <!-- ── 6. SENSORS MACRO ──────────────────────────────────────────── -->
+    <xacro:mecanum_wheel name="front_left"  x_sign=" 1" y_sign=" 1" fdir1_y=" 1" mu_val="1.0"/>
+    <xacro:mecanum_wheel name="front_right" x_sign=" 1" y_sign="-1" fdir1_y="-1" mu_val="1.0"/>
+    <xacro:mecanum_wheel name="rear_left"   x_sign="-1" y_sign=" 1" fdir1_y="-1" mu_val="1.0"/>
+    <xacro:mecanum_wheel name="rear_right"  x_sign="-1" y_sign="-1" fdir1_y=" 1" mu_val="1.0"/>
+  </xacro:macro>
+  <!-- ════════════════════════════════════════════════════════════════════
+       6.  SENSORS
+       ════════════════════════════════════════════════════════════════════ -->
   <xacro:macro name="sensors">
     <!-- LiDAR mast -->
@@ -305,5 +378,5 @@
               <resolution>1</resolution>
               <min_angle>-3.14159</min_angle>
-              <max_angle>3.14159</max_angle>
+              <max_angle> 3.14159</max_angle>
             </horizontal>
           </scan>
@@ -313,9 +386,5 @@
             <resolution>0.01</resolution>
           </range>
-          <noise>
-            <type>gaussian</type>
-            <mean>0.0</mean>
-            <stddev>0.01</stddev>
-          </noise>
+          <noise><type>gaussian</type><mean>0.0</mean><stddev>0.01</stddev></noise>
         </lidar>
         <always_on>true</always_on>
@@ -328,7 +397,5 @@
       <visual>
         <origin xyz="0 0 0"/>
-        <geometry>
-          <box size="${imu_xyz} ${imu_xyz} ${imu_xyz}"/>
-        </geometry>
+        <geometry><box size="${imu_xyz} ${imu_xyz} ${imu_xyz}"/></geometry>
         <material name="dark_grey"/>
       </visual>
@@ -336,6 +403,5 @@
         <mass value="0.05"/>
         <origin xyz="0 0 0"/>
-        <inertia ixx="0.001" iyy="0.001" izz="0.001"
-                 ixy="0" ixz="0" iyz="0"/>
+        <inertia ixx="0.001" iyy="0.001" izz="0.001" ixy="0" ixz="0" iyz="0"/>
       </inertial>
     </link>
@@ -366,285 +432,338 @@
     </gazebo>
   </xacro:macro>
-  <!-- ── 7. ARM MACRO ──────────────────────────────────────────────── -->
+  <!-- ════════════════════════════════════════════════════════════════════
+       7.  ARM
+       Chain: shoulder_link → upper_arm_link → forearm_link → gripper
+       All revolutes rotate about +Y (sagittal plane).
+       Ball-and-socket gripper: 3 × revolute at same point (pitch/yaw/roll).
+       ════════════════════════════════════════════════════════════════════ -->
   <xacro:macro name="arm">
-    <!-- Shoulder -->
+    <!-- ── Shoulder link (vertical stub, rotates about +Y at base front) ── -->
     <link name="shoulder_link">
       <visual>
         <origin xyz="0 0 ${shoulder_h/2.0}" rpy="0 0 0"/>
-        <geometry><cylinder radius="${r0}" length="${shoulder_h}"/></geometry>
-        <material name="grey"/>
-      </visual>
-      <visual>
+        <geometry><cylinder radius="${r_shoulder}" length="${shoulder_h}"/></geometry>
+        <material name="grey"/>
+      </visual>
+      <visual>  <!-- collar ring at base of stub -->
         <origin xyz="0 0 0.010" rpy="0 0 0"/>
-        <geometry><cylinder radius="${r0*1.9}" length="0.020"/></geometry>
+        <geometry><cylinder radius="${r_shoulder*1.9}" length="0.020"/></geometry>
         <material name="dark_grey"/>
       </visual>
       <collision>
         <origin xyz="0 0 ${shoulder_h/2.0}" rpy="0 0 0"/>
-        <geometry><cylinder radius="${r0}" length="${shoulder_h}"/></geometry>
-      </collision>
-      <xacro:inertia_cyl_z m="${m_shoulder}" r="${r0}" l="${shoulder_h}"/>
+        <geometry><cylinder radius="${r_shoulder}" length="${shoulder_h}"/></geometry>
+      </collision>
+      <xacro:inertia_cyl_z m="${m_shoulder}" r="${r_shoulder}" l="${shoulder_h}"/>
     </link>
     <joint name="shoulder_joint" type="revolute">
       <parent link="base_link"/>
       <child  link="shoulder_link"/>
-      <!-- Arm mounted at front face of base at centre height.
-           base_link origin is at base centre, so x=base_x/2 = front face, z=0 = centre height. -->
-      <origin xyz="${base_x/2.0} 0 0" rpy="0 0 0"/>
+      <origin xyz="${shoulder_mount_x} 0 ${shoulder_mount_z}" rpy="0 0 0"/>
       <axis xyz="0 1 0"/>
-      <limit lower="-0.73" upper="1.30" effort="5.0" velocity="0.10"/>
-      <dynamics damping="0.08" friction="0.10"/>
-    </joint>
-    <!-- Upper arm -->
+      <limit lower="${shoulder_lo}" upper="${shoulder_hi}"
+             effort="${arm_effort}" velocity="${arm_vel}"/>
+      <dynamics damping="${shoulder_damp}" friction="${shoulder_fric}"/>
+    </joint>
+    <!-- ── Upper arm link (extends along +X from top of shoulder stub) ── -->
     <link name="upper_arm_link">
       <visual>
         <origin xyz="${upper_arm_l/2.0} 0 0" rpy="0 ${pi/2} 0"/>
-        <geometry><cylinder radius="${r1}" length="${upper_arm_l}"/></geometry>
-        <material name="grey"/>
-      </visual>
-      <visual>
+        <geometry><cylinder radius="${r_upper_arm}" length="${upper_arm_l}"/></geometry>
+        <material name="grey"/>
+      </visual>
+      <visual>  <!-- elbow collar -->
         <origin xyz="${upper_arm_l} 0 0" rpy="0 ${pi/2} 0"/>
-        <geometry><cylinder radius="${r1*1.7}" length="0.018"/></geometry>
+        <geometry><cylinder radius="${r_upper_arm*1.7}" length="0.018"/></geometry>
         <material name="dark_grey"/>
       </visual>
       <collision>
         <origin xyz="${upper_arm_l/2.0} 0 0" rpy="0 ${pi/2} 0"/>
-        <geometry><cylinder radius="${r1}" length="${upper_arm_l}"/></geometry>
-      </collision>
-      <xacro:inertia_cyl_x m="${m_upper_arm}" r="${r1}" l="${upper_arm_l}"/>
+        <geometry><cylinder radius="${r_upper_arm}" length="${upper_arm_l}"/></geometry>
+      </collision>
+      <xacro:inertia_cyl_x m="${m_upper_arm}" r="${r_upper_arm}" l="${upper_arm_l}"/>
     </link>
     <joint name="elbow_joint" type="revolute">
       <parent link="shoulder_link"/>
       <child  link="upper_arm_link"/>
-      <origin xyz="0 0 ${shoulder_h}" rpy="0 0 0"/>
+      <origin xyz="0 0 ${shoulder_h}" rpy="0 0 0"/>  <!-- top of shoulder stub -->
       <axis xyz="0 1 0"/>
-      <!-- lower=-0.25 keeps forearm tip above base top surface with 10mm clearance
-           (recalculated for forearm_l=145mm, shoulder_z=90mm) -->
-      <limit lower="-0.25" upper="0.57" effort="5.0" velocity="0.10"/>
-      <dynamics damping="0.06" friction="0.08"/>
-    </joint>
-    <!-- Forearm -->
+      <limit lower="${elbow_lo}" upper="${elbow_hi}"
+             effort="${arm_effort}" velocity="${arm_vel}"/>
+      <dynamics damping="${elbow_damp}" friction="${elbow_fric}"/>
+    </joint>
+    <!-- ── Forearm link (extends along +X from elbow tip) ─────────────── -->
     <link name="forearm_link">
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