Commit message: sync

File: orion_ws/src/orion_description/xacro/orion.xacro (robot description, xacro)
@@ -5,80 +5,67 @@
   <xacro:arg name="controllers_file" default="config/ros2_controllers.yaml"/>
 <!--CONSTANTS-->
-  <!-- ── Base ─────────────────────────────────────────────────────────── -->
-  <xacro:property name="base_x"    value="0.320"/>  <!-- length  [m] -->
-  <xacro:property name="base_y"    value="0.350"/>  <!-- width   [m] -->
-  <xacro:property name="base_z"    value="0.080"/>  <!-- height  [m] -->
-  <xacro:property name="base_mass" value="3.5"/>    <!-- kg -->
-  <!-- Wheels -->
-  <xacro:property name="wheel_radius" value="0.050"/>              <!-- m -->
-  <xacro:property name="wheel_width"  value="0.040"/>              <!-- m -->
-  <xacro:property name="wheel_mass"   value="0.3"/>                <!-- kg -->
-  <xacro:property name="wheel_x_off"  value="0.112"/>              <!-- m from base centre -->
-  <xacro:property name="wheel_y_off"  value="0.195"/>              <!-- m from base centre -->
-  <xacro:property name="wheel_z_off"  value="${-base_z/2.0}"/>     <!-- m (wheel axle at base bottom) -->
-  <xacro:property name="wheel_mu"     value="1.0"/>                <!-- longitudinal friction -->
-  <xacro:property name="wheel_mu2"    value="0.001"/>              <!-- lateral friction -->
-<!-- Sensors -->
-  <xacro:property name="mast_r"  value="0.010"/>   <!-- LiDAR mast radius  [m] -->
-  <xacro:property name="mast_h"  value="0.300"/>   <!-- LiDAR mast height  [m] -->
-  <xacro:property name="mast_x"  value="0.000"/>   <!-- mast X offset from base centre [m] -->
-  <xacro:property name="mast_y"  value="0.000"/>   <!-- mast Y offset from base centre [m] -->
-  <xacro:property name="lidar_r" value="0.038"/>   <!-- LiDAR body radius  [m] -->
-  <xacro:property name="lidar_h" value="0.041"/>   <!-- LiDAR body height  [m] -->
-  <xacro:property name="lidar_m" value="0.185"/>   <!-- LiDAR mass         [kg] -->
-  <xacro:property name="imu_xyz" value="0.02"/>    <!-- IMU cube side      [m] -->
-  <xacro:property name="shoulder_mount_x" value="${base_x/2.0}"/>  <!-- = 0.160 m -->
-  <xacro:property name="shoulder_mount_z" value="0.0"/>            <!-- base_link origin is mid-height -->
-  <!-- Link lengths [m] -->
-  <xacro:property name="shoulder_h"   value="0.050"/>  <!-- shoulder stub (vertical, +Z) -->
-  <xacro:property name="upper_arm_l"  value="0.220"/>  <!-- upper arm (along +X after elbow) -->
-  <xacro:property name="forearm_l"    value="0.145"/>  <!-- forearm (along +X after wrist) -->
-  <xacro:property name="gripper_l"    value="0.055"/>  <!-- gripper body depth along +X -->
-  <xacro:property name="gripper_tcp"  value="0.050"/>  <!-- gripper base → TCP tip along +X -->
-  <!-- Link cross-section radii [m] (cylinder approximations) -->
+  <xacro:property name="base_x"    value="0.320"/>
+  <xacro:property name="base_y"    value="0.350"/>
+  <xacro:property name="base_z"    value="0.080"/>
+  <xacro:property name="base_mass" value="3.5"/>
+  <xacro:property name="wheel_radius" value="0.050"/>
+  <xacro:property name="wheel_width"  value="0.040"/>
+  <xacro:property name="wheel_mass"   value="0.3"/>
+  <xacro:property name="wheel_x_off"  value="0.112"/>
+  <xacro:property name="wheel_y_off"  value="0.195"/>
+  <xacro:property name="wheel_z_off"  value="${-base_z/2.0}"/>
+  <xacro:property name="wheel_mu"     value="1.0"/>
+  <xacro:property name="wheel_mu2"    value="0.001"/>
+  <xacro:property name="mast_r"  value="0.010"/>
+  <xacro:property name="mast_h"  value="0.300"/>
+  <xacro:property name="mast_x"  value="0.000"/>
+  <xacro:property name="mast_y"  value="0.000"/>
+  <xacro:property name="lidar_r" value="0.038"/>
+  <xacro:property name="lidar_h" value="0.041"/>
+  <xacro:property name="lidar_m" value="0.185"/>
+  <xacro:property name="imu_xyz" value="0.02"/>
+  <xacro:property name="shoulder_mount_x" value="${base_x/2.0}"/>
+  <xacro:property name="shoulder_mount_z" value="0.0"/>
+  <xacro:property name="shoulder_h"   value="0.050"/>
+  <xacro:property name="upper_arm_l"  value="0.220"/>
+  <xacro:property name="forearm_l"    value="0.145"/>
+  <xacro:property name="gripper_l"    value="0.055"/>
+  <xacro:property name="gripper_tcp"  value="0.050"/>
   <xacro:property name="r_shoulder"  value="0.020"/>
   <xacro:property name="r_upper_arm" value="0.018"/>
   <xacro:property name="r_forearm"   value="0.015"/>
   <xacro:property name="r_gripper"   value="0.012"/>
-  <!-- Link masses [kg] -->
   <xacro:property name="m_shoulder"  value="0.300"/>
   <xacro:property name="m_upper_arm" value="0.308"/>
   <xacro:property name="m_forearm"   value="0.199"/>
-  <xacro:property name="m_gripper"   value="0.120"/>  <!-- gripper body (fingers split below) -->
-  <!-- Joint limits [rad] — arm revolutes -->
-  <xacro:property name="shoulder_lo"  value="-0.73"/>  <!-- −41.8 ° -->
-  <xacro:property name="shoulder_hi"  value=" 1.30"/>  <!--  74.5 ° -->
-  <xacro:property name="elbow_lo"     value="-0.25"/>  <!-- −14.3 ° -->
-  <xacro:property name="elbow_hi"     value=" 0.57"/>  <!--  32.7 ° -->
-  <xacro:property name="wrist_lo"     value=" 0.00"/>  <!--   0.0 ° -->
-  <xacro:property name="wrist_hi"     value=" 2.70"/>  <!-- 154.7 ° -->
-  <!-- Joint limits [rad] — ball-and-socket (gripper) -->
-  <xacro:property name="gp_lo"  value="-1.57"/>  <!-- pitch ±90 ° -->
+  <xacro:property name="m_gripper"   value="0.120"/>
+  <xacro:property name="shoulder_lo"  value="-0.73"/>
+  <xacro:property name="shoulder_hi"  value=" 1.30"/>
+  <xacro:property name="elbow_lo"     value="-0.25"/>
+  <xacro:property name="elbow_hi"     value=" 0.57"/>
+  <xacro:property name="wrist_lo"     value=" 0.00"/>
+  <xacro:property name="wrist_hi"     value=" 2.70"/>
+  <xacro:property name="gp_lo"  value="-1.57"/>
   <xacro:property name="gp_hi"  value=" 1.57"/>
-  <xacro:property name="gy_lo"  value="-1.57"/>  <!-- yaw   ±90 ° -->
+  <xacro:property name="gy_lo"  value="-1.57"/>
   <xacro:property name="gy_hi"  value=" 1.57"/>
-  <xacro:property name="gr_lo"  value="-1.57"/>  <!-- roll  ±90 ° -->
+  <xacro:property name="gr_lo"  value="-1.57"/>
   <xacro:property name="gr_hi"  value=" 1.57"/>
-  <!-- Joint dynamics -->
   <xacro:property name="shoulder_damp"  value="0.08"/>  <xacro:property name="shoulder_fric" value="0.10"/>
   <xacro:property name="elbow_damp"     value="0.06"/>  <xacro:property name="elbow_fric"    value="0.08"/>
   <xacro:property name="wrist_damp"     value="0.04"/>  <xacro:property name="wrist_fric"    value="0.06"/>
   <xacro:property name="gripper_damp"   value="0.02"/>  <xacro:property name="gripper_fric"  value="0.03"/>
-  <!-- Actuator limits -->
-  <xacro:property name="arm_effort"    value="5.0"/>   <!-- Nm, all arm joints -->
-  <xacro:property name="arm_vel"       value="1.0"/>   <!-- rad/s (raised from 0.10 for sim) -->
-  <xacro:property name="gripper_effort" value="5.0"/>  <!-- N -->
-  <xacro:property name="gripper_vel"    value="0.10"/> <!-- m/s -->
-  <xacro:property name="gripper_stroke" value="0.025"/><!-- m, each finger from centre -->
-  <!-- Gripper finger geometry (L-shaped: rail + jaw) -->
-  <xacro:property name="finger_w"         value="0.012"/>  <!-- rail width (thin slab along base side) [m] -->
-  <xacro:property name="finger_h"         value="0.018"/>  <!-- finger height — matches gripper_base [m] -->
-  <xacro:property name="finger_jaw_l"     value="0.055"/>  <!-- jaw forward protrusion past base [m] -->
-  <xacro:property name="finger_jaw_w"     value="0.020"/>  <!-- jaw width (inward-facing pad) [m] -->
-  <xacro:property name="finger_bracket_l" value="0.018"/>  <!-- rear bracket depth behind base [m] -->
-  <xacro:property name="finger_bracket_w" value="0.028"/>  <!-- rear bracket inward span [m] -->
-  <!-- ════════════════════════════════════════════════════════════════════
-       2.  MATERIALS
-       ════════════════════════════════════════════════════════════════════ -->
+  <xacro:property name="arm_effort"    value="5.0"/>
+  <xacro:property name="arm_vel"       value="1.0"/>
+  <xacro:property name="gripper_effort" value="5.0"/>
+  <xacro:property name="gripper_vel"    value="0.10"/>
+  <xacro:property name="gripper_stroke" value="0.025"/>
+  <xacro:property name="finger_w"         value="0.012"/>
+  <xacro:property name="finger_h"         value="0.018"/>
+  <xacro:property name="finger_jaw_l"     value="0.055"/>
+  <xacro:property name="finger_jaw_w"     value="0.020"/>
+  <xacro:property name="finger_bracket_l" value="0.018"/>
+  <xacro:property name="finger_bracket_w" value="0.028"/>
+<!--colours-->
   <material name="grey">      <color rgba="0.60 0.60 0.60 1.0"/></material>
   <material name="dark_grey"> <color rgba="0.25 0.25 0.25 1.0"/></material>
@@ -95,8 +82,5 @@
     </gazebo>
   </xacro:macro>
-  <!-- ════════════════════════════════════════════════════════════════════
-       3.  INERTIA HELPER MACROS
-       ════════════════════════════════════════════════════════════════════ -->
-  <!-- Cylinder with long axis along +Z, CoM at geometric centre -->
+<!--inertia macro-->
   <xacro:macro name="inertia_cyl_z" params="m r l">
     <inertial>
@@ -110,5 +94,4 @@
     </inertial>
   </xacro:macro>
-  <!-- Cylinder with long axis along +X, CoM at geometric centre -->
   <xacro:macro name="inertia_cyl_x" params="m r l">
     <inertial>
@@ -122,5 +105,4 @@
     </inertial>
   </xacro:macro>
-  <!-- Box with CoM at (ox, oy, oz) from the link origin -->
   <xacro:macro name="inertia_box" params="m x y z ox oy oz">
     <inertial>
@@ -134,5 +116,4 @@
     </inertial>
   </xacro:macro>
-  <!-- Point mass (for zero-length ball-socket intermediate links) -->
   <xacro:macro name="inertia_point" params="m">
     <inertial>
@@ -142,10 +123,8 @@
     </inertial>
   </xacro:macro>
-  <!-- ════════════════════════════════════════════════════════════════════
-       4.  BASE
-       ════════════════════════════════════════════════════════════════════ -->
+<!--base macros-->
   <xacro:macro name="base">
     <link name="base_link">
-      <!-- Outer shell -->
+      <!-- outer shell -->
       <visual>
         <origin xyz="0 0 0" rpy="0 0 0"/>
@@ -153,5 +132,5 @@
         <material name="dark_grey"/>
       </visual>
-      <!-- Top plate -->
+      <!-- upper plate -->
       <visual>
         <origin xyz="0 0 ${base_z/2.0 - 0.004}" rpy="0 0 0"/>
@@ -159,5 +138,5 @@
         <material name="grey"/>
       </visual>
-      <!-- Battery layer -->
+      <!-- battery layer -->
       <visual>
         <origin xyz="-0.050 0 ${-base_z/2.0 + 0.0175}" rpy="0 0 0"/>
@@ -165,5 +144,5 @@
         <material name="black"/>
       </visual>
-      <!-- Motor driver layer -->
+      <!-- motor driver layer -->
       <visual>
         <origin xyz="-0.04 0 ${-base_z/2.0 + 0.048}" rpy="0 0 0"/>
@@ -171,5 +150,5 @@
         <material name="dark_grey"/>
       </visual>
-      <!-- Power + ESP32 layer -->
+      <!-- power layer -->
       <visual>
         <origin xyz="0 0 ${-base_z/2.0 + 0.068}" rpy="0 0 0"/>
@@ -177,5 +156,5 @@
         <material name="dark_grey"/>
       </visual>
-      <!-- Raspberry Pi 5 PCB -->
+      <!--pi pcb-->
       <visual>
         <origin xyz="-0.07 0.03 ${-base_z/2.0 + 0.060}" rpy="0 0 0"/>
@@ -189,5 +168,5 @@
       <inertial>
         <mass value="${base_mass}"/>
-        <origin xyz="-0.056 0 0" rpy="0 0 0"/>  <!-- CoM: electronics in rear third -->
+        <origin xyz="-0.056 0 0" rpy="0 0 0"/>
         <inertia
           ixx="${(1.0/12.0)*base_mass*(base_y*base_y + base_z*base_z)}"
@@ -213,7 +192,5 @@
     </gazebo>
   </xacro:macro>
-  <!-- ════════════════════════════════════════════════════════════════════
-       5.  WHEELS (mecanum)
-       ════════════════════════════════════════════════════════════════════ -->
+<!--mecanum wheel macro-->
   <xacro:macro name="mecanum_wheel" params="name x_sign y_sign fdir1_y mu_val">
     <link name="${name}_wheel_link">
@@ -277,9 +254,7 @@
     <xacro:mecanum_wheel name="rear_right"  x_sign="-1" y_sign="-1" fdir1_y=" 1" mu_val="1.0"/>
   </xacro:macro>
-  <!-- ════════════════════════════════════════════════════════════════════
-       6.  SENSORS
-       ════════════════════════════════════════════════════════════════════ -->
+  <!--sensor macros-->
   <xacro:macro name="sensors">
-    <!-- LiDAR mast -->
+    <!-- lidar mast -->
     <link name="lidar_mast_link">
       <visual>
@@ -307,5 +282,5 @@
       <origin xyz="${mast_x} ${mast_y} ${base_z/2.0}" rpy="0 0 0"/>
     </joint>
-    <!-- LiDAR sensor link -->
+    <!--lidar-->
     <link name="lidar_link">
       <visual>
@@ -407,12 +382,6 @@
     </gazebo>
   </xacro:macro>
-  <!-- ════════════════════════════════════════════════════════════════════
-       7.  ARM
-       Chain: shoulder_link → upper_arm_link → forearm_link → gripper
-       All revolutes rotate about +Y (sagittal plane).
-       Ball-and-socket gripper: 3 × revolute at same point (pitch/yaw/roll).
-       ════════════════════════════════════════════════════════════════════ -->
+  <!--arm marco-->
   <xacro:macro name="arm">
-    <!-- ── Shoulder link (vertical stub, rotates about +Y at base front) ── -->
     <link name="shoulder_link">
       <visual>
@@ -421,5 +390,5 @@
         <material name="grey"/>
       </visual>
-      <visual>  <!-- collar ring at base of stub -->
+      <visual>
         <origin xyz="0 0 0.010" rpy="0 0 0"/>
         <geometry><cylinder radius="${r_shoulder*1.9}" length="0.020"/></geometry>
@@ -441,5 +410,4 @@
       <dynamics damping="${shoulder_damp}" friction="${shoulder_fric}"/>
     </joint>
-    <!-- ── Upper arm link (extends along +X from top of shoulder stub) ── -->
     <link name="upper_arm_link">
       <visual>
@@ -448,5 +416,5 @@
         <material name="grey"/>
       </visual>
-      <visual>  <!-- elbow collar -->
+      <visual>
         <origin xyz="${upper_arm_l} 0 0" rpy="0 ${pi/2} 0"/>
         <geometry><cylinder radius="${r_upper_arm*1.7}" length="0.018"/></geometry>
@@ -462,5 +430,5 @@
       <parent link="shoulder_link"/>
       <child  link="upper_arm_link"/>
-      <origin xyz="0 0 ${shoulder_h}" rpy="0 0 0"/>  <!-- top of shoulder stub -->
+      <origin xyz="0 0 ${shoulder_h}" rpy="0 0 0"/>
       <axis xyz="0 1 0"/>
       <limit lower="${elbow_lo}" upper="${elbow_hi}"
@@ -468,5 +436,4 @@
       <dynamics damping="${elbow_damp}" friction="${elbow_fric}"/>
     </joint>
-    <!-- ── Forearm link (extends along +X from elbow tip) ─────────────── -->
     <link name="forearm_link">
       <visual>
@@ -475,5 +442,5 @@
         <material name="grey"/>
       </visual>
-      <visual>  <!-- wrist collar -->
+      <visual>
         <origin xyz="${forearm_l} 0 0" rpy="0 ${pi/2} 0"/>
         <geometry><cylinder radius="${r_forearm*1.6}" length="0.015"/></geometry>
@@ -489,5 +456,5 @@
       <parent link="upper_arm_link"/>
       <child  link="forearm_link"/>
-      <origin xyz="${upper_arm_l} 0 0" rpy="0 0 0"/>  <!-- tip of upper arm -->
+      <origin xyz="${upper_arm_l} 0 0" rpy="0 0 0"/>
       <axis xyz="0 1 0"/>
       <limit lower="${wrist_lo}" upper="${wrist_hi}"
@@ -495,15 +462,4 @@
       <dynamics damping="${wrist_damp}" friction="${wrist_fric}"/>
     </joint>
-    <!-- ── Ball-and-socket gripper joint ──────────────────────────────────
-         URDF has no native spherical joint type.  We approximate it with
-         three consecutive revolute joints sharing the same physical origin
-         (forearm tip), connected by massless zero-length intermediate links.
-         Order: pitch (+Y) → yaw (+Z) → roll (+X)
-         This decomposition matches the intuitive "point and twist" motion:
-           pitch raises/lowers the gripper
-           yaw sweeps it left/right
-           roll spins the fingers about the approach axis
-    ──────────────────────────────────────────────────────────────────── -->
-    <!-- Pitch intermediate link (massless) -->
     <link name="gripper_pitch_link">
       <xacro:inertia_point m="0.001"/>
@@ -512,5 +468,5 @@
       <parent link="forearm_link"/>
       <child  link="gripper_pitch_link"/>
-      <origin xyz="${forearm_l} 0 0" rpy="0 0 0"/>  <!-- tip of forearm -->
+      <origin xyz="${forearm_l} 0 0" rpy="0 0 0"/>
       <axis xyz="0 1 0"/>
       <limit lower="${gp_lo}" upper="${gp_hi}"
@@ -518,5 +474,4 @@
       <dynamics damping="${gripper_damp}" friction="${gripper_fric}"/>
     </joint>
-    <!-- Yaw intermediate link (massless) -->
     <link name="gripper_yaw_link">
       <xacro:inertia_point m="0.001"/>
@@ -525,5 +480,5 @@
       <parent link="gripper_pitch_link"/>
       <child  link="gripper_yaw_link"/>
-      <origin xyz="0 0 0" rpy="0 0 0"/>  <!-- same physical point -->
+      <origin xyz="0 0 0" rpy="0 0 0"/>
       <axis xyz="0 0 1"/>
       <limit lower="${gy_lo}" upper="${gy_hi}"
@@ -531,5 +486,4 @@
       <dynamics damping="${gripper_damp}" friction="${gripper_fric}"/>
     </joint>
-    <!-- Roll intermediate link (massless) -->
     <link name="gripper_roll_link">
       <xacro:inertia_point m="0.001"/>
@@ -538,5 +492,5 @@
       <parent link="gripper_yaw_link"/>
       <child  link="gripper_roll_link"/>
-      <origin xyz="0 0 0" rpy="0 0 0"/>  <!-- same physical point -->
+      <origin xyz="0 0 0" rpy="0 0 0"/>
       <axis xyz="1 0 0"/>
       <limit lower="${gr_lo}" upper="${gr_hi}"
@@ -544,5 +498,4 @@
       <dynamics damping="${gripper_damp}" friction="${gripper_fric}"/>
     </joint>
-    <!-- ── Gripper body ─────────────────────────────────────────────────── -->
     <link name="gripper_base_link">
       <visual>
@@ -563,18 +516,5 @@
       <origin xyz="0 0 0" rpy="0 0 0"/>
     </joint>
-    <!--
-      L-shaped fingers: each finger has two boxes sharing the same link/joint.
-        • rail  : thin slab (finger_w × finger_h) spanning the full gripper_base length in X.
-                  Its outer Y face is flush with the outer face of gripper_base (0.052/2).
-                  Because it rides along the base side, it always covers the base — no gap.
-        • jaw   : thicker forward-protruding pad (finger_jaw_l × finger_jaw_w × finger_h)
-                  starting at the front of the base and extending outward in X.
-                  It sits at the inner Y edge of the rail so it forms the ─┘ corner.
-      Joint origin is at X=0, Y = ±(0.052/2 − finger_w/2) so the rail outer face stays
-      flush with the gripper base outer face at all joint positions.
-    -->
-    <!-- Left finger (active, commanded by gripper_controller) -->
     <link name="gripper_left_link">
-      <!-- Rail: covers full base length, thin, outer-face flush with base -->
       <visual>
         <origin xyz="${gripper_l/2.0} 0 0" rpy="0 0 0"/>
@@ -586,5 +526,4 @@
         <geometry><box size="${gripper_l} ${finger_w} ${finger_h}"/></geometry>
       </collision>
-      <!-- Jaw: protrudes forward, inset toward centre by finger_w -->
       <visual>
         <origin xyz="${gripper_l + finger_jaw_l/2.0} ${-(finger_jaw_w - finger_w)/2.0} 0" rpy="0 0 0"/>
@@ -596,5 +535,4 @@
         <geometry><box size="${finger_jaw_l} ${finger_jaw_w} ${finger_h}"/></geometry>
       </collision>
-      <!-- Rear bracket: horizontal bar behind gripper_base, spans inward → looks mechanically mounted -->
       <visual>
         <origin xyz="${-finger_bracket_l/2.0} ${-(finger_bracket_w - finger_w)/2.0} 0" rpy="0 0 0"/>
@@ -618,7 +556,5 @@
       <dynamics damping="0.01" friction="0.01"/>
     </joint>
-    <!-- Right finger (mirrors left via mimic) -->
     <link name="gripper_right_link">
-      <!-- Rail -->
       <visual>
         <origin xyz="${gripper_l/2.0} 0 0" rpy="0 0 0"/>
@@ -630,5 +566,4 @@
         <geometry><box size="${gripper_l} ${finger_w} ${finger_h}"/></geometry>
       </collision>
-      <!-- Jaw: protrudes forward, inset toward centre by finger_w -->
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
Commit message: Edited shoulder to also be aligned in +X for easier IK and convention to be aligned in primary translational axis

File: orion_ws/src/orion_description/xacro/orion.xacro (robot description, xacro)
@@ -25,6 +25,6 @@
   <xacro:property name="lidar_m" value="0.185"/>
   <xacro:property name="imu_xyz" value="0.02"/>
-  <xacro:property name="shoulder_mount_x" value="${base_x/2.0}"/>
-  <xacro:property name="shoulder_mount_z" value="0.0"/>
+  <xacro:property name="shoulder_mount_x" value="${base_x/2.0 - r_shoulder - 0.006}"/>
+  <xacro:property name="shoulder_mount_z" value="${base_z/2.0}"/>
   <xacro:property name="shoulder_h"   value="0.050"/>
   <xacro:property name="upper_arm_l"  value="0.220"/>
@@ -40,8 +40,8 @@
   <xacro:property name="m_forearm"   value="0.199"/>
   <xacro:property name="m_gripper"   value="0.120"/>
-  <xacro:property name="shoulder_lo"  value="-0.73"/>
-  <xacro:property name="shoulder_hi"  value=" 1.30"/>
+  <xacro:property name="shoulder_lo"  value="-1.58"/>
+  <xacro:property name="shoulder_hi"  value="0.79"/>
   <xacro:property name="elbow_lo"     value="-0.25"/>
-  <xacro:property name="elbow_hi"     value=" 0.57"/>
+  <xacro:property name="elbow_hi"     value=" 1.57"/>
   <xacro:property name="wrist_lo"     value=" 0.00"/>
   <xacro:property name="wrist_hi"     value=" 2.70"/>
@@ -386,18 +386,18 @@
     <link name="shoulder_link">
       <visual>
-        <origin xyz="0 0 ${shoulder_h/2.0}" rpy="0 0 0"/>
+        <origin xyz="${shoulder_h/2.0} 0 0" rpy="0 ${pi/2} 0"/>
         <geometry><cylinder radius="${r_shoulder}" length="${shoulder_h}"/></geometry>
         <material name="grey"/>
       </visual>
       <visual>
-        <origin xyz="0 0 0.010" rpy="0 0 0"/>
+        <origin xyz="0.010 0 0" rpy="0 ${pi/2} 0"/>
         <geometry><cylinder radius="${r_shoulder*1.9}" length="0.020"/></geometry>
         <material name="dark_grey"/>
       </visual>
       <collision>
-        <origin xyz="0 0 ${shoulder_h/2.0}" rpy="0 0 0"/>
+        <origin xyz="${shoulder_h/2.0} 0 0" rpy="0 ${pi/2} 0"/>
         <geometry><cylinder radius="${r_shoulder}" length="${shoulder_h}"/></geometry>
       </collision>
-      <xacro:inertia_cyl_z m="${m_shoulder}" r="${r_shoulder}" l="${shoulder_h}"/>
+      <xacro:inertia_cyl_x m="${m_shoulder}" r="${r_shoulder}" l="${shoulder_h}"/>
     </link>
     <joint name="shoulder_joint" type="revolute">
@@ -430,5 +430,5 @@
       <parent link="shoulder_link"/>
       <child  link="upper_arm_link"/>
-      <origin xyz="0 0 ${shoulder_h}" rpy="0 0 0"/>
+      <origin xyz="${shoulder_h} 0 0" rpy="0 0 0"/>
       <axis xyz="0 1 0"/>
       <limit lower="${elbow_lo}" upper="${elbow_hi}"
