Commit message: Updating orion.urdf and orion.xacro to Model 1

File: orion_ws/src/orion_description/urdf/orion.urdf (robot description, URDF)
Before this commit: robot orion, 2 links, 1 joints
Links:
- added link camera_link; visual box size=0.03 0.03 0.03
- added link caster; visual sphere radius=0.03
- added link imu_link
- added link left_wheel, mass 0.5; visual cylinder length=0.02 radius=0.05
- added link lidar_link; visual cylinder length=0.05 radius=0.03
- added link link1, mass 1.0; visual cylinder length=0.2 radius=0.02
- added link link2, mass 0.8; visual cylinder length=0.2 radius=0.02
- added link right_wheel, mass 0.5; visual cylinder length=0.02 radius=0.05
- link base_link: mass None -> 2.0; geometry collision box size=0.3 0.2 0.1; visual box size=0.3 0.2 0.1
- link shoulder_link: mass 1 -> 0.3; geometry visual box size=0.05 0.05 0.05
Joints:
- added joint camera_joint: type fixed, parent base_link, child camera_link, origin xyz=0.15 0 0.2
- added joint caster_joint: type fixed, parent base_link, child caster, origin xyz=-0.1 0 -0.05
- added joint imu_joint: type fixed, parent base_link, child imu_link, origin xyz=0 0 0.1
- added joint joint1: type revolute, parent shoulder_link, child link1, origin xyz=0 0 0.05, axis 0 1 0
- added joint joint2: type revolute, parent link1, child link2, origin xyz=0 0 0.2, axis 0 1 0
- added joint left_wheel_joint: type continuous, parent base_link, child left_wheel, origin xyz=0 0.1 -0.05, axis 0 1 0
- added joint lidar_joint: type fixed, parent base_link, child lidar_link, origin xyz=0.1 0 0.15
- added joint right_wheel_joint: type continuous, parent base_link, child right_wheel, origin xyz=0 -0.1 -0.05, axis 0 1 0
- joint shoulder_joint: origin xyz=0 0 0.1 rpy=0 0 0 -> xyz=0 0 0.1; type continuous -> revolute

File: orion_ws/src/orion_description/xacro/orion.xacro (robot description, xacro)
@@ -2,25 +2,28 @@
 <robot name="orion" xmlns:xacro="http://www.ros.org/wiki/xacro">
   <!-- ================= PARAMETERS ================= -->
-  <xacro:property name="wheel_radius" value="0.05"/>
-  <xacro:property name="wheel_width" value="0.02"/>
-  <xacro:property name="wheel_sep" value="0.20"/>
-  <xacro:property name="arm_length" value="0.2"/>
-  <xacro:property name="arm_radius" value="0.02"/>
+  <xacro:property name="wheel_radius" value="0.08"/>
+  <xacro:property name="wheel_width" value="0.04"/>
+  <xacro:property name="wheel_sep" value="0.30"/>
+  <xacro:property name="arm_length" value="0.30"/>
+  <xacro:property name="arm_radius" value="0.03"/>
   <!-- ================= BASE ================= -->
   <link name="base_link">
     <visual>
       <geometry>
-        <box size="0.3 0.2 0.1"/>
+        <box size="0.3 0.2 0.15"/>
       </geometry>
+      <material name="Blue">
+      <color rgba="0 0 1 1"/>
+      </material>
     </visual>
     <collision>
       <geometry>
-        <box size="0.3 0.2 0.1"/>
+        <box size="0.5 0.4 0.15"/>
       </geometry>
     </collision>
     <inertial>
-      <mass value="2.0"/>
+      <mass value="5.0"/>
       <origin xyz="0 0 0"/>
-      <inertia ixx="0.02" iyy="0.02" izz="0.02"
+      <inertia ixx="0.1" iyy="0.1" izz="0.1"
                ixy="0.0" ixz="0.0" iyz="0.0"/>
     </inertial>
@@ -36,7 +39,7 @@
       </visual>
       <inertial>
-        <mass value="0.5"/>
+        <mass value="1.0"/>
         <origin xyz="0 0 0"/>
-        <inertia ixx="0.001" iyy="0.001" izz="0.0005"
+        <inertia ixx="0.005" iyy="0.005" izz="0.01"
                  ixy="0.0" ixz="0.0" iyz="0.0"/>
       </inertial>
@@ -55,5 +58,5 @@
     <visual>
       <geometry>
-        <sphere radius="0.03"/>
+        <sphere radius="0.05"/>
       </geometry>
     </visual>
@@ -68,18 +71,18 @@
     <visual>
       <geometry>
-        <box size="0.05 0.05 0.05"/>
+        <cylinder radius="0.05" length="0.2"/>
       </geometry>
     </visual>
     <inertial>
-      <mass value="0.3"/>
+      <mass value="0.5"/>
       <origin xyz="0 0 0"/>
-      <inertia ixx="0.000125" iyy="0.000125" izz="0.000125"
+      <inertia ixx="0.0005" iyy="0.0005" izz="0.0005"
                ixy="0.0" ixz="0.0" iyz="0.0"/>
     </inertial>
   </link>
-  <joint name="shoulder_joint" type="revolute">
+  <joint name="shoulder_joint" type="continuous">
     <parent link="base_link"/>
     <child link="shoulder_link"/>
-    <origin xyz="0 0 0.1"/>
+    <origin xyz="0 0 0.075"/>
     <axis xyz="0 0 1"/>
   </joint>
@@ -90,10 +93,13 @@
         <cylinder radius="${arm_radius}" length="${arm_length}"/>
       </geometry>
-      <origin rpy="0 1.57 0"/>
+      <origin xyz= "0.15 0 0" rpy="0 1.57 0"/>
+      <material name="Blue">
+      <color rgba="0 0 1 1"/>
+      </material>
     </visual>
     <inertial>
-      <mass value="1.0"/>
+      <mass value="2.0"/>
       <origin xyz="0 0 0"/>
-      <inertia ixx="0.0034" iyy="0.0034" izz="0.0002"
+      <inertia ixx="0.01" iyy="0.01" izz="0.005"
                ixy="0.0" ixz="0.0" iyz="0.0"/>
     </inertial>
@@ -102,6 +108,7 @@
     <parent link="shoulder_link"/>
     <child link="link1"/>
-    <origin xyz="0 0 0.05"/>
+    <origin xyz="0 0 0.1"/>
     <axis xyz="0 1 0"/>
+    <limit lower="-3.71" upper="0.5" effort="10" velocity="1.0"/>
   </joint>
   <!-- ================= ARM LINK 2 ================= -->
@@ -111,10 +118,10 @@
         <cylinder radius="${arm_radius}" length="${arm_length}"/>
       </geometry>
-      <origin rpy="0 1.57 0"/>
+      <origin xyz="0.15 0 0" rpy="0 1.57 0"/>
     </visual>
     <inertial>
-      <mass value="0.8"/>
+      <mass value="1.5"/>
       <origin xyz="0 0 0"/>
-      <inertia ixx="0.0027" iyy="0.0027" izz="0.00016"
+      <inertia ixx="0.0075" iyy="0.0075" izz="0.00375"
                ixy="0.0" ixz="0.0" iyz="0.0"/>
     </inertial>
@@ -123,6 +130,7 @@
     <parent link="link1"/>
     <child link="link2"/>
-    <origin xyz="0 0 ${arm_length}"/>
+    <origin xyz="0.3 0 0"/>
     <axis xyz="0 1 0"/>
+    <limit lower="-1.57" upper="1.57" effort="10" velocity="1.0"/>
   </joint>
   <!-- ================= SENSORS ================= -->
@@ -138,25 +146,12 @@
     <parent link="base_link"/>
     <child link="lidar_link"/>
-    <origin xyz="0.1 0 0.15"/>
+    <origin xyz="0.1 0 0.07"/>
   </joint>
   <!-- IMU -->
   <link name="imu_link"/>
   <joint name="imu_joint" type="fixed">
-    <parent link="base_link"/>
+    <parent link="shoulder_link"/>
     <child link="imu_link"/>
     <origin xyz="0 0 0.1"/>
-  </joint>
-  <!-- Camera -->
-  <link name="camera_link">
-    <visual>
-      <geometry>
-        <box size="0.03 0.03 0.03"/>
-      </geometry>
-    </visual>
-  </link>
-  <joint name="camera_joint" type="fixed">
-    <parent link="base_link"/>
-    <child link="camera_link"/>
-    <origin xyz="0.15 0 0.2"/>
   </joint>
   <!-- ================= ROS2 CONTROL ================= -->
