Commit message: Clean ORION ROS2 workspace (remove vscode + build artifacts)

File: orion_ws/src/orion_description/urdf/orion.urdf (robot description, URDF)
Before this commit: robot orion, 10 links, 9 joints
Links:
- removed link camera_link
- removed link caster
- removed link left_wheel
- removed link link1
- removed link link2
- removed link right_wheel
- added link base_footprint
- added link forearm_link, mass 0.18; collision cylinder length=0.12 radius=0.015; visual cylinder length=0.015 radius=0.024
- added link front_left_wheel_link, mass 0.3; collision cylinder length=0.04 radius=0.05; visual cylinder length=0.012 radius=0.008
- added link front_right_wheel_link, mass 0.3; collision cylinder length=0.04 radius=0.05; visual cylinder length=0.012 radius=0.008
- added link gripper_base_link, mass 0.06; collision box size=0.028 0.052 0.018; visual box size=0.028 0.052 0.018
- added link gripper_left_link, mass 0.03; collision box size=0.044 0.009 0.014; visual box size=0.044 0.009 0.014
- added link gripper_right_link, mass 0.03; collision box size=0.044 0.009 0.014; visual box size=0.044 0.009 0.014
- added link hand_link, mass 0.1; collision cylinder length=0.055 radius=0.012; visual cylinder length=0.055 radius=0.012
- added link lidar_mast_link, mass 0.080; collision cylinder length=0.36 radius=0.01; visual cylinder length=0.36 radius=0.01
- added link rear_left_wheel_link, mass 0.3; collision cylinder length=0.04 radius=0.05; visual cylinder length=0.012 radius=0.008
- added link rear_right_wheel_link, mass 0.3; collision cylinder length=0.04 radius=0.05; visual cylinder length=0.012 radius=0.008
- added link tcp_link
- added link upper_arm_link, mass 0.24; collision cylinder length=0.15 radius=0.018; visual cylinder length=0.018 radius=0.030599999999999995
- link base_link: mass 2.0 -> 3.5; geometry collision box size=0.28 0.32 0.105; visual box size=0.085 0.056 0.004
- link imu_link: mass None -> 0.05; geometry visual box size=0.02 0.02 0.02
- link lidar_link: mass None -> 0.185; geometry collision cylinder length=0.041 radius=0.038; visual box size=0.004 0.012 0.0205
- link shoulder_link: geometry collision cylinder length=0.055 radius=0.02; visual cylinder length=0.020 radius=0.038
Joints:
- removed joint camera_joint
- removed joint caster_joint
- removed joint joint1
- removed joint joint2
- removed joint left_wheel_joint
- removed joint right_wheel_joint
- added joint base_footprint_joint: type fixed, parent base_footprint, child base_link, origin xyz=0 0 0.10250000000000001 rpy=0 0 0
- added joint elbow_joint: type revolute, parent shoulder_link, child upper_arm_link, origin xyz=0 0 0.055 rpy=0 0 0, axis 0 1 0, limit lower=-1.57 upper=0.57 effort=5.0 velocity=0.10
- added joint front_left_wheel_joint: type continuous, parent base_link, child front_left_wheel_link, origin xyz=0.095 0.13 -0.0525 rpy=0 0 0, axis 0 1 0
- added joint front_right_wheel_joint: type continuous, parent base_link, child front_right_wheel_link, origin xyz=0.095 -0.13 -0.0525 rpy=0 0 0, axis 0 1 0
- added joint gripper_base_joint: type fixed, parent hand_link, child gripper_base_link, origin xyz=0.055 0 0 rpy=0 0 0
- added joint gripper_left_joint: type prismatic, parent gripper_base_link, child gripper_left_link, origin xyz=0 0.022 0 rpy=0 0 0, axis 0 1 0, limit lower=0.0 upper=0.025 effort=5.0 velocity=0.10
- added joint gripper_right_joint: type prismatic, parent gripper_base_link, child gripper_right_link, origin xyz=0 -0.022 0 rpy=0 0 0, axis 0 -1 0, limit lower=0.0 upper=0.025 effort=5.0 velocity=0.10
- added joint lidar_mast_joint: type fixed, parent base_link, child lidar_mast_link, origin xyz=-0.1 0.0 0.0525 rpy=0 0 0
- added joint rear_left_wheel_joint: type continuous, parent base_link, child rear_left_wheel_link, origin xyz=-0.095 0.13 -0.0525 rpy=0 0 0, axis 0 1 0
- added joint rear_right_wheel_joint: type continuous, parent base_link, child rear_right_wheel_link, origin xyz=-0.095 -0.13 -0.0525 rpy=0 0 0, axis 0 1 0
- added joint tcp_joint: type fixed, parent gripper_base_link, child tcp_link, origin xyz=0.050 0 0 rpy=0 0 0
- added joint wrist_joint: type revolute, parent upper_arm_link, child forearm_link, origin xyz=0.15 0 0 rpy=0 0 0, axis 0 1 0, limit lower=0.0 upper=2.7 effort=5.0 velocity=0.10
- added joint wrist_roll_joint: type revolute, parent forearm_link, child hand_link, origin xyz=0.12 0 0 rpy=0 0 0, axis 1 0 0, limit lower=-1.0 upper=1.0 effort=5.0 velocity=0.10
- joint imu_joint: origin xyz=0 0 0.1 -> xyz=0 0 0.105 rpy=0 0 0
- joint lidar_joint: origin xyz=0.1 0 0.15 -> xyz=0 0 0.36 rpy=0 0 0; parent base_link -> lidar_mast_link
- joint shoulder_joint: axis 0 0 1 -> 0 1 0; limit (none) -> lower=-1.3 upper=1.57 effort=5.0 velocity=0.10; origin xyz=0 0 0.1 -> xyz=0 0 0.0765 rpy=0 0 0

File: orion_ws/src/orion_description/xacro/arm.xacro (robot description, xacro)
@@ -1,23 +1,10 @@
 <?xml version="1.0"?>
 <robot xmlns:xacro="http://www.ros.org/wiki/xacro">
-  <!-- ================================================================
-       ORION ARM  —  3-DOF planar arm + 2-finger gripper
-         All rotation axes are Y (pitch), giving a fully planar arm.
-         Yaw is provided by the mecanum base — no shoulder yaw joint.
-         Kinematic chain:
-           base_link
-             └─ shoulder_joint    (pitch Y) → shoulder_link
-                  └─ elbow_joint      (pitch Y) → upper_arm_link
-                       └─ wrist_joint     (pitch Y) → forearm_link
-                            └─ wrist_roll_joint (roll X) → hand_link
-                                 └─ gripper_base_joint (fixed)
-                                      ├─ gripper_left_joint  (prismatic +Y)
-                                      └─ gripper_right_joint (prismatic -Y)
-       ================================================================ -->
+  <!--Defining xacro properties-->
   <xacro:property name="base_z"        value="0.105"/>
   <xacro:property name="arm_mount_h"   value="0.024"/>
-  <xacro:property name="shoulder_h"    value="0.12"/>
-  <xacro:property name="upper_arm_l"   value="0.15"/>
-  <xacro:property name="forearm_l"     value="0.06"/>
+  <xacro:property name="shoulder_h"    value="0.055"/>
+  <xacro:property name="upper_arm_l"   value="0.150"/>
+  <xacro:property name="forearm_l"     value="0.120"/>
   <xacro:property name="hand_l"        value="0.055"/>
   <xacro:property name="r0"  value="0.020"/>
@@ -30,4 +17,5 @@
   <xacro:property name="m_hand"       value="0.10"/>
   <xacro:property name="m_gripper"    value="0.12"/>
+  <!--Inertia-->
   <xacro:macro name="inertia_cyl_z" params="m r l">
     <inertial>
@@ -63,6 +51,7 @@
     </inertial>
   </xacro:macro>
+  <!-- ================================================================ -->
   <xacro:macro name="arm">
-    <!-- ── 1. Shoulder link (vertical riser) ─────────────────────── -->
+    <!--Shoulder link-->
     <link name="shoulder_link">
       <visual>
@@ -82,6 +71,4 @@
       <xacro:inertia_cyl_z m="${m_shoulder}" r="${r0}" l="${shoulder_h}"/>
     </link>
-    <!-- base_link → shoulder  ── PITCH (Y)  ─────────────────────── -->
-    <!-- No yaw: the mecanum base handles in-place rotation entirely.  -->
     <joint name="shoulder_joint" type="revolute">
       <parent link="base_link"/>
@@ -89,8 +76,8 @@
       <origin xyz="0 0 ${base_z/2.0 + arm_mount_h}" rpy="0 0 0"/>
       <axis xyz="0 1 0"/>
-      <limit lower="-0.5" upper="1.5" effort="25.0" velocity="1.5"/>
+      <limit lower="-1.3" upper="1.57" effort="5.0" velocity="0.10"/>
       <dynamics damping="0.08" friction="0.10"/>
     </joint>
-    <!-- ── 2. Upper arm (along X) ─────────────────────────────────── -->
+    <!--Upper arm link-->
     <link name="upper_arm_link">
       <visual>
@@ -110,5 +97,4 @@
       <xacro:inertia_cyl_x m="${m_upper_arm}" r="${r1}" l="${upper_arm_l}"/>
     </link>
-    <!-- shoulder → upper_arm  ── PITCH (Y) ──────────────────────── -->
     <joint name="elbow_joint" type="revolute">
       <parent link="shoulder_link"/>
@@ -116,8 +102,8 @@
       <origin xyz="0 0 ${shoulder_h}" rpy="0 0 0"/>
       <axis xyz="0 1 0"/>
-      <limit lower="-1" upper="1" effort="20.0" velocity="1.5"/>
+      <limit lower="-1.57" upper="0.57" effort="5.0" velocity="0.10"/>
       <dynamics damping="0.06" friction="0.08"/>
     </joint>
-    <!-- ── 3. Forearm (along X) ───────────────────────────────────── -->
+    <!--Forearm link-->
     <link name="forearm_link">
       <visual>
@@ -137,5 +123,4 @@
       <xacro:inertia_cyl_x m="${m_forearm}" r="${r2}" l="${forearm_l}"/>
     </link>
-    <!-- upper_arm → forearm  ── PITCH (Y) ───────────────────────── -->
     <joint name="wrist_joint" type="revolute">
       <parent link="upper_arm_link"/>
@@ -143,8 +128,8 @@
       <origin xyz="${upper_arm_l} 0 0" rpy="0 0 0"/>
       <axis xyz="0 1 0"/>
-      <limit lower="0" upper="2.79" effort="15.0" velocity="2.0"/>
+      <limit lower="0.0" upper="2.7" effort="5.0" velocity="0.10"/>
       <dynamics damping="0.04" friction="0.06"/>
     </joint>
-    <!-- ── 4. Hand / tool mount (along X) ────────────────────────── -->
+    <!--Hand link-->
     <link name="hand_link">
       <visual>
@@ -159,13 +144,13 @@
       <xacro:inertia_cyl_x m="${m_hand}" r="${r3}" l="${hand_l}"/>
     </link>
-    <!-- forearm → hand  ── ROLL (X) ─────────────────────────────── -->
-    <joint name="wrist_roll_joint" type="continuous">
+    <joint name="wrist_roll_joint" type="revolute">
       <parent link="forearm_link"/>
       <child  link="hand_link"/>
       <origin xyz="${forearm_l} 0 0" rpy="0 0 0"/>
       <axis xyz="1 0 0"/>
+      <limit lower="-1.0" upper="1.0" effort="5.0" velocity="0.10"/>
       <dynamics damping="0.02" friction="0.03"/>
     </joint>
-    <!-- ── 5. Gripper base ────────────────────────────────────────── -->
+    <!--Gripper base link-->
     <link name="gripper_base_link">
       <visual>
@@ -186,5 +171,5 @@
       <origin xyz="${hand_l} 0 0" rpy="0 0 0"/>
     </joint>
-    <!-- ── 6. Left finger ─────────────────────────────────────────── -->
+    <!--Left gripper-->
     <link name="gripper_left_link">
       <visual>
@@ -208,5 +193,5 @@
       <dynamics damping="0.01" friction="0.01"/>
     </joint>
-    <!-- ── 7. Right finger ────────────────────────────────────────── -->
+    <!--Right gripper-->
     <link name="gripper_right_link">
       <visual>
@@ -230,5 +215,5 @@
       <dynamics damping="0.01" friction="0.01"/>
     </joint>
-    <!-- ── TCP ────────────────────────────────────────────────────── -->
+    <!--TCP-->
     <link name="tcp_link"/>
     <joint name="tcp_joint" type="fixed">
@@ -237,4 +222,87 @@
       <origin xyz="0.050 0 0" rpy="0 0 0"/>
     </joint>
+    <!--Gazebo link colours-->
+    <gazebo reference="shoulder_link">   <material>Gazebo/Grey</material></gazebo>
+    <gazebo reference="upper_arm_link">  <material>Gazebo/Grey</material></gazebo>
+    <gazebo reference="forearm_link">    <material>Gazebo/Grey</material></gazebo>
+    <gazebo reference="hand_link">       <material>Gazebo/Grey</material></gazebo>
+    <gazebo reference="gripper_base_link"><material>Gazebo/DarkGrey</material></gazebo>
+    <gazebo reference="gripper_left_link"><material>Gazebo/Grey</material></gazebo>
+    <gazebo reference="gripper_right_link"><material>Gazebo/Grey</material></gazebo>
+    <!--Gazebo joint friction-->
+    <gazebo reference="shoulder_joint">
+      <implicitSpringDamper>true</implicitSpringDamper>
+      <provideFeedback>true</provideFeedback>
+    </gazebo>
+    <gazebo reference="elbow_joint">
+      <implicitSpringDamper>true</implicitSpringDamper>
+      <provideFeedback>true</provideFeedback>
+    </gazebo>
+    <gazebo reference="wrist_joint">
+      <implicitSpringDamper>true</implicitSpringDamper>
+      <provideFeedback>true</provideFeedback>
+    </gazebo>
+    <gazebo reference="wrist_roll_joint">
+      <implicitSpringDamper>true</implicitSpringDamper>
+      <provideFeedback>true</provideFeedback>
+    </gazebo>
+    <!--ROS2 Control plugin-->
+    <ros2_control name="orion_arm" type="system">
+      <hardware>
+        <plugin>gz_ros2_control/GazeboSimSystem</plugin>
+      </hardware>
+      <joint name="shoulder_joint">
+        <command_interface name="position"/>
+        <state_interface   name="position">
+          <param name="initial_value">0.0</param>
+        </state_interface>
+        <state_interface name="velocity"/>
+        <state_interface name="effort"/>
+      </joint>
+      <joint name="elbow_joint">
+        <command_interface name="position"/>
+        <state_interface   name="position">
+          <param name="initial_value">0.0</param>
+        </state_interface>
+        <state_interface name="velocity"/>
+        <state_interface name="effort"/>
+      </joint>
+      <joint name="wrist_joint">
+        <command_interface name="position"/>
+        <state_interface   name="position">
+          <param name="initial_value">0.0</param>
+        </state_interface>
+        <state_interface name="velocity"/>
+        <state_interface name="effort"/>
+      </joint>
+      <joint name="wrist_roll_joint">
+        <command_interface name="position"/>
+        <state_interface   name="position">
+          <param name="initial_value">0.0</param>
+        </state_interface>
+        <state_interface name="velocity"/>
+        <state_interface name="effort"/>
+      </joint>
+      <joint name="gripper_left_joint">
+        <command_interface name="position">
+          <param name="min">0.0</param>
+          <param name="max">0.025</param>
+        </command_interface>
+        <state_interface name="position">
+          <param name="initial_value">0.0</param>
+        </state_interface>
+        <state_interface name="velocity"/>
+      </joint>
+      <joint name="gripper_right_joint">
+        <command_interface name="position">
+          <param name="min">0.0</param>
+          <param name="max">0.025</param>
+        </command_interface>
+        <state_interface name="position">
+          <param name="initial_value">0.0</param>
+        </state_interface>
+        <state_interface name="velocity"/>
+      </joint>
+    </ros2_control>
   </xacro:macro>
 </robot>

File: orion_ws/src/orion_description/xacro/base.xacro (robot description, xacro)
@@ -2,7 +2,9 @@
 <robot xmlns:xacro="http://www.ros.org/wiki/xacro">
   <!-- ================================================================
-       ORION BASE  —  Model 2 dimensions
-         280 mm (x, front-back)  ×  320 mm (y, left-right)  ×  105 mm (z)
-       Layered internals: Battery → Drivers → Power/ESP32 → Pi5 → Top plate
+       ORION BASE  —  Gazebo-ready
+         Gazebo additions:
+           • <gazebo reference> surface/friction for base_link
+           • Gazebo material colours
+           • gz_ros2_control + JointStateBroadcaster plugin
        ================================================================ -->
   <xacro:property name="base_x"     value="0.280"/>
@@ -10,10 +12,8 @@
   <xacro:property name="base_z"     value="0.105"/>
   <xacro:property name="base_mass"  value="3.5"/>
-  <!-- Wheel params needed to compute base_link height above ground -->
   <xacro:property name="wheel_radius" value="0.050"/>
-  <!-- base_link sits at wheel_radius + half chassis height above the ground -->
-  <xacro:property name="base_link_z" value="${wheel_radius + base_z / 2.0}"/>
+  <xacro:property name="base_link_z"  value="${wheel_radius + base_z / 2.0}"/>
   <xacro:macro name="base">
-    <!-- ── Ground reference frame (no geometry / no inertia) ── -->
+    <!-- ── Ground reference frame ──────────────────────────────── -->
     <link name="base_footprint"/>
     <joint name="base_footprint_joint" type="fixed">
@@ -22,5 +22,5 @@
       <origin xyz="0 0 ${base_link_z}" rpy="0 0 0"/>
     </joint>
-    <!-- ── Main chassis ── -->
+    <!-- ── Main chassis ─────────────────────────────────────────── -->
     <link name="base_link">
       <!-- Outer shell -->
@@ -30,5 +30,5 @@
         <material name="dark_grey"/>
       </visual>
-      <!-- Top plate (slightly proud) -->
+      <!-- Top plate -->
       <visual>
         <origin xyz="0 0 ${base_z/2.0 - 0.004}" rpy="0 0 0"/>
@@ -36,5 +36,5 @@
         <material name="grey"/>
       </visual>
-      <!-- Layer 1 – Battery (bottom, tallest) -->
+      <!-- Battery layer -->
       <visual>
         <origin xyz="0 0 ${-base_z/2.0 + 0.0175}" rpy="0 0 0"/>
@@ -42,5 +42,5 @@
         <material name="black"/>
       </visual>
-      <!-- Layer 2 – Motor Drivers -->
+      <!-- Motor driver layer -->
       <visual>
         <origin xyz="-0.04 0 ${-base_z/2.0 + 0.048}" rpy="0 0 0"/>
@@ -48,5 +48,5 @@
         <material name="dark_grey"/>
       </visual>
-      <!-- Layer 3 – Power distribution + ESP32 -->
+      <!-- Power + ESP32 layer -->
       <visual>
         <origin xyz="0 0 ${-base_z/2.0 + 0.068}" rpy="0 0 0"/>
@@ -54,5 +54,5 @@
         <material name="dark_grey"/>
       </visual>
-      <!-- Layer 4 – Raspberry Pi 5 (green PCB) -->
+      <!-- Raspberry Pi 5 PCB -->
       <visual>
         <origin xyz="-0.03 0.03 ${-base_z/2.0 + 0.088}" rpy="0 0 0"/>
@@ -60,5 +60,5 @@
         <material name="green"/>
       </visual>
-      <!-- Arm mount boss on top-centre -->
+      <!-- Arm mount boss -->
       <visual>
         <origin xyz="0.0 0.0 ${base_z/2.0 + 0.012}" rpy="0 0 0"/>
@@ -66,5 +66,4 @@
         <material name="black"/>
       </visual>
-      <!-- Collision uses the full bounding box only -->
       <collision>
         <origin xyz="0 0 0" rpy="0 0 0"/>
@@ -74,12 +73,53 @@
         <mass value="${base_mass}"/>
         <origin xyz="0 0 0" rpy="0 0 0"/>
-        <!-- Box inertia  I = (1/12) m (a² + b²) -->
         <inertia
-          ixx="${(1.0/12.0) * base_mass * (base_y*base_y + base_z*base_z)}"
-          iyy="${(1.0/12.0) * base_mass * (base_x*base_x + base_z*base_z)}"
-          izz="${(1.0/12.0) * base_mass * (base_x*base_x + base_y*base_y)}"
+          ixx="${(1.0/12.0)*base_mass*(base_y*base_y + base_z*base_z)}"
+          iyy="${(1.0/12.0)*base_mass*(base_x*base_x + base_z*base_z)}"
+          izz="${(1.0/12.0)*base_mass*(base_x*base_x + base_y*base_y)}"
           ixy="0" ixz="0" iyz="0"/>
       </inertial>
     </link>
+    <!-- ================================================================
+         GAZEBO — base_link surface
+         Low friction chassis body (it shouldn't drag on anything).
+         Gazebo Harmonic uses <gz> namespace for surface params.
+       ================================================================ -->
+    <gazebo reference="base_link">
+      <material>Gazebo/DarkGrey</material>
+      <surface>
+        <friction>
+          <ode>
+            <mu>0.3</mu>
+            <mu2>0.3</mu2>
+          </ode>
+        </friction>
+        <contact>
+          <ode>
+            <kp>1e6</kp>
+            <kd>100.0</kd>
+          </ode>
+        </contact>
+      </surface>
+    </gazebo>
+    <gazebo reference="base_footprint">
+      <material>Gazebo/Black</material>
+    </gazebo>
+    <!-- ================================================================
+         GAZEBO — ros2_control plugin
+         Loads the GazeboSimROS2ControlPlugin which drives all
+         hardware interfaces declared in arm.xacro and wheels.xacro.
+         Also spawns a JointStateBroadcaster automatically.
+       ================================================================ -->
+    <gazebo>
+      <plugin filename="gz_ros2_control-system"
+              name="gz_ros2_control::GazeboSimROS2ControlPlugin">
+        <!-- Path to the controllers YAML — adjust to your config dir -->
+        <parameters>$(find orion_description)/config/ros2_controllers.yaml</parameters>
+        <ros>
+          <remapping>~/robot_description:=/robot_description</remapping>
+        </ros>
+      </plugin>
+    </gazebo>
+    <!-- Clock bridging is handled in the launch file via ros_gz_bridge -->
   </xacro:macro>
 </robot>

File: orion_ws/src/orion_description/xacro/materials.xacro (robot description, xacro)
@@ -1,4 +1,12 @@
 <?xml version="1.0"?>
 <robot xmlns:xacro="http://www.ros.org/wiki/xacro">
+  <!-- ================================================================
+       ORION MATERIALS
+         RViz2 colours are set via <material> tags on each <visual>.
+         Gazebo ignores those tags — colours are set separately via
+         <gazebo reference="link_name"><material>...</material></gazebo>.
+         Use the xacro:gz_material macro below in each component file.
+       ================================================================ -->
+  <!-- ── RViz2 materials ─────────────────────────────────────────── -->
   <material name="grey">      <color rgba="0.60 0.60 0.60 1.0"/></material>
   <material name="dark_grey"> <color rgba="0.25 0.25 0.25 1.0"/></material>
@@ -10,3 +18,10 @@
   <material name="orange">    <color rgba="1.00 0.45 0.00 1.0"/></material>
   <material name="yellow">    <color rgba="1.00 0.85 0.00 1.0"/></material>
+  <!-- ── Gazebo/Ogre material helper ────────────────────────────── -->
+  <!-- Usage: <xacro:gz_material link="my_link" gz_mat="Gazebo/Grey"/> -->
+  <xacro:macro name="gz_material" params="link gz_mat">
+    <gazebo reference="${link}">
+      <material>${gz_mat}</material>
+    </gazebo>
+  </xacro:macro>
 </robot>
