Commit message: Clean ORION ROS2 workspace (remove vscode + build artifacts)

File: orion_ws/src/orion_description/xacro/orion.xacro (robot description, xacro)
@@ -1,5 +1,20 @@
 <?xml version="1.0"?>
 <robot name="orion" xmlns:xacro="http://www.ros.org/wiki/xacro">
-  <!-- Materials defined ONCE here — do NOT include in sub-files -->
+  <!-- ================================================================
+       ORION  —  Top-level xacro (Gazebo Harmonic + ROS2 Jazzy)
+       Plugin summary (all declared in sub-files):
+         base.xacro    → gz_ros2_control (arm joint control)
+         wheels.xacro  → gz-sim-mecanum-drive-system (/cmd_vel → /odom)
+         sensors.xacro → gpu_lidar sensor on lidar_link (/scan)
+         HERE          → gz-sim-sensors-system (needed to activate sensors)
+                       → gz-sim-imu-system     (future IMU support)
+       TODO: Bridge topics: (add to gazebo.launch.py)
+         /scan         → sensor_msgs/msg/LaserScan
+         /odom         → nav_msgs/msg/Odometry
+         /cmd_vel      → geometry_msgs/msg/Twist
+         /tf           → tf2_msgs/msg/TFMessage
+         /clock        → rosgraph_msgs/msg/Clock
+       ================================================================ -->
+  <!--Import-->
   <xacro:include filename="$(find orion_description)/xacro/materials.xacro"/>
   <xacro:include filename="$(find orion_description)/xacro/base.xacro"/>
@@ -7,7 +22,20 @@
   <xacro:include filename="$(find orion_description)/xacro/sensors.xacro"/>
   <xacro:include filename="$(find orion_description)/xacro/arm.xacro"/>
+  <!--Instantiate-->
   <xacro:base/>
   <xacro:wheels/>
   <xacro:sensors/>
   <xacro:arm/>
+  <!--GZ Sensor activation system-->
+  <gazebo>
+    <plugin filename="gz-sim-sensors-system"
+            name="gz::sim::systems::Sensors">
+      <render_engine>ogre2</render_engine>
+    </plugin>
+  </gazebo>
+  <gazebo>
+    <plugin filename="gz-sim-imu-system"
+            name="gz::sim::systems::Imu"/>
+  </gazebo>
+  <!-- gz_ros2_control is loaded once in base.xacro -->
 </robot>

File: orion_ws/src/orion_description/xacro/sensors.xacro (robot description, xacro)
@@ -2,15 +2,14 @@
 <robot xmlns:xacro="http://www.ros.org/wiki/xacro">
   <xacro:property name="base_z"    value="0.105"/>
-  <!-- Mast -->
   <xacro:property name="mast_r"    value="0.010"/>
   <xacro:property name="mast_h"    value="0.360"/>
-  <xacro:property name="mast_x"    value="-0.100"/>   <!-- rear of base -->
+  <xacro:property name="mast_x"    value="-0.100"/>
   <xacro:property name="mast_y"    value="0.000"/>
-  <!-- LiDAR (RPLIDAR A2 profile) -->
   <xacro:property name="lidar_r"   value="0.038"/>
   <xacro:property name="lidar_h"   value="0.041"/>
   <xacro:property name="lidar_m"   value="0.185"/>
+  <xacro:property name="imu_xyz"   value="0.02"/>
   <xacro:macro name="sensors">
-    <!-- ── Mast link ─────────────────────────────────────────────── -->
+    <!--Mast-->
     <link name="lidar_mast_link">
       <visual>
@@ -33,4 +32,5 @@
       </inertial>
     </link>
+    <!--LiDAR to Mast Joint-->
     <joint name="lidar_mast_joint" type="fixed">
       <parent link="base_link"/>
@@ -38,7 +38,6 @@
       <origin xyz="${mast_x} ${mast_y} ${base_z/2.0}" rpy="0 0 0"/>
     </joint>
-    <!-- ── LiDAR link ─────────────────────────────────────────────── -->
+    <!--LiDAR Link-->
     <link name="lidar_link">
-      <!-- Body -->
       <visual>
         <origin xyz="0 0 ${lidar_h/2.0}" rpy="0 0 0"/>
@@ -46,5 +45,4 @@
         <material name="black"/>
       </visual>
-      <!-- Rotating scan head -->
       <visual>
         <origin xyz="0 0 ${lidar_h + 0.009}" rpy="0 0 0"/>
@@ -52,5 +50,4 @@
         <material name="dark_grey"/>
       </visual>
-      <!-- Indicator LED -->
       <visual>
         <origin xyz="${lidar_r - 0.003} 0 ${lidar_h/2.0}" rpy="0 0 0"/>
@@ -72,5 +69,5 @@
       </inertial>
     </link>
-    <!-- Mast top → LiDAR -->
+    <!--LiDAR Joint-->
     <joint name="lidar_joint" type="fixed">
       <parent link="lidar_mast_link"/>
@@ -78,4 +75,88 @@
       <origin xyz="0 0 ${mast_h}" rpy="0 0 0"/>
     </joint>
+    <!--LiDAR GZ Plugin-->
+    <gazebo reference="lidar_link">
+      <material>Gazebo/Black</material>
+      <sensor name="lidar_sensor" type="gpu_lidar">
+        <pose>0 0 ${lidar_h/2.0} 0 0 0</pose>
+        <topic>/scan</topic>
+        <gz_frame_id>lidar_link</gz_frame_id>
+        <update_rate>10</update_rate>
+        <visualize>false</visualize>
+        <always_on>true</always_on>
+        <lidar>
+          <scan>
+            <horizontal>
+              <samples>360</samples>
+              <resolution>1</resolution>
+              <min_angle>-3.14159265</min_angle>
+              <max_angle> 3.14159265</max_angle>
+            </horizontal>
+            <vertical>
+              <samples>1</samples>
+              <resolution>1</resolution>
+              <min_angle>0</min_angle>
+              <max_angle>0</max_angle>
+            </vertical>
+          </scan>
+          <range>
+            <min>0.15</min>
+            <max>12.0</max>
+            <resolution>0.01</resolution>
+          </range>
+          <noise>
+            <type>gaussian</type>
+            <mean>0.0</mean>
+            <stddev>0.005</stddev>
+          </noise>
+        </lidar>
+      </sensor>
+    </gazebo>
+    <!-- Mast colour -->
+    <gazebo reference="lidar_mast_link">
+      <material>Gazebo/DarkGrey</material>
+    </gazebo>
+    <!--IMU Link-->
+    <link name="imu_link">
+      <visual>
+        <origin xyz="0 0 0"/>
+        <geometry>
+          <box size="${imu_xyz} ${imu_xyz} ${imu_xyz}"/>
+        </geometry>
+      </visual>
+      <inertial>
+        <mass value="0.05"/>
+        <origin xyz="0 0 0"/>
+        <inertia ixx="0.001" iyy="0.001" izz="0.001"
+                ixy="0" ixz="0" iyz="0"/>
+      </inertial>
+    </link>
+    <!--IMU Joint-->
+    <joint name="imu_joint" type="fixed">
+      <parent link="base_link"/>
+      <child link="imu_link"/>
+      <origin xyz="0 0 ${base_z}" rpy="0 0 0"/>
+    </joint>
+    <!--IMU Gz plugin-->
+    <gazebo reference="imu_link">
+      <sensor name="imu_sensor" type="imu">
+        <always_on>true</always_on>
+        <update_rate>100</update_rate>
+        <topic>/imu/data</topic>
+        <gz_frame_id>imu_link</gz_frame_id>
+        <imu>
+          <angular_velocity>
+            <x><noise type="gaussian" mean="0" stddev="0.001"/></x>
+            <y><noise type="gaussian" mean="0" stddev="0.001"/></y>
+            <z><noise type="gaussian" mean="0" stddev="0.001"/></z>
+          </angular_velocity>
+          <linear_acceleration>
+            <x><noise type="gaussian" mean="0" stddev="0.01"/></x>
+            <y><noise type="gaussian" mean="0" stddev="0.01"/></y>
+            <z><noise type="gaussian" mean="0" stddev="0.01"/></z>
+          </linear_acceleration>
+        </imu>
+      </sensor>
+    </gazebo>
   </xacro:macro>
 </robot>

File: orion_ws/src/orion_description/xacro/wheels.xacro (robot description, xacro)
@@ -2,8 +2,12 @@
 <robot xmlns:xacro="http://www.ros.org/wiki/xacro">
   <!-- ================================================================
-       ORION MECANUM WHEELS  —  4-wheel omnidirectional drive
-         wheel_radius : 50 mm  (standard 100 mm diameter mecanum)
-         wheel_width  : 40 mm
-         Positioned at four corners of the 280 × 320 mm chassis
+       ORION MECANUM WHEELS  —  Gazebo-ready
+         Gazebo additions:
+           • Per-wheel <gazebo reference> with mecanum-style friction:
+               mu  (longitudinal, along wheel spin) = high  ≈ 1.0
+               mu2 (lateral, across rollers)        = low   ≈ 0.1
+               fdir1 set to the wheel's forward direction in its frame
+           • MecanumDrive plugin (gz-sim-mecanum-drive-system)
+             Publishes odometry and subscribes to /cmd_vel (Twist).
        ================================================================ -->
   <xacro:property name="wheel_radius"  value="0.050"/>
@@ -11,31 +15,23 @@
   <xacro:property name="wheel_mass"    value="0.300"/>
   <xacro:property name="base_z"        value="0.105"/>
-  <!-- Wheel centre offsets relative to base_link origin (centre of chassis) -->
-  <xacro:property name="wheel_x_off"  value="0.095"/>   <!-- ±95 mm front/rear  -->
-  <xacro:property name="wheel_y_off"  value="0.130"/>   <!-- ±130 mm left/right -->
-  <!-- Wheel centres flush with bottom of chassis -->
+  <xacro:property name="wheel_x_off"  value="0.095"/>
+  <xacro:property name="wheel_y_off"  value="0.130"/>
   <xacro:property name="wheel_z_off"  value="${-base_z / 2.0}"/>
-  <!-- Roller stripe count (visual only) -->
-  <xacro:property name="roller_count"  value="9"/>
   <!-- ── Single mecanum wheel ── -->
-  <xacro:macro name="mecanum_wheel" params="name x_sign y_sign roller_sign">
+  <xacro:macro name="mecanum_wheel" params="name x_sign y_sign">
     <link name="${name}_wheel_link">
-      <!-- Main tyre body -->
+      <!-- Tyre -->
       <visual>
         <origin xyz="0 0 0" rpy="${pi/2} 0 0"/>
-        <geometry>
-          <cylinder radius="${wheel_radius}" length="${wheel_width}"/>
-        </geometry>
+        <geometry><cylinder radius="${wheel_radius}" length="${wheel_width}"/></geometry>
         <material name="black"/>
       </visual>
-      <!-- Hub (lighter centre) -->
+      <!-- Hub -->
       <visual>
         <origin xyz="0 0 0" rpy="${pi/2} 0 0"/>
-        <geometry>
-          <cylinder radius="${wheel_radius * 0.38}" length="${wheel_width + 0.002}"/>
-        </geometry>
+        <geometry><cylinder radius="${wheel_radius * 0.38}" length="${wheel_width + 0.002}"/></geometry>
         <material name="grey"/>
       </visual>
-      <!-- Axle stub (left side) -->
+      <!-- Axle stubs -->
       <visual>
         <origin xyz="0  ${wheel_width/2.0 + 0.006} 0" rpy="${pi/2} 0 0"/>
@@ -43,5 +39,4 @@
         <material name="dark_grey"/>
       </visual>
-      <!-- Axle stub (right side) -->
       <visual>
         <origin xyz="0 ${-(wheel_width/2.0 + 0.006)} 0" rpy="${pi/2} 0 0"/>
@@ -49,21 +44,15 @@
         <material name="dark_grey"/>
       </visual>
-      <!-- Collision is a simple cylinder -->
       <collision>
         <origin xyz="0 0 0" rpy="${pi/2} 0 0"/>
-        <geometry>
-          <cylinder radius="${wheel_radius}" length="${wheel_width}"/>
-        </geometry>
+        <geometry><cylinder radius="${wheel_radius}" length="${wheel_width}"/></geometry>
       </collision>
-      <!-- Cylinder inertia about Y (spin axis):
-             Ixx = Izz = (1/12) m (3r² + h²)      (h = wheel_width here)
-             Iyy         = (1/2) m r²   ← spin axis -->
       <inertial>
         <mass value="${wheel_mass}"/>
         <origin xyz="0 0 0" rpy="0 0 0"/>
         <inertia
-          ixx="${(1.0/12.0) * wheel_mass * (3.0*wheel_radius*wheel_radius + wheel_width*wheel_width)}"
-          iyy="${0.5         * wheel_mass * wheel_radius * wheel_radius}"
-          izz="${(1.0/12.0) * wheel_mass * (3.0*wheel_radius*wheel_radius + wheel_width*wheel_width)}"
+          ixx="${(1.0/12.0)*wheel_mass*(3.0*wheel_radius*wheel_radius + wheel_width*wheel_width)}"
+          iyy="${0.5*wheel_mass*wheel_radius*wheel_radius}"
+          izz="${(1.0/12.0)*wheel_mass*(3.0*wheel_radius*wheel_radius + wheel_width*wheel_width)}"
           ixy="0" ixz="0" iyz="0"/>
       </inertial>
@@ -72,23 +61,83 @@
       <parent link="base_link"/>
       <child  link="${name}_wheel_link"/>
-      <origin xyz="${x_sign * wheel_x_off}
-                   ${y_sign * wheel_y_off}
-                   ${wheel_z_off}"
+      <origin xyz="${x_sign * wheel_x_off} ${y_sign * wheel_y_off} ${wheel_z_off}"
               rpy="0 0 0"/>
-      <!-- Mecanum wheels spin about the Y axis -->
       <axis xyz="0 1 0"/>
       <dynamics damping="0.01" friction="0.05"/>
     </joint>
+    <!-- ── Gazebo wheel colour + mecanum friction ── -->
+    <gazebo reference="${name}_wheel_link">
+      <material>Gazebo/Black</material>
+      <collision>
+        <surface>
+          <friction>
+            <ode>
+              <!-- High longitudinal grip, low lateral slip = mecanum roller effect -->
+              <mu>1.0</mu>
+              <mu2>0.1</mu2>
+              <!-- fdir1 in link frame: wheel rolls along X, rotated pi/2 about X
+                   so forward direction maps to Z in the collision frame -->
+              <fdir1>0 0 1</fdir1>
+              <slip1>0.0</slip1>
+              <slip2>0.05</slip2>
+            </ode>
+          </friction>
+          <contact>
+            <ode>
+              <kp>1e6</kp>
+              <kd>1.0</kd>
+              <min_depth>0.001</min_depth>
+              <max_vel>0.1</max_vel>
+            </ode>
+          </contact>
+        </surface>
+      </collision>
+    </gazebo>
+    <!-- ── ros2_control hardware interface for this wheel ── -->
+    <!-- Declared here so each wheel macro registers its own interface.
+         gz_ros2_control will pick these up automatically.             -->
   </xacro:macro>
-  <!-- ================================================================
-       Four wheel instances
-         roller_sign: +1 = rollers at +45° (FL, RR)
-                      -1 = rollers at -45° (FR, RL)
-       ================================================================ -->
+  <!-- ── Four wheel instances ── -->
   <xacro:macro name="wheels">
-    <xacro:mecanum_wheel name="front_left"  x_sign=" 1" y_sign=" 1" roller_sign=" 1"/>
-    <xacro:mecanum_wheel name="front_right" x_sign=" 1" y_sign="-1" roller_sign="-1"/>
-    <xacro:mecanum_wheel name="rear_left"   x_sign="-1" y_sign=" 1" roller_sign="-1"/>
-    <xacro:mecanum_wheel name="rear_right"  x_sign="-1" y_sign="-1" roller_sign=" 1"/>
+    <xacro:mecanum_wheel name="front_left"  x_sign=" 1" y_sign=" 1"/>
+    <xacro:mecanum_wheel name="front_right" x_sign=" 1" y_sign="-1"/>
+    <xacro:mecanum_wheel name="rear_left"   x_sign="-1" y_sign=" 1"/>
+    <xacro:mecanum_wheel name="rear_right"  x_sign="-1" y_sign="-1"/>
+    <!-- ==============================================================
+         GAZEBO — MecanumDrive plugin
+           Subscribes : /cmd_vel  (geometry_msgs/Twist)
+           Publishes  : /odom     (nav_msgs/Odometry)
+                        /tf       (odom → base_footprint)
+         Wheel names must match joint names exactly.
+         front_left  / front_right rollers are at +45° (X pattern),
+         rear_left   / rear_right  rollers are at -45°.
+         The plugin uses these signs internally.
+         ============================================================== -->
+    <gazebo>
+      <plugin filename="gz-sim-mecanum-drive-system"
+              name="gz::sim::systems::MecanumDrive">
+        <!-- Wheel joints -->
+        <front_left_joint>front_left_wheel_joint</front_left_joint>
+        <front_right_joint>front_right_wheel_joint</front_right_joint>
+        <rear_left_joint>rear_left_wheel_joint</rear_left_joint>
+        <rear_right_joint>rear_right_wheel_joint</rear_right_joint>
+        <!-- Physical parameters  (must match xacro properties above) -->
+        <wheel_separation>${wheel_y_off * 2.0}</wheel_separation>
+        <wheelbase>${wheel_x_off * 2.0}</wheelbase>
+        <wheel_radius>${wheel_radius}</wheel_radius>
+        <!-- ROS topics -->
+        <topic>/cmd_vel</topic>
+        <odom_topic>/odom</odom_topic>
+        <tf_topic>/tf</tf_topic>
+        <frame_id>odom</frame_id>
+        <child_frame_id>base_footprint</child_frame_id>
+        <!-- Publish odometry TF -->
+        <publish_odom>true</publish_odom>
+        <publish_odom_tf>true</publish_odom_tf>
+        <!-- Max velocity limits -->
+        <max_linear_velocity>1.0</max_linear_velocity>
+        <max_angular_velocity>2.0</max_angular_velocity>
+      </plugin>
+    </gazebo>
   </xacro:macro>
 </robot>
