Commit message: Total changes: Added a mecanum_ik_node.py to handle the messages between /cmd_vel and /wheel_velocity/controller/commands. BUG: lin x vel and ang z vel work as expected, but when lin y vel is passed a value (using /cmd_vel) the robot spins in place. Also changed ros2_controllers.yaml to include a wheel_velocity controller. Continuous changes to wheels.xacro (chagning friction coeffs/plugins all in hope to fix the mentioned bug - VAIN). Added a bridge.yaml file to handle ros_gz_bridge.

File: orion_ws/src/orion_description/urdf/orion.urdf (robot description, URDF)
Before this commit: robot orion, 17 links, 16 joints
Links:
- removed link base_footprint
- link front_left_wheel_link: geometry collision cylinder length=0.04 radius=0.05; visual box size=0.002 0.04 0.1
- link front_right_wheel_link: geometry collision cylinder length=0.04 radius=0.05; visual box size=0.002 0.04 0.1
- link rear_left_wheel_link: geometry collision cylinder length=0.04 radius=0.05; visual box size=0.002 0.04 0.1
- link rear_right_wheel_link: geometry collision cylinder length=0.04 radius=0.05; visual box size=0.002 0.04 0.1
Joints:
- removed joint base_footprint_joint

File: orion_ws/src/orion_description/xacro/base.xacro (robot description, xacro)
@@ -1,26 +1,10 @@
 <?xml version="1.0"?>
 <robot xmlns:xacro="http://www.ros.org/wiki/xacro">
-  <!-- ================================================================
-       ORION BASE  —  Gazebo-ready
-         Gazebo additions:
-           • <gazebo reference> surface/friction for base_link
-           • Gazebo material colours
-           • gz_ros2_control + JointStateBroadcaster plugin
-       ================================================================ -->
-  <xacro:property name="base_x"     value="0.280"/>
-  <xacro:property name="base_y"     value="0.320"/>
-  <xacro:property name="base_z"     value="0.105"/>
-  <xacro:property name="base_mass"  value="3.5"/>
+  <xacro:property name="base_x"      value="0.280"/>
+  <xacro:property name="base_y"      value="0.320"/>
+  <xacro:property name="base_z"      value="0.105"/>
+  <xacro:property name="base_mass"   value="3.5"/>
   <xacro:property name="wheel_radius" value="0.050"/>
-  <xacro:property name="base_link_z"  value="${wheel_radius + base_z / 2.0}"/>
   <xacro:macro name="base">
-    <!-- ── Ground reference frame ──────────────────────────────── -->
-    <link name="base_footprint"/>
-    <joint name="base_footprint_joint" type="fixed">
-      <parent link="base_footprint"/>
-      <child  link="base_link"/>
-      <origin xyz="0 0 ${base_link_z}" rpy="0 0 0"/>
-    </joint>
-    <!-- ── Main chassis ─────────────────────────────────────────── -->
     <link name="base_link">
       <!-- Outer shell -->
@@ -80,9 +64,4 @@
       </inertial>
     </link>
-    <!-- ================================================================
-         GAZEBO — base_link surface
-         Low friction chassis body (it shouldn't drag on anything).
-         Gazebo Harmonic uses <gz> namespace for surface params.
-       ================================================================ -->
     <gazebo reference="base_link">
       <material>Gazebo/DarkGrey</material>
@@ -102,17 +81,7 @@
       </surface>
     </gazebo>
-    <gazebo reference="base_footprint">
-      <material>Gazebo/Black</material>
-    </gazebo>
-    <!-- ================================================================
-         GAZEBO — ros2_control plugin
-         Loads the GazeboSimROS2ControlPlugin which drives all
-         hardware interfaces declared in arm.xacro and wheels.xacro.
-         Also spawns a JointStateBroadcaster automatically.
-       ================================================================ -->
     <gazebo>
       <plugin filename="gz_ros2_control-system"
               name="gz_ros2_control::GazeboSimROS2ControlPlugin">
-        <!-- Path to the controllers YAML — adjust to your config dir -->
         <parameters>$(find orion_description)/config/ros2_controllers.yaml</parameters>
         <ros>
@@ -121,5 +90,4 @@
       </plugin>
     </gazebo>
-    <!-- Clock bridging is handled in the launch file via ros_gz_bridge -->
   </xacro:macro>
 </robot>

File: orion_ws/src/orion_description/xacro/materials.xacro (robot description, xacro)
@@ -1,11 +1,4 @@
 <?xml version="1.0"?>
 <robot xmlns:xacro="http://www.ros.org/wiki/xacro">
-  <!-- ================================================================
-       ORION MATERIALS
-         RViz2 colours are set via <material> tags on each <visual>.
-         Gazebo ignores those tags — colours are set separately via
-         <gazebo reference="link_name"><material>...</material></gazebo>.
-         Use the xacro:gz_material macro below in each component file.
-       ================================================================ -->
   <!-- ── RViz2 materials ─────────────────────────────────────────── -->
   <material name="grey">      <color rgba="0.60 0.60 0.60 1.0"/></material>
@@ -18,6 +11,4 @@
   <material name="orange">    <color rgba="1.00 0.45 0.00 1.0"/></material>
   <material name="yellow">    <color rgba="1.00 0.85 0.00 1.0"/></material>
-  <!-- ── Gazebo/Ogre material helper ────────────────────────────── -->
-  <!-- Usage: <xacro:gz_material link="my_link" gz_mat="Gazebo/Grey"/> -->
   <xacro:macro name="gz_material" params="link gz_mat">
     <gazebo reference="${link}">

File: orion_ws/src/orion_description/xacro/orion.xacro (robot description, xacro)
@@ -1,19 +1,4 @@
 <?xml version="1.0"?>
 <robot name="orion" xmlns:xacro="http://www.ros.org/wiki/xacro">
-  <!-- ================================================================
-       ORION  —  Top-level xacro (Gazebo Harmonic + ROS2 Jazzy)
-       Plugin summary (all declared in sub-files):
-         base.xacro    → gz_ros2_control (arm joint control)
-         wheels.xacro  → gz-sim-mecanum-drive-system (/cmd_vel → /odom)
-         sensors.xacro → gpu_lidar sensor on lidar_link (/scan)
-         HERE          → gz-sim-sensors-system (needed to activate sensors)
-                       → gz-sim-imu-system     (future IMU support)
-       TODO: Bridge topics: (add to gazebo.launch.py)
-         /scan         → sensor_msgs/msg/LaserScan
-         /odom         → nav_msgs/msg/Odometry
-         /cmd_vel      → geometry_msgs/msg/Twist
-         /tf           → tf2_msgs/msg/TFMessage
-         /clock        → rosgraph_msgs/msg/Clock
-       ================================================================ -->
   <!--Import-->
   <xacro:include filename="$(find orion_description)/xacro/materials.xacro"/>
@@ -38,4 +23,3 @@
             name="gz::sim::systems::Imu"/>
   </gazebo>
-  <!-- gz_ros2_control is loaded once in base.xacro -->
 </robot>

File: orion_ws/src/orion_description/xacro/wheels.xacro (robot description, xacro)
@@ -1,25 +1,13 @@
 <?xml version="1.0"?>
 <robot xmlns:xacro="http://www.ros.org/wiki/xacro">
-  <!-- ================================================================
-       ORION MECANUM WHEELS  —  Gazebo-ready
-         Gazebo additions:
-           • Per-wheel <gazebo reference> with mecanum-style friction:
-               mu  (longitudinal, along wheel spin) = high  ≈ 1.0
-               mu2 (lateral, across rollers)        = low   ≈ 0.1
-               fdir1 set to the wheel's forward direction in its frame
-           • MecanumDrive plugin (gz-sim-mecanum-drive-system)
-             Publishes odometry and subscribes to /cmd_vel (Twist).
-       ================================================================ -->
-  <xacro:property name="wheel_radius"  value="0.050"/>
-  <xacro:property name="wheel_width"   value="0.040"/>
-  <xacro:property name="wheel_mass"    value="0.300"/>
-  <xacro:property name="base_z"        value="0.105"/>
+  <xacro:property name="wheel_radius" value="0.05"/>
+  <xacro:property name="wheel_width"  value="0.04"/>
+  <xacro:property name="wheel_mass"   value="0.3"/>
+  <xacro:property name="base_z"       value="0.105"/>
   <xacro:property name="wheel_x_off"  value="0.095"/>
-  <xacro:property name="wheel_y_off"  value="0.130"/>
-  <xacro:property name="wheel_z_off"  value="${-base_z / 2.0}"/>
-  <!-- ── Single mecanum wheel ── -->
-  <xacro:macro name="mecanum_wheel" params="name x_sign y_sign">
+  <xacro:property name="wheel_y_off"  value="0.13"/>
+  <xacro:property name="wheel_z_off"  value="${-base_z/2.0}"/>
+  <xacro:macro name="mecanum_wheel" params="name x_sign y_sign fdir1_y">
     <link name="${name}_wheel_link">
-      <!-- Tyre -->
       <visual>
         <origin xyz="0 0 0" rpy="${pi/2} 0 0"/>
@@ -27,20 +15,8 @@
         <material name="black"/>
       </visual>
-      <!-- Hub -->
       <visual>
         <origin xyz="0 0 0" rpy="${pi/2} 0 0"/>
-        <geometry><cylinder radius="${wheel_radius * 0.38}" length="${wheel_width + 0.002}"/></geometry>
+        <geometry><cylinder radius="${wheel_radius*0.38}" length="${wheel_width+0.002}"/></geometry>
         <material name="grey"/>
-      </visual>
-      <!-- Axle stubs -->
-      <visual>
-        <origin xyz="0  ${wheel_width/2.0 + 0.006} 0" rpy="${pi/2} 0 0"/>
-        <geometry><cylinder radius="0.008" length="0.012"/></geometry>
-        <material name="dark_grey"/>
-      </visual>
-      <visual>
-        <origin xyz="0 ${-(wheel_width/2.0 + 0.006)} 0" rpy="${pi/2} 0 0"/>
-        <geometry><cylinder radius="0.008" length="0.012"/></geometry>
-        <material name="dark_grey"/>
       </visual>
       <collision>
@@ -50,9 +26,9 @@
       <inertial>
         <mass value="${wheel_mass}"/>
-        <origin xyz="0 0 0" rpy="0 0 0"/>
+        <origin xyz="0 0 0"/>
         <inertia
-          ixx="${(1.0/12.0)*wheel_mass*(3.0*wheel_radius*wheel_radius + wheel_width*wheel_width)}"
+          ixx="${(1.0/12.0)*wheel_mass*(3*wheel_radius*wheel_radius+wheel_width*wheel_width)}"
           iyy="${0.5*wheel_mass*wheel_radius*wheel_radius}"
-          izz="${(1.0/12.0)*wheel_mass*(3.0*wheel_radius*wheel_radius + wheel_width*wheel_width)}"
+          izz="${(1.0/12.0)*wheel_mass*(3*wheel_radius*wheel_radius+wheel_width*wheel_width)}"
           ixy="0" ixz="0" iyz="0"/>
       </inertial>
@@ -61,10 +37,8 @@
       <parent link="base_link"/>
       <child  link="${name}_wheel_link"/>
-      <origin xyz="${x_sign * wheel_x_off} ${y_sign * wheel_y_off} ${wheel_z_off}"
-              rpy="0 0 0"/>
+      <origin xyz="${x_sign*wheel_x_off} ${y_sign*wheel_y_off} ${wheel_z_off}" rpy="0 0 0"/>
       <axis xyz="0 1 0"/>
-      <dynamics damping="0.01" friction="0.05"/>
+      <dynamics damping="0.01" friction="0.01"/>
     </joint>
-    <!-- ── Gazebo wheel colour + mecanum friction ── -->
     <gazebo reference="${name}_wheel_link">
       <material>Gazebo/Black</material>
@@ -73,12 +47,7 @@
           <friction>
             <ode>
-              <!-- High longitudinal grip, low lateral slip = mecanum roller effect -->
               <mu>1.0</mu>
               <mu2>0.1</mu2>
-              <!-- fdir1 in link frame: wheel rolls along X, rotated pi/2 about X
-                   so forward direction maps to Z in the collision frame -->
-              <fdir1>0 0 1</fdir1>
-              <slip1>0.0</slip1>
-              <slip2>0.05</slip2>
+              <fdir1>0.7071 ${fdir1_y} 0</fdir1>
             </ode>
           </friction>
@@ -94,50 +63,38 @@
       </collision>
     </gazebo>
-    <!-- ── ros2_control hardware interface for this wheel ── -->
-    <!-- Declared here so each wheel macro registers its own interface.
-         gz_ros2_control will pick these up automatically.             -->
   </xacro:macro>
-  <!-- ── Four wheel instances ── -->
   <xacro:macro name="wheels">
-    <xacro:mecanum_wheel name="front_left"  x_sign=" 1" y_sign=" 1"/>
-    <xacro:mecanum_wheel name="front_right" x_sign=" 1" y_sign="-1"/>
-    <xacro:mecanum_wheel name="rear_left"   x_sign="-1" y_sign=" 1"/>
-    <xacro:mecanum_wheel name="rear_right"  x_sign="-1" y_sign="-1"/>
-    <!-- ==============================================================
-         GAZEBO — MecanumDrive plugin
-           Subscribes : /cmd_vel  (geometry_msgs/Twist)
-           Publishes  : /odom     (nav_msgs/Odometry)
-                        /tf       (odom → base_footprint)
-         Wheel names must match joint names exactly.
-         front_left  / front_right rollers are at +45° (X pattern),
-         rear_left   / rear_right  rollers are at -45°.
-         The plugin uses these signs internally.
-         ============================================================== -->
-    <gazebo>
-      <plugin filename="gz-sim-mecanum-drive-system"
-              name="gz::sim::systems::MecanumDrive">
-        <!-- Wheel joints -->
-        <front_left_joint>front_left_wheel_joint</front_left_joint>
-        <front_right_joint>front_right_wheel_joint</front_right_joint>
-        <rear_left_joint>rear_left_wheel_joint</rear_left_joint>
-        <rear_right_joint>rear_right_wheel_joint</rear_right_joint>
-        <!-- Physical parameters  (must match xacro properties above) -->
-        <wheel_separation>${wheel_y_off * 2.0}</wheel_separation>
-        <wheelbase>${wheel_x_off * 2.0}</wheelbase>
-        <wheel_radius>${wheel_radius}</wheel_radius>
-        <!-- ROS topics -->
-        <topic>/cmd_vel</topic>
-        <odom_topic>/odom</odom_topic>
-        <tf_topic>/tf</tf_topic>
-        <frame_id>odom</frame_id>
-        <child_frame_id>base_footprint</child_frame_id>
-        <!-- Publish odometry TF -->
-        <publish_odom>true</publish_odom>
-        <publish_odom_tf>true</publish_odom_tf>
-        <!-- Max velocity limits -->
-        <max_linear_velocity>1.0</max_linear_velocity>
-        <max_angular_velocity>2.0</max_angular_velocity>
-      </plugin>
-    </gazebo>
+    <!-- Signs have NO leading spaces: "1" not " 1", "-1" not "-1" -->
+    <xacro:mecanum_wheel name="front_left"  x_sign="1"  y_sign="1"  fdir1_y="-0.7071"/>
+    <xacro:mecanum_wheel name="front_right" x_sign="1"  y_sign="-1" fdir1_y="0.7071"/>
+    <xacro:mecanum_wheel name="rear_left"   x_sign="-1" y_sign="1"  fdir1_y="0.7071"/>
+    <xacro:mecanum_wheel name="rear_right"  x_sign="-1" y_sign="-1" fdir1_y="-0.7071"/>
+    <!-- ros2_control block — all 4 wheels velocity-controlled via
+         forward_command_controller + mecanum_ik_node. -->
+    <ros2_control name="orion_base" type="system">
+      <hardware>
+        <plugin>gz_ros2_control/GazeboSimSystem</plugin>
+      </hardware>
+      <joint name="front_left_wheel_joint">
+        <command_interface name="velocity"/>
+        <state_interface name="position"/>
+        <state_interface name="velocity"/>
+      </joint>
+      <joint name="front_right_wheel_joint">
+        <command_interface name="velocity"/>
+        <state_interface name="position"/>
+        <state_interface name="velocity"/>
+      </joint>
+      <joint name="rear_left_wheel_joint">
+        <command_interface name="velocity"/>
+        <state_interface name="position"/>
+        <state_interface name="velocity"/>
+      </joint>
+      <joint name="rear_right_wheel_joint">
+        <command_interface name="velocity"/>
+        <state_interface name="position"/>
+        <state_interface name="velocity"/>
+      </joint>
+    </ros2_control>
   </xacro:macro>
 </robot>

Commit message: updated urdf

File: orion_ws/src/orion_description/urdf/orion.urdf (robot description, URDF)
Before this commit: robot orion, 16 links, 15 joints
Links:
- link front_left_wheel_link: geometry collision cylinder length=0.04 radius=0.05; visual cylinder length=0.04 radius=0.05
- link front_right_wheel_link: geometry collision cylinder length=0.04 radius=0.05; visual cylinder length=0.04 radius=0.05
- link rear_left_wheel_link: geometry collision cylinder length=0.04 radius=0.05; visual cylinder length=0.04 radius=0.05
- link rear_right_wheel_link: geometry collision cylinder length=0.04 radius=0.05; visual cylinder length=0.04 radius=0.05
