Commit message: Changes to mecanum drive system (added exec tags to package.xml, experimented with velocity and friction in wheel macro). Issue: linear x velocity and angular z velocity work perfectly, but linear y velocity doesn't strafe properly

File: orion_ws/src/orion_description/urdf/orion.urdf (robot description, URDF)
Before this commit: robot orion, 16 links, 15 joints
Links:
- link front_left_wheel_link: geometry collision sphere radius=0.05; visual cylinder length=0.04 radius=0.05
- link front_right_wheel_link: geometry collision sphere radius=0.05; visual cylinder length=0.04 radius=0.05
- link rear_left_wheel_link: geometry collision sphere radius=0.05; visual cylinder length=0.04 radius=0.05
- link rear_right_wheel_link: geometry collision sphere radius=0.05; visual cylinder length=0.04 radius=0.05
Joints:
- joint gripper_right_joint: axis 0 -1 0 -> 0 1 0; limit lower=0.0 upper=0.025 effort=5.0 velocity=0.10 -> lower=-0.025 upper=0.0 effort=5.0 velocity=0.10; mimic (none) -> joint=gripper_left_joint multiplier=-1 offset=0

File: orion_ws/src/orion_description/xacro/orion.xacro (robot description, xacro)
@@ -1,15 +1,7 @@
 <?xml version="1.0"?>
-<robot name="orion" xmlns:xacro="http://www.ros.org/wiki/xacro">
-  <!-- ================================================================
-       orion.xacro  –  single-file robot description
-       Sections:  1. Materials
-                  2. Properties
-                  3. Inertia helper macros  (arm)
-                  4. Base macro
-                  5. Wheels macro
-                  6. Sensors macro
-                  7. Arm macro
-                  8. Instantiation
-       ================================================================ -->
+<robot name="orion"
+       xmlns:xacro="http://www.ros.org/wiki/xacro"
+       xmlns:gz="http://gazebosim.org/schema">
+  <xacro:arg name="controllers_file" default="config/ros2_controllers.yaml"/>
   <!-- ── 1. MATERIALS ─────────────────────────────────────────────── -->
   <material name="grey">      <color rgba="0.60 0.60 0.60 1.0"/></material>
@@ -40,4 +32,7 @@
   <xacro:property name="wheel_y_off"  value="0.130"/>
   <xacro:property name="wheel_z_off"  value="${-base_z/2.0}"/>
+  <!-- Gazebo Harmonic mecanum: mu/mu2 anisotropic + fdir1 in base_link. -->
+  <xacro:property name="wheel_mu"  value="1.0"/>
+  <xacro:property name="wheel_mu2" value="0.0"/>
   <!-- Sensors -->
   <xacro:property name="mast_r"    value="0.010"/>
@@ -157,7 +152,23 @@
       </inertial>
     </link>
+    <!-- Low friction if the chassis box grazes the ground; high mu here blocks strafing. -->
+    <gazebo reference="base_link">
+      <collision>
+        <surface>
+          <friction>
+            <ode>
+              <mu>0.01</mu>
+              <mu2>0.01</mu2>
+            </ode>
+          </friction>
+        </surface>
+      </collision>
+    </gazebo>
     <gazebo>
-      <plugin filename="gz_ros2_control-system" name="gz_ros2_control::GazeboSimROS2ControlPlugin">
-        <parameters>$(find orion_description)/config/ros2_controllers.yaml</parameters>
+      <plugin filename="libgz_ros2_control-system.so"
+              name="gz_ros2_control::GazeboSimROS2ControlPlugin">
+        <parameters>$(arg controllers_file)</parameters>
+        <robot_param>robot_description</robot_param>
+        <robot_param_node>robot_state_publisher</robot_param_node>
       </plugin>
     </gazebo>
@@ -171,4 +182,5 @@
         <material name="black"/>
       </visual>
+      <!-- Hub detail -->
       <visual>
         <origin xyz="0 0 0" rpy="${pi/2} 0 0"/>
@@ -176,7 +188,8 @@
         <material name="grey"/>
       </visual>
-      <collision>
-        <origin xyz="0 0 0" rpy="${pi/2} 0 0"/>
-        <geometry><cylinder radius="${wheel_radius}" length="${wheel_width}"/></geometry>
+      <!-- Sphere contact (gz-sim mecanum demo) — symmetric patch, less arc drift than cylinder -->
+      <collision>
+        <origin xyz="0 0 0" rpy="0 0 0"/>
+        <geometry><sphere radius="${wheel_radius}"/></geometry>
       </collision>
       <inertial>
@@ -184,7 +197,7 @@
         <origin xyz="0 0 0"/>
         <inertia
-          ixx="${(1.0/12.0)*wheel_mass*(3*wheel_radius*wheel_radius+wheel_width*wheel_width)}"
-          iyy="${0.5*wheel_mass*wheel_radius*wheel_radius}"
-          izz="${(1.0/12.0)*wheel_mass*(3*wheel_radius*wheel_radius+wheel_width*wheel_width)}"
+          ixx="${0.4*wheel_mass*wheel_radius*wheel_radius}"
+          iyy="${0.4*wheel_mass*wheel_radius*wheel_radius}"
+          izz="${0.4*wheel_mass*wheel_radius*wheel_radius}"
           ixy="0" ixz="0" iyz="0"/>
       </inertial>
@@ -197,5 +210,4 @@
       <dynamics damping="0.01" friction="0.01"/>
     </joint>
-    <ros2_control name = ""
     <gazebo reference="${name}_wheel_link">
       <collision>
@@ -203,7 +215,7 @@
           <friction>
             <ode>
-              <mu>1.0</mu>
-              <mu2>0.1</mu2>
-              <fdir1>1 ${fdir1_y} 0 </fdir1>
+              <mu>${wheel_mu}</mu>
+              <mu2>${wheel_mu2}</mu2>
+              <fdir1 gz:expressed_in="base_link">1 ${fdir1_y} 0</fdir1>
             </ode>
           </friction>
@@ -220,5 +232,5 @@
   <!-- ── 6. SENSORS MACRO ──────────────────────────────────────────── -->
   <xacro:macro name="sensors">
-    <!-- Mast -->
+    <!-- LiDAR mast -->
     <link name="lidar_mast_link">
       <visual>
@@ -246,5 +258,5 @@
       <origin xyz="${mast_x} ${mast_y} ${base_z/2.0}" rpy="0 0 0"/>
     </joint>
-    <!-- LiDAR -->
+    <!-- LiDAR sensor link -->
     <link name="lidar_link">
       <visual>
@@ -282,4 +294,33 @@
       <origin xyz="0 0 ${mast_h}" rpy="0 0 0"/>
     </joint>
+    <gazebo reference="lidar_link">
+      <sensor name="lidar" type="gpu_lidar">
+        <topic>scan</topic>
+        <update_rate>10</update_rate>
+        <lidar>
+          <scan>
+            <horizontal>
+              <samples>360</samples>
+              <resolution>1</resolution>
+              <min_angle>-3.14159</min_angle>
+              <max_angle>3.14159</max_angle>
+            </horizontal>
+          </scan>
+          <range>
+            <min>0.12</min>
+            <max>12.0</max>
+            <resolution>0.01</resolution>
+          </range>
+          <noise>
+            <type>gaussian</type>
+            <mean>0.0</mean>
+            <stddev>0.01</stddev>
+          </noise>
+        </lidar>
+        <always_on>true</always_on>
+        <visualize>false</visualize>
+        <gz_frame_id>lidar_link</gz_frame_id>
+      </sensor>
+    </gazebo>
     <!-- IMU -->
     <link name="imu_link">
@@ -289,4 +330,5 @@
           <box size="${imu_xyz} ${imu_xyz} ${imu_xyz}"/>
         </geometry>
+        <material name="dark_grey"/>
       </visual>
       <inertial>
@@ -294,12 +336,32 @@
         <origin xyz="0 0 0"/>
         <inertia ixx="0.001" iyy="0.001" izz="0.001"
-                ixy="0" ixz="0" iyz="0"/>
+                 ixy="0" ixz="0" iyz="0"/>
       </inertial>
     </link>
     <joint name="imu_joint" type="fixed">
       <parent link="base_link"/>
-      <child link="imu_link"/>
+      <child  link="imu_link"/>
       <origin xyz="0 0 ${base_z}" rpy="0 0 0"/>
     </joint>
+    <gazebo reference="imu_link">
+      <sensor name="imu" type="imu">
+        <topic>imu/data</topic>
+        <update_rate>100</update_rate>
+        <always_on>true</always_on>
+        <imu>
+          <angular_velocity>
+            <x><noise type="gaussian"><mean>0</mean><stddev>0.009</stddev></noise></x>
+            <y><noise type="gaussian"><mean>0</mean><stddev>0.009</stddev></noise></y>
+            <z><noise type="gaussian"><mean>0</mean><stddev>0.009</stddev></noise></z>
+          </angular_velocity>
+          <linear_acceleration>
+            <x><noise type="gaussian"><mean>0</mean><stddev>0.021</stddev></noise></x>
+            <y><noise type="gaussian"><mean>0</mean><stddev>0.021</stddev></noise></y>
+            <z><noise type="gaussian"><mean>0</mean><stddev>0.021</stddev></noise></z>
+          </linear_acceleration>
+        </imu>
+        <gz_frame_id>imu_link</gz_frame_id>
+      </sensor>
+    </gazebo>
   </xacro:macro>
   <!-- ── 7. ARM MACRO ──────────────────────────────────────────────── -->
@@ -423,5 +485,5 @@
       <origin xyz="${hand_l} 0 0" rpy="0 0 0"/>
     </joint>
-    <!-- Left gripper finger -->
+    <!-- Left gripper finger — ACTIVE joint, commanded by gripper_controller -->
     <link name="gripper_left_link">
       <visual>
@@ -445,5 +507,4 @@
       <dynamics damping="0.01" friction="0.01"/>
     </joint>
-    <!-- Right gripper finger -->
     <link name="gripper_right_link">
       <visual>
@@ -461,11 +522,12 @@
     <joint name="gripper_right_joint" type="prismatic">
       <parent link="gripper_base_link"/>
-      <child link="gripper_right_link"/>
+      <child  link="gripper_right_link"/>
       <origin xyz="0 -0.022 0" rpy="0 0 0"/>
-      <axis xyz="0 -1 0"/>
-      <limit lower="0.0" upper="0.025" effort="5.0" velocity="0.10"/>
-      <mimic joint="gripper_left_joint" multiplier="-1"/>
-    </joint>
-    <!-- TCP -->
+      <axis xyz="0 1 0"/>
+      <limit lower="-0.025" upper="0.0" effort="5.0" velocity="0.10"/>
+      <dynamics damping="0.01" friction="0.01"/>
+      <mimic joint="gripper_left_joint" multiplier="-1" offset="0"/>
+    </joint>
+    <!-- TCP frame -->
     <link name="tcp_link"/>
     <joint name="tcp_joint" type="fixed">
@@ -475,5 +537,83 @@
     </joint>
   </xacro:macro>
-  <!-- ── 8. INSTANTIATION ──────────────────────────────────────────── -->
+  <ros2_control name="OrionSystem" type="system">
+    <hardware>
+      <plugin>gz_ros2_control/GazeboSimSystem</plugin>
+    </hardware>
+    <!-- MECANUM DRIVE  (velocity commands)      -->
+    <joint name="front_left_wheel_joint">
+      <command_interface name="velocity">
+        <param name="min">-10.0</param>
+        <param name="max"> 10.0</param>
+      </command_interface>
+      <state_interface name="position"/>
+      <state_interface name="velocity"/>
+    </joint>
+    <joint name="front_right_wheel_joint">
+      <command_interface name="velocity">
+        <param name="min">-10.0</param>
+        <param name="max"> 10.0</param>
+      </command_interface>
+      <state_interface name="position"/>
+      <state_interface name="velocity"/>
+    </joint>
+    <joint name="rear_left_wheel_joint">
+      <command_interface name="velocity">
+        <param name="min">-10.0</param>
+        <param name="max"> 10.0</param>
+      </command_interface>
+      <state_interface name="position"/>
+      <state_interface name="velocity"/>
+    </joint>
+    <joint name="rear_right_wheel_joint">
+      <command_interface name="velocity">
+        <param name="min">-10.0</param>
+        <param name="max"> 10.0</param>
+      </command_interface>
+      <state_interface name="position"/>
+      <state_interface name="velocity"/>
+    </joint>
+    <!-- ARM  (position commands)               -->
+    <joint name="shoulder_joint">
+      <command_interface name="position">
+        <param name="min">-1.3</param>
+        <param name="max"> 1.57</param>
+      </command_interface>
+      <state_interface name="position"/>
+      <state_interface name="velocity"/>
+    </joint>
+    <joint name="elbow_joint">
+      <command_interface name="position">
+        <param name="min">-1.57</param>
+        <param name="max"> 0.57</param>
+      </command_interface>
+      <state_interface name="position"/>
+      <state_interface name="velocity"/>
+    </joint>
+    <joint name="wrist_joint">
+      <command_interface name="position">
+        <param name="min">0.0</param>
+        <param name="max">2.7</param>
+      </command_interface>
+      <state_interface name="position"/>
+      <state_interface name="velocity"/>
+    </joint>
+    <joint name="wrist_roll_joint">
+      <command_interface name="position">
+        <param name="min">-1.0</param>
+        <param name="max"> 1.0</param>
+      </command_interface>
+      <state_interface name="position"/>
+      <state_interface name="velocity"/>
+    </joint>
+    <joint name="gripper_left_joint">
+      <command_interface name="position">
+        <param name="min">0.0</param>
+        <param name="max">0.025</param>
+      </command_interface>
+      <state_interface name="position"/>
+      <state_interface name="velocity"/>
+    </joint>
+  </ros2_control>
   <xacro:base/>
   <xacro:wheels/>
